Commit message: Clearpath fixes and modifications.

File: jaco_model/urdf/standalone_arm.xacro (robot description, xacro)
@@ -20,5 +20,5 @@
 	  <box size = "0 0 0"/> <!--making it slightly bigger in x and z direction-->
 	</geometry>
-	<material name="Black" />
+	<!--<material name="Black" /> -->
       </visual>
       <collision>
@@ -29,5 +29,4 @@
       </collision>
     </link>
--->
 <xacro:jaco_arm  parent="root"/>
 </robot>
