Commit message: working on arm urdf

File: jaco_model/urdf/jaco_arm.xacro (robot description, xacro)
@@ -1,14 +1,14 @@
 <?xml version="1.0"?>
-<robot xmlns:xacro="http://www.ros.org/wiki/xacro" name="jaco_arm">
-<xacro:property name="width" value=".2" />
-<xacro:property name="bodylen" value=".6" />
-<link name="link_base">
-        <visual>
+<robot xmlns:xacro="http://www.ros.org/wiki/xacro" name="jaco_arm_link">
+  <property name="M_PI" value="3.1415926535897931" />
+<xacro:macro name="jaco_link" params="link_name link_origin_xyz link_origin_rpy">
+<link name="${link_name}">
+      <visual>
  <origin
-        xyz="0 0 0"
-        rpy="0 0 0" />
-                <geometry>
+        xyz="${link_origin_xyz}"
+        rpy="${link_origin_rpy}" />
+                 <geometry>
                          <mesh
-          filename="package://jaco_model/meshes/link_base.dae"/>
+          filename="package://jaco_model/meshes/${link_name}.dae"/>
                 </geometry>
                 <material name="carbon_fiber">
@@ -17,12 +17,41 @@
         </visual>
         <collision>
- <origin
-        xyz="0 0 0"
-        rpy="0 0 0" />
+  <origin
+        xyz="${link_origin_xyz}"
+        rpy="${link_origin_rpy}" />
                 <geometry>
                          <mesh
-          filename="package://jaco_model/meshes/link_base.dae"/>
+          filename="package://jaco_model/meshes/${link_name}.dae"/>
                 </geometry>
         </collision>
 </link>
+</xacro:macro>
+<xacro:macro name="jaco_joint" params="joint_name parent child">
+<joint name="${joint_name}" type="continuous">
+    <parent link="${parent}"/>
+    <child link="${child}"/>
+ </joint>
+</xacro:macro>
+  <property name="link_base" value="jaco_link_base" />
+  <property name="link_1" value="jaco_link_1" />
+  <property name="link_2" value="jaco_link_2" />
+  <property name="link_3" value="jaco_link_3" />
+  <property name="link_4" value="jaco_link_4" />
+  <property name="link_5" value="jaco_link_5" />
+  <property name="link_hand" value="jaco_link_hand" />
+  <property name="joint_1" value="jaco_joint_1" />
+  <property name="joint_2" value="jaco_joint_2" />
+  <property name="joint_3" value="jaco_joint_3" />
+  <property name="joint_4" value="jaco_joint_4" />
+  <property name="joint_5" value="jaco_joint_5" />
+  <property name="joint_6" value="jaco_joint_6" />
+<xacro:jaco_link link_name="${link_base}" link_origin_xyz="0 0 0" link_origin_rpy="0 0 0"/>
+<xacro:jaco_link link_name="${link_1}" link_origin_xyz="0 0 0.1535" link_origin_rpy="${M_PI} 0 0"/>
+<xacro:jaco_joint joint_name="${joint_1}" parent="${link_base}" child="${link_1}"/>
+<xacro:jaco_link link_name="${link_2}" link_origin_xyz="0 0 0.272" link_origin_rpy="0 ${M_PI/2} -${M_PI/2}"/>
+<xacro:jaco_joint joint_name="${joint_2}" parent="${link_1}" child="${link_2}"/>
+<xacro:jaco_link link_name="${link_3}" link_origin_xyz="0 0 -0.138" link_origin_rpy="0 -${M_PI/2} -${M_PI/2}"/>
+<xacro:jaco_joint joint_name="${joint_3}" parent="${link_2}" child="${link_3}"/>
+<xacro:jaco_link link_name="${link_4}" link_origin_xyz="0 0 -0.138" link_origin_rpy="0 -${M_PI/2} -${M_PI/2}"/>
+<xacro:jaco_joint joint_name="${joint_4}" parent="${link_3}" child="${link_4}"/>
 </robot>

Commit message: completed urdf.  still does not work with moveit

File: jaco_model/urdf/jaco_arm.xacro (robot description, xacro)
@@ -2,10 +2,7 @@
 <robot xmlns:xacro="http://www.ros.org/wiki/xacro" name="jaco_arm_link">
   <property name="M_PI" value="3.1415926535897931" />
-<xacro:macro name="jaco_link" params="link_name link_origin_xyz link_origin_rpy">
+<xacro:macro name="jaco_link" params="link_name">
 <link name="${link_name}">
       <visual>
- <origin
-        xyz="${link_origin_xyz}"
-        rpy="${link_origin_rpy}" />
                  <geometry>
                          <mesh
@@ -17,7 +14,4 @@
         </visual>
         <collision>
-  <origin
-        xyz="${link_origin_xyz}"
-        rpy="${link_origin_rpy}" />
                 <geometry>
                          <mesh
@@ -27,8 +21,10 @@
 </link>
 </xacro:macro>
-<xacro:macro name="jaco_joint" params="joint_name parent child">
-<joint name="${joint_name}" type="continuous">
+<xacro:macro name="jaco_joint" params="joint_name type parent child joint_axis_xyz joint_origin_xyz joint_origin_rpy">
+<joint name="${joint_name}" type="${type}">
     <parent link="${parent}"/>
     <child link="${child}"/>
+    <axis xyz="${joint_axis_xyz}"/>
+<origin xyz="${joint_origin_xyz}" rpy="${joint_origin_rpy}"/>
  </joint>
 </xacro:macro>
@@ -40,22 +36,46 @@
   <property name="link_5" value="jaco_link_5" />
   <property name="link_hand" value="jaco_link_hand" />
+  <property name="world" value="world" />
+  <property name="joint_base" value="jaco_joint_base" />
+  <property name="joint_base_axis_xyz" value="0 0 0" />
+  <property name="joint_base_origin_xyz" value="0 0 0" />
+  <property name="joint_base_origin_rpy" value="0 0 0" />
   <property name="joint_1" value="jaco_joint_1" />
+  <property name="joint_1_axis_xyz" value="0 0 1" />
+  <property name="joint_1_origin_xyz" value="0 0 0.1535" />
+  <property name="joint_1_origin_rpy" value="${M_PI} 0 0" />
   <property name="joint_2" value="jaco_joint_2" />
+  <property name="joint_2_axis_xyz" value="0 0 1" />
+  <property name="joint_2_origin_xyz" value="0 0 -0.1185" />
+  <property name="joint_2_origin_rpy" value="-${M_PI/2} -${M_PI/2} 0" />
   <property name="joint_3" value="jaco_joint_3" />
+  <property name="joint_3_axis_xyz" value="0 0 1" />
+  <property name="joint_3_origin_xyz" value="0.41 0 0" />
+  <property name="joint_3_origin_rpy" value="${M_PI} 0 ${M_PI}" />
   <property name="joint_4" value="jaco_joint_4" />
+  <property name="joint_4_axis_xyz" value="0 0 1" />
+  <property name="joint_4_origin_xyz" value="0.207 0 -0.01125" />
+  <property name="joint_4_origin_rpy" value="0 -${M_PI/2} 0" />
   <property name="joint_5" value="jaco_joint_5" />
+  <property name="joint_5_axis_xyz" value="0 0 1" />
+  <property name="joint_5_origin_xyz" value="0.0343 0 -0.06588" />
+  <property name="joint_5_origin_rpy" value="0 ${M_PI/36*11} ${M_PI}" />
   <property name="joint_6" value="jaco_joint_6" />
-<xacro:jaco_link link_name="${link_base}" link_origin_xyz="0 0 0" link_origin_rpy="0 0 0"/>
-<xacro:jaco_link link_name="${link_1}" link_origin_xyz="0 0 0.1535" link_origin_rpy="${M_PI} 0 0"/>
-<xacro:jaco_joint joint_name="${joint_1}" parent="${link_base}" child="${link_1}"/>
-<xacro:jaco_link link_name="${link_2}" link_origin_xyz="0 0 0.272" link_origin_rpy="0 ${M_PI/2} -${M_PI/2}"/>
-<xacro:jaco_joint joint_name="${joint_2}" parent="${link_1}" child="${link_2}"/>
-<xacro:jaco_link link_name="${link_3}" link_origin_xyz="0 0 -0.138" link_origin_rpy="0 -${M_PI/2} -${M_PI/2}"/>
-<xacro:jaco_joint joint_name="${joint_3}" parent="${link_2}" child="${link_3}"/>
-<xacro:jaco_link link_name="${link_4}" link_origin_xyz="0 -0.01125 0.069" link_origin_rpy="${M_PI} 0 ${M_PI/2}"/>
-<xacro:jaco_joint joint_name="${joint_4}" parent="${link_3}" child="${link_4}"/>
-<xacro:jaco_link link_name="${link_5}" link_origin_xyz="0 0.02305 0.13488" link_origin_rpy="0 -${M_PI/2+M_PI/36*7} ${M_PI/2}"/>
-<xacro:jaco_joint joint_name="${joint_5}" parent="${link_4}" child="${link_5}"/>
-<xacro:jaco_link link_name="${link_hand}" link_origin_xyz="0 0.05735 0.20076" link_origin_rpy="${M_PI/2} ${M_PI/2} 0"/>
-<xacro:jaco_joint joint_name="${joint_6}" parent="${link_5}" child="${link_hand}"/>
+  <property name="joint_6_axis_xyz" value="0 0 1" />
+  <property name="joint_hand_origin_xyz" value="0.0343 0 -0.06588" />
+  <property name="joint_hand_origin_rpy" value="0 ${M_PI/36*11} ${M_PI}" />
+<xacro:jaco_link link_name="${link_base}"/>
+<!--<xacro:jaco_joint joint_name="${joint_base}" type="fixed" parent="${world}" child="${link_base}" joint_axis_xyz="${joint_base_axis_xyz}" joint_origin_xyz="${joint_base_origin_xyz}" joint_origin_rpy="${joint_base_origin_rpy}"/>-->
+<xacro:jaco_link link_name="${link_1}"/>
+<xacro:jaco_joint joint_name="${joint_1}" type="continuous" parent="${link_base}" child="${link_1}" joint_axis_xyz="${joint_1_axis_xyz}" joint_origin_xyz="${joint_1_origin_xyz}" joint_origin_rpy="${joint_1_origin_rpy}"/>
+<xacro:jaco_link link_name="${link_2}"/>
+<xacro:jaco_joint joint_name="${joint_2}" type="continuous" parent="${link_1}" child="${link_2}" joint_axis_xyz="${joint_2_axis_xyz}" joint_origin_xyz="${joint_2_origin_xyz}" joint_origin_rpy="${joint_2_origin_rpy}"/>
+<xacro:jaco_link link_name="${link_3}"/>
+<xacro:jaco_joint joint_name="${joint_3}" type="continuous" parent="${link_2}" child="${link_3}" joint_axis_xyz="${joint_3_axis_xyz}" joint_origin_xyz="${joint_3_origin_xyz}" joint_origin_rpy="${joint_3_origin_rpy}"/>
+<xacro:jaco_link link_name="${link_4}"/>
+<xacro:jaco_joint joint_name="${joint_4}" type="continuous" parent="${link_3}" child="${link_4}" joint_axis_xyz="${joint_4_axis_xyz}" joint_origin_xyz="${joint_4_origin_xyz}" joint_origin_rpy="${joint_4_origin_rpy}"/>
+<xacro:jaco_link link_name="${link_5}"/>
+<xacro:jaco_joint joint_name="${joint_5}" type="continuous" parent="${link_4}" child="${link_5}" joint_axis_xyz="${joint_5_axis_xyz}" joint_origin_xyz="${joint_5_origin_xyz}" joint_origin_rpy="${joint_5_origin_rpy}"/>
+<xacro:jaco_link link_name="${link_hand}"/>
+<xacro:jaco_joint joint_name="${joint_6}" type="continuous" parent="${link_5}" child="${link_hand}" joint_axis_xyz="${joint_6_axis_xyz}" joint_origin_xyz="${joint_hand_origin_xyz}" joint_origin_rpy="${joint_hand_origin_rpy}"/>
 </robot>

Commit message: added moveit files

File: jaco_model/urdf/jaco_arm.xacro (robot description, xacro)
@@ -1,5 +1,52 @@
 <?xml version="1.0"?>
-<robot xmlns:xacro="http://www.ros.org/wiki/xacro" name="jaco_arm_link">
-  <property name="M_PI" value="3.1415926535897931" />
+<root xmlns:xi="http://www.w3.org/2001/XInclude"
+	xmlns:gazebo="http://playerstage.sourceforge.net/gazebo/xmlschema/#gz"
+    xmlns:model="http://playerstage.sourceforge.net/gazebo/xmlschema/#model"
+	xmlns:sensor="http://playerstage.sourceforge.net/gazebo/xmlschema/#sensor"
+	xmlns:body="http://playerstage.sourceforge.net/gazebo/xmlschema/#body"
+    xmlns:geom="http://playerstage.sourceforge.net/gazebo/xmlschema/#geom"
+    xmlns:joint="http://playerstage.sourceforge.net/gazebo/xmlschema/#joint"
+	xmlns:controller="http://playerstage.sourceforge.net/gazebo/xmlschema/#controller"
+	xmlns:interface="http://playerstage.sourceforge.net/gazebo/xmlschema/#interface"
+	xmlns:rendering="http://playerstage.sourceforge.net/gazebo/xmlschema/#rendering"
+    xmlns:renderable="http://playerstage.sourceforge.net/gazebo/xmlschema/#renderable"
+    xmlns:physics="http://playerstage.sourceforge.net/gazebo/xmlschema/#physics"
+	xmlns:xacro="http://ros.org/wiki/xacro">
+  <property name="J_PI" value="3.1415926535897931" />
+  <property name="link_base" value="jaco_link_base" />
+  <property name="link_1" value="jaco_link_1" />
+  <property name="link_2" value="jaco_link_2" />
+  <property name="link_3" value="jaco_link_3" />
+  <property name="link_4" value="jaco_link_4" />
+  <property name="link_5" value="jaco_link_5" />
+  <property name="link_hand" value="jaco_link_hand" />
+  <property name="joint_base" value="jaco_joint_base" />
+  <property name="joint_base_axis_xyz" value="0 0 0" />
+  <property name="joint_base_origin_xyz" value="0 0 0" />
+  <property name="joint_base_origin_rpy" value="0 0 0" />
+  <property name="joint_1" value="jaco_joint_1" />
+  <property name="joint_1_axis_xyz" value="0 0 1" />
+  <property name="joint_1_origin_xyz" value="0 0 0.1535" />
+  <property name="joint_1_origin_rpy" value="${J_PI} 0 0" />
+  <property name="joint_2" value="jaco_joint_2" />
+  <property name="joint_2_axis_xyz" value="0 0 1" />
+  <property name="joint_2_origin_xyz" value="0 0 -0.1185" />
+  <property name="joint_2_origin_rpy" value="-${J_PI/2} -${J_PI/2} 0" />
+  <property name="joint_3" value="jaco_joint_3" />
+  <property name="joint_3_axis_xyz" value="0 0 1" />
+  <property name="joint_3_origin_xyz" value="0.41 0 0" />
+  <property name="joint_3_origin_rpy" value="${J_PI} 0 ${J_PI}" />
+  <property name="joint_4" value="jaco_joint_4" />
+  <property name="joint_4_axis_xyz" value="0 0 1" />
+  <property name="joint_4_origin_xyz" value="0.207 0 -0.01125" />
+  <property name="joint_4_origin_rpy" value="0 -${J_PI/2} 0" />
+  <property name="joint_5" value="jaco_joint_5" />
+  <property name="joint_5_axis_xyz" value="0 0 1" />
+  <property name="joint_5_origin_xyz" value="0.0343 0 -0.06588" />
+  <property name="joint_5_origin_rpy" value="0 ${J_PI/36*11} ${J_PI}" />
+  <property name="joint_6" value="jaco_joint_6" />
+  <property name="joint_6_axis_xyz" value="0 0 1" />
+  <property name="joint_hand_origin_xyz" value="0.0343 0 -0.06588" />
+  <property name="joint_hand_origin_rpy" value="0 ${J_PI/36*11} ${J_PI}" />
 <xacro:macro name="jaco_link" params="link_name">
 <link name="${link_name}">
@@ -29,53 +76,19 @@
  </joint>
 </xacro:macro>
-  <property name="link_base" value="jaco_link_base" />
-  <property name="link_1" value="jaco_link_1" />
-  <property name="link_2" value="jaco_link_2" />
-  <property name="link_3" value="jaco_link_3" />
-  <property name="link_4" value="jaco_link_4" />
-  <property name="link_5" value="jaco_link_5" />
-  <property name="link_hand" value="jaco_link_hand" />
-  <property name="world" value="world" />
-  <property name="joint_base" value="jaco_joint_base" />
-  <property name="joint_base_axis_xyz" value="0 0 0" />
-  <property name="joint_base_origin_xyz" value="0 0 0" />
-  <property name="joint_base_origin_rpy" value="0 0 0" />
-  <property name="joint_1" value="jaco_joint_1" />
-  <property name="joint_1_axis_xyz" value="0 0 1" />
-  <property name="joint_1_origin_xyz" value="0 0 0.1535" />
-  <property name="joint_1_origin_rpy" value="${M_PI} 0 0" />
-  <property name="joint_2" value="jaco_joint_2" />
-  <property name="joint_2_axis_xyz" value="0 0 1" />
-  <property name="joint_2_origin_xyz" value="0 0 -0.1185" />
-  <property name="joint_2_origin_rpy" value="-${M_PI/2} -${M_PI/2} 0" />
-  <property name="joint_3" value="jaco_joint_3" />
-  <property name="joint_3_axis_xyz" value="0 0 1" />
-  <property name="joint_3_origin_xyz" value="0.41 0 0" />
-  <property name="joint_3_origin_rpy" value="${M_PI} 0 ${M_PI}" />
-  <property name="joint_4" value="jaco_joint_4" />
-  <property name="joint_4_axis_xyz" value="0 0 1" />
-  <property name="joint_4_origin_xyz" value="0.207 0 -0.01125" />
-  <property name="joint_4_origin_rpy" value="0 -${M_PI/2} 0" />
-  <property name="joint_5" value="jaco_joint_5" />
-  <property name="joint_5_axis_xyz" value="0 0 1" />
-  <property name="joint_5_origin_xyz" value="0.0343 0 -0.06588" />
-  <property name="joint_5_origin_rpy" value="0 ${M_PI/36*11} ${M_PI}" />
-  <property name="joint_6" value="jaco_joint_6" />
-  <property name="joint_6_axis_xyz" value="0 0 1" />
-  <property name="joint_hand_origin_xyz" value="0.0343 0 -0.06588" />
-  <property name="joint_hand_origin_rpy" value="0 ${M_PI/36*11} ${M_PI}" />
-<xacro:jaco_link link_name="${link_base}"/>
-<!--<xacro:jaco_joint joint_name="${joint_base}" type="fixed" parent="${world}" child="${link_base}" joint_axis_xyz="${joint_base_axis_xyz}" joint_origin_xyz="${joint_base_origin_xyz}" joint_origin_rpy="${joint_base_origin_rpy}"/>-->
-<xacro:jaco_link link_name="${link_1}"/>
-<xacro:jaco_joint joint_name="${joint_1}" type="continuous" parent="${link_base}" child="${link_1}" joint_axis_xyz="${joint_1_axis_xyz}" joint_origin_xyz="${joint_1_origin_xyz}" joint_origin_rpy="${joint_1_origin_rpy}"/>
-<xacro:jaco_link link_name="${link_2}"/>
-<xacro:jaco_joint joint_name="${joint_2}" type="continuous" parent="${link_1}" child="${link_2}" joint_axis_xyz="${joint_2_axis_xyz}" joint_origin_xyz="${joint_2_origin_xyz}" joint_origin_rpy="${joint_2_origin_rpy}"/>
-<xacro:jaco_link link_name="${link_3}"/>
-<xacro:jaco_joint joint_name="${joint_3}" type="continuous" parent="${link_2}" child="${link_3}" joint_axis_xyz="${joint_3_axis_xyz}" joint_origin_xyz="${joint_3_origin_xyz}" joint_origin_rpy="${joint_3_origin_rpy}"/>
-<xacro:jaco_link link_name="${link_4}"/>
-<xacro:jaco_joint joint_name="${joint_4}" type="continuous" parent="${link_3}" child="${link_4}" joint_axis_xyz="${joint_4_axis_xyz}" joint_origin_xyz="${joint_4_origin_xyz}" joint_origin_rpy="${joint_4_origin_rpy}"/>
-<xacro:jaco_link link_name="${link_5}"/>
-<xacro:jaco_joint joint_name="${joint_5}" type="continuous" parent="${link_4}" child="${link_5}" joint_axis_xyz="${joint_5_axis_xyz}" joint_origin_xyz="${joint_5_origin_xyz}" joint_origin_rpy="${joint_5_origin_rpy}"/>
-<xacro:jaco_link link_name="${link_hand}"/>
-<xacro:jaco_joint joint_name="${joint_6}" type="continuous" parent="${link_5}" child="${link_hand}" joint_axis_xyz="${joint_6_axis_xyz}" joint_origin_xyz="${joint_hand_origin_xyz}" joint_origin_rpy="${joint_hand_origin_rpy}"/>
-</robot>
+<xacro:macro name="jaco_arm" params="parent">
+   <xacro:jaco_link link_name="${link_base}"/>
+   <xacro:jaco_joint joint_name="${joint_base}" type="fixed" parent="${parent}" child="${link_base}" joint_axis_xyz="${joint_base_axis_xyz}" joint_origin_xyz="${joint_base_origin_xyz}" joint_origin_rpy="${joint_base_origin_rpy}"/>
+   <xacro:jaco_link link_name="${link_1}"/>
+   <xacro:jaco_joint joint_name="${joint_1}" type="continuous" parent="${link_base}" child="${link_1}" joint_axis_xyz="${joint_1_axis_xyz}" joint_origin_xyz="${joint_1_origin_xyz}" joint_origin_rpy="${joint_1_origin_rpy}"/>
+   <xacro:jaco_link link_name="${link_2}"/>
+   <xacro:jaco_joint joint_name="${joint_2}" type="continuous" parent="${link_1}" child="${link_2}" joint_axis_xyz="${joint_2_axis_xyz}" joint_origin_xyz="${joint_2_origin_xyz}" joint_origin_rpy="${joint_2_origin_rpy}"/>
+   <xacro:jaco_link link_name="${link_3}"/>
+   <xacro:jaco_joint joint_name="${joint_3}" type="continuous" parent="${link_2}" child="${link_3}" joint_axis_xyz="${joint_3_axis_xyz}" joint_origin_xyz="${joint_3_origin_xyz}" joint_origin_rpy="${joint_3_origin_rpy}"/>
+   <xacro:jaco_link link_name="${link_4}"/>
+   <xacro:jaco_joint joint_name="${joint_4}" type="continuous" parent="${link_3}" child="${link_4}" joint_axis_xyz="${joint_4_axis_xyz}" joint_origin_xyz="${joint_4_origin_xyz}" joint_origin_rpy="${joint_4_origin_rpy}"/>
+   <xacro:jaco_link link_name="${link_5}"/>
+   <xacro:jaco_joint joint_name="${joint_5}" type="continuous" parent="${link_4}" child="${link_5}" joint_axis_xyz="${joint_5_axis_xyz}" joint_origin_xyz="${joint_5_origin_xyz}" joint_origin_rpy="${joint_5_origin_rpy}"/>
+   <xacro:jaco_link link_name="${link_hand}"/>
+   <xacro:jaco_joint joint_name="${joint_6}" type="continuous" parent="${link_5}" child="${link_hand}" joint_axis_xyz="${joint_6_axis_xyz}" joint_origin_xyz="${joint_hand_origin_xyz}" joint_origin_rpy="${joint_hand_origin_rpy}"/>
+</xacro:macro>
+</root>
