Commit message: updated model

File: jaco_model/urdf/jaco_arm.xacro (robot description, xacro)
@@ -56,12 +56,18 @@
   <property name="joint_finger_1_origin_xyz" value="-0.03978 0 -0.10071" />
   <property name="joint_finger_1_origin_rpy" value="-1.7983 1.117 3.1416" />
+  <property name="joint_finger_1_lower_limit" value="0" />
+  <property name="joint_finger_1_upper_limit" value="${J_PI/180*40}" />
   <property name="joint_finger_2" value="jaco_joint_finger_2" />
   <property name="joint_finger_2_axis_xyz" value="0 0 1" />
   <property name="joint_finger_2_origin_xyz" value="0.03569 -0.0216 -0.10071" />
   <property name="joint_finger_2_origin_rpy" value="-1.6222 1.117 -0.23615" />
+  <property name="joint_finger_2_lower_limit" value="0" />
+  <property name="joint_finger_2_upper_limit" value="${J_PI/180*40}" />
   <property name="joint_finger_3" value="jaco_joint_finger_3" />
   <property name="joint_finger_3_axis_xyz" value="0 0 1" />
   <property name="joint_finger_3_origin_xyz" value="0.03569 0.0216 -0.10071" />
   <property name="joint_finger_3_origin_rpy" value="-1.5161 1.1459 0.23978" />
+  <property name="joint_finger_3_lower_limit" value="0" />
+  <property name="joint_finger_3_upper_limit" value="${J_PI/180*40}" />
 <xacro:macro name="jaco_link" params="link_name">
 <link name="${link_name}">
@@ -91,4 +97,13 @@
  </joint>
 </xacro:macro>
+<xacro:macro name="jaco_finger_joint" params="joint_name type parent child joint_axis_xyz joint_origin_xyz joint_origin_rpy lower_limit upper_limit">
+<joint name="${joint_name}" type="${type}">
+    <parent link="${parent}"/>
+    <child link="${child}"/>
+    <axis xyz="${joint_axis_xyz}"/>
+<origin xyz="${joint_origin_xyz}" rpy="${joint_origin_rpy}"/>
+    <limit lower="${lower_limit}" upper="${upper_limit}" effort="30" velocity="5"/>
+ </joint>
+</xacro:macro>
 <xacro:macro name="jaco_arm" params="parent">
    <xacro:jaco_link link_name="${link_base}"/>
@@ -107,9 +122,9 @@
    <xacro:jaco_joint joint_name="${joint_6}" type="continuous" parent="${link_5}" child="${link_hand}" joint_axis_xyz="${joint_6_axis_xyz}" joint_origin_xyz="${joint_6_origin_xyz}" joint_origin_rpy="${joint_6_origin_rpy}"/>
    <xacro:jaco_link link_name="${link_finger_1}"/>
-   <xacro:jaco_joint joint_name="${joint_finger_1}" type="continuous" parent="${link_hand}" child="${link_finger_1}" joint_axis_xyz="${joint_finger_1_axis_xyz}" joint_origin_xyz="${joint_finger_1_origin_xyz}" joint_origin_rpy="${joint_finger_1_origin_rpy}"/>
+   <xacro:jaco_finger_joint joint_name="${joint_finger_1}" type="revolute" parent="${link_hand}" child="${link_finger_1}" joint_axis_xyz="${joint_finger_1_axis_xyz}" joint_origin_xyz="${joint_finger_1_origin_xyz}" joint_origin_rpy="${joint_finger_1_origin_rpy}" lower_limit="${joint_finger_1_lower_limit}" upper_limit="${joint_finger_1_upper_limit}"/>
    <xacro:jaco_link link_name="${link_finger_2}"/>
-   <xacro:jaco_joint joint_name="${joint_finger_2}" type="continuous" parent="${link_hand}" child="${link_finger_2}" joint_axis_xyz="${joint_finger_2_axis_xyz}" joint_origin_xyz="${joint_finger_2_origin_xyz}" joint_origin_rpy="${joint_finger_2_origin_rpy}"/>
+   <xacro:jaco_finger_joint joint_name="${joint_finger_2}" type="revolute" parent="${link_hand}" child="${link_finger_2}" joint_axis_xyz="${joint_finger_2_axis_xyz}" joint_origin_xyz="${joint_finger_2_origin_xyz}" joint_origin_rpy="${joint_finger_2_origin_rpy}" lower_limit="${joint_finger_2_lower_limit}" upper_limit="${joint_finger_2_upper_limit}"/>
    <xacro:jaco_link link_name="${link_finger_3}"/>
-   <xacro:jaco_joint joint_name="${joint_finger_3}" type="continuous" parent="${link_hand}" child="${link_finger_3}" joint_axis_xyz="${joint_finger_3_axis_xyz}" joint_origin_xyz="${joint_finger_3_origin_xyz}" joint_origin_rpy="${joint_finger_3_origin_rpy}"/>
+   <xacro:jaco_finger_joint joint_name="${joint_finger_3}" type="revolute" parent="${link_hand}" child="${link_finger_3}" joint_axis_xyz="${joint_finger_3_axis_xyz}" joint_origin_xyz="${joint_finger_3_origin_xyz}" joint_origin_rpy="${joint_finger_3_origin_rpy}" lower_limit="${joint_finger_3_lower_limit}" upper_limit="${joint_finger_3_upper_limit}"/>
 </xacro:macro>
 </root>

File: jaco_model/urdf/standalone_arm.urdf (robot description, URDF)
Before this commit: robot jaco, 8 links, 7 joints
Links:
- added link jaco_link_finger_1; collision mesh filename=package://jaco_model/meshes/jaco_link_finger_1.dae; visual mesh filename=package://jaco_model/meshes/jaco_link_finger_1.dae
- added link jaco_link_finger_2; collision mesh filename=package://jaco_model/meshes/jaco_link_finger_2.dae; visual mesh filename=package://jaco_model/meshes/jaco_link_finger_2.dae
- added link jaco_link_finger_3; collision mesh filename=package://jaco_model/meshes/jaco_link_finger_3.dae; visual mesh filename=package://jaco_model/meshes/jaco_link_finger_3.dae
Joints:
- added joint jaco_joint_finger_1: type revolute, parent jaco_link_hand, child jaco_link_finger_1, origin xyz=-0.03978 0 -0.10071 rpy=-1.7983 1.117 3.1416, axis 0 0 1, limit lower=0 upper=0.698131700798 effort=30 velocity=5
- added joint jaco_joint_finger_2: type revolute, parent jaco_link_hand, child jaco_link_finger_2, origin xyz=0.03569 -0.0216 -0.10071 rpy=-1.6222 1.117 -0.23615, axis 0 0 1, limit lower=0 upper=0.698131700798 effort=30 velocity=5
- added joint jaco_joint_finger_3: type revolute, parent jaco_link_hand, child jaco_link_finger_3, origin xyz=0.03569 0.0216 -0.10071 rpy=-1.5161 1.1459 0.23978, axis 0 0 1, limit lower=0 upper=0.698131700798 effort=30 velocity=5

Commit message: Missing updates from commit 3b7211b.

File: jaco_model/urdf/jaco_arm.xacro (robot description, xacro)
@@ -24,4 +24,6 @@
   <property name="link_finger_2" value="jaco_link_finger_2" />
   <property name="link_finger_3" value="jaco_link_finger_3" />
+  <property name="api_offset" value="0.028" />
+  <property name="api_origin" value="jaco_api_origin" />
   <property name="joint_base" value="jaco_joint_base" />
   <property name="joint_base_axis_xyz" value="0 0 0" />
@@ -70,61 +72,13 @@
   <property name="joint_finger_3_lower_limit" value="0" />
   <property name="joint_finger_3_upper_limit" value="${J_PI/180*40}" />
-<xacro:macro name="jaco_link" params="link_name">
-<link name="${link_name}">
-      <visual>
-                 <geometry>
-                         <mesh
-          filename="package://jaco_model/meshes/${link_name}.dae"/>
-                </geometry>
-                <material name="carbon_fiber">
- 			<color rgba="0.792156862745098 0.819607843137255 0.933333333333333 1" />
-                </material>
-        </visual>
-        <collision>
-                <geometry>
-                         <mesh
-          filename="package://jaco_model/meshes/${link_name}.dae"/>
-                </geometry>
-        </collision>
-</link>
-</xacro:macro>
-<xacro:macro name="jaco_joint" params="joint_name type parent child joint_axis_xyz joint_origin_xyz joint_origin_rpy">
-<joint name="${joint_name}" type="${type}">
-    <parent link="${parent}"/>
-    <child link="${child}"/>
-    <axis xyz="${joint_axis_xyz}"/>
-<origin xyz="${joint_origin_xyz}" rpy="${joint_origin_rpy}"/>
- </joint>
-</xacro:macro>
-<xacro:macro name="jaco_finger_joint" params="joint_name type parent child joint_axis_xyz joint_origin_xyz joint_origin_rpy lower_limit upper_limit">
-<joint name="${joint_name}" type="${type}">
-    <parent link="${parent}"/>
-    <child link="${child}"/>
-    <axis xyz="${joint_axis_xyz}"/>
-<origin xyz="${joint_origin_xyz}" rpy="${joint_origin_rpy}"/>
-    <limit lower="${lower_limit}" upper="${upper_limit}" effort="30" velocity="5"/>
- </joint>
-</xacro:macro>
-<xacro:macro name="jaco_arm" params="parent">
-   <xacro:jaco_link link_name="${link_base}"/>
-   <xacro:jaco_joint joint_name="${joint_base}" type="fixed" parent="${parent}" child="${link_base}" joint_axis_xyz="${joint_base_axis_xyz}" joint_origin_xyz="${joint_base_origin_xyz}" joint_origin_rpy="${joint_base_origin_rpy}"/>
-   <xacro:jaco_link link_name="${link_1}"/>
-   <xacro:jaco_joint joint_name="${joint_1}" type="continuous" parent="${link_base}" child="${link_1}" joint_axis_xyz="${joint_1_axis_xyz}" joint_origin_xyz="${joint_1_origin_xyz}" joint_origin_rpy="${joint_1_origin_rpy}"/>
-   <xacro:jaco_link link_name="${link_2}"/>
-   <xacro:jaco_joint joint_name="${joint_2}" type="continuous" parent="${link_1}" child="${link_2}" joint_axis_xyz="${joint_2_axis_xyz}" joint_origin_xyz="${joint_2_origin_xyz}" joint_origin_rpy="${joint_2_origin_rpy}"/>
-   <xacro:jaco_link link_name="${link_3}"/>
-   <xacro:jaco_joint joint_name="${joint_3}" type="continuous" parent="${link_2}" child="${link_3}" joint_axis_xyz="${joint_3_axis_xyz}" joint_origin_xyz="${joint_3_origin_xyz}" joint_origin_rpy="${joint_3_origin_rpy}"/>
-   <xacro:jaco_link link_name="${link_4}"/>
-   <xacro:jaco_joint joint_name="${joint_4}" type="continuous" parent="${link_3}" child="${link_4}" joint_axis_xyz="${joint_4_axis_xyz}" joint_origin_xyz="${joint_4_origin_xyz}" joint_origin_rpy="${joint_4_origin_rpy}"/>
-   <xacro:jaco_link link_name="${link_5}"/>
-   <xacro:jaco_joint joint_name="${joint_5}" type="continuous" parent="${link_4}" child="${link_5}" joint_axis_xyz="${joint_5_axis_xyz}" joint_origin_xyz="${joint_5_origin_xyz}" joint_origin_rpy="${joint_5_origin_rpy}"/>
-   <xacro:jaco_link link_name="${link_hand}"/>
-   <xacro:jaco_joint joint_name="${joint_6}" type="continuous" parent="${link_5}" child="${link_hand}" joint_axis_xyz="${joint_6_axis_xyz}" joint_origin_xyz="${joint_6_origin_xyz}" joint_origin_rpy="${joint_6_origin_rpy}"/>
-   <xacro:jaco_link link_name="${link_finger_1}"/>
-   <xacro:jaco_finger_joint joint_name="${joint_finger_1}" type="revolute" parent="${link_hand}" child="${link_finger_1}" joint_axis_xyz="${joint_finger_1_axis_xyz}" joint_origin_xyz="${joint_finger_1_origin_xyz}" joint_origin_rpy="${joint_finger_1_origin_rpy}" lower_limit="${joint_finger_1_lower_limit}" upper_limit="${joint_finger_1_upper_limit}"/>
-   <xacro:jaco_link link_name="${link_finger_2}"/>
-   <xacro:jaco_finger_joint joint_name="${joint_finger_2}" type="revolute" parent="${link_hand}" child="${link_finger_2}" joint_axis_xyz="${joint_finger_2_axis_xyz}" joint_origin_xyz="${joint_finger_2_origin_xyz}" joint_origin_rpy="${joint_finger_2_origin_rpy}" lower_limit="${joint_finger_2_lower_limit}" upper_limit="${joint_finger_2_upper_limit}"/>
-   <xacro:jaco_link link_name="${link_finger_3}"/>
-   <xacro:jaco_finger_joint joint_name="${joint_finger_3}" type="revolute" parent="${link_hand}" child="${link_finger_3}" joint_axis_xyz="${joint_finger_3_axis_xyz}" joint_origin_xyz="${joint_finger_3_origin_xyz}" joint_origin_rpy="${joint_finger_3_origin_rpy}" lower_limit="${joint_finger_3_lower_limit}" upper_limit="${joint_finger_3_upper_limit}"/>
-</xacro:macro>
+  <xacro:include filename="$(find jaco_model)/urdf/jaco_common.xacro" />
+  <xacro:macro name="jaco_arm" params="parent">
+    <xacro:jaco_struct parent="${parent}" basename="jaco"/>
+    <xacro:jaco_link link_name="${link_finger_1}"/>
+    <xacro:jaco_finger_joint joint_name="${joint_finger_1}" type="revolute" parent="${link_hand}" child="${link_finger_1}" joint_axis_xyz="${joint_finger_1_axis_xyz}" joint_origin_xyz="${joint_finger_1_origin_xyz}" joint_origin_rpy="${joint_finger_1_origin_rpy}" lower_limit="${joint_finger_1_lower_limit}" upper_limit="${joint_finger_1_upper_limit}"/>
+    <xacro:jaco_link link_name="${link_finger_2}"/>
+    <xacro:jaco_finger_joint joint_name="${joint_finger_2}" type="revolute" parent="${link_hand}" child="${link_finger_2}" joint_axis_xyz="${joint_finger_2_axis_xyz}" joint_origin_xyz="${joint_finger_2_origin_xyz}" joint_origin_rpy="${joint_finger_2_origin_rpy}" lower_limit="${joint_finger_2_lower_limit}" upper_limit="${joint_finger_2_upper_limit}"/>
+    <xacro:jaco_link link_name="${link_finger_3}"/>
+    <xacro:jaco_finger_joint joint_name="${joint_finger_3}" type="revolute" parent="${link_hand}" child="${link_finger_3}" joint_axis_xyz="${joint_finger_3_axis_xyz}" joint_origin_xyz="${joint_finger_3_origin_xyz}" joint_origin_rpy="${joint_finger_3_origin_rpy}" lower_limit="${joint_finger_3_lower_limit}" upper_limit="${joint_finger_3_upper_limit}"/>
+  </xacro:macro>
 </root>

File: jaco_model/urdf/mico_arm.xacro (robot description, xacro)
@@ -24,4 +24,6 @@
   <property name="link_finger_2" value="mico_link_finger_2" />
   <property name="link_finger_3" value="mico_link_finger_3" />
+  <property name="api_offset" value="0.028" />
+  <property name="api_origin" value="mico_api_origin" />
   <property name="joint_base" value="mico_joint_base" />
   <property name="joint_base_axis_xyz" value="0 0 0" />
@@ -64,59 +66,11 @@
   <property name="joint_finger_2_lower_limit" value="0" />
   <property name="joint_finger_2_upper_limit" value="${J_PI/180*40}" />
-<xacro:macro name="mico_link" params="link_name">
-<link name="${link_name}">
-      <visual>
-                 <geometry>
-                         <mesh
-          filename="package://jaco_model/meshes/${link_name}.dae"/>
-                </geometry>
-                <material name="carbon_fiber">
- 			<color rgba="0.792156862745098 0.819607843137255 0.933333333333333 1" />
-                </material>
-        </visual>
-        <collision>
-                <geometry>
-                         <mesh
-          filename="package://jaco_model/meshes/${link_name}.dae"/>
-                </geometry>
-        </collision>
-</link>
-</xacro:macro>
-<xacro:macro name="mico_joint" params="joint_name type parent child joint_axis_xyz joint_origin_xyz joint_origin_rpy">
-<joint name="${joint_name}" type="${type}">
-    <parent link="${parent}"/>
-    <child link="${child}"/>
-    <axis xyz="${joint_axis_xyz}"/>
-<origin xyz="${joint_origin_xyz}" rpy="${joint_origin_rpy}"/>
- </joint>
-</xacro:macro>
-<xacro:macro name="mico_finger_joint" params="joint_name type parent child joint_axis_xyz joint_origin_xyz joint_origin_rpy lower_limit upper_limit">
-<joint name="${joint_name}" type="${type}">
-    <parent link="${parent}"/>
-    <child link="${child}"/>
-    <axis xyz="${joint_axis_xyz}"/>
-<origin xyz="${joint_origin_xyz}" rpy="${joint_origin_rpy}"/>
-    <limit lower="${lower_limit}" upper="${upper_limit}" effort="30" velocity="5"/>
- </joint>
-</xacro:macro>
-<xacro:macro name="mico_arm" params="parent">
-   <xacro:mico_link link_name="${link_base}"/>
-   <xacro:mico_joint joint_name="${joint_base}" type="fixed" parent="${parent}" child="${link_base}" joint_axis_xyz="${joint_base_axis_xyz}" joint_origin_xyz="${joint_base_origin_xyz}" joint_origin_rpy="${joint_base_origin_rpy}"/>
-   <xacro:mico_link link_name="${link_1}"/>
-   <xacro:mico_joint joint_name="${joint_1}" type="continuous" parent="${link_base}" child="${link_1}" joint_axis_xyz="${joint_1_axis_xyz}" joint_origin_xyz="${joint_1_origin_xyz}" joint_origin_rpy="${joint_1_origin_rpy}"/>
-   <xacro:mico_link link_name="${link_2}"/>
-   <xacro:mico_joint joint_name="${joint_2}" type="continuous" parent="${link_1}" child="${link_2}" joint_axis_xyz="${joint_2_axis_xyz}" joint_origin_xyz="${joint_2_origin_xyz}" joint_origin_rpy="${joint_2_origin_rpy}"/>
-   <xacro:mico_link link_name="${link_3}"/>
-   <xacro:mico_joint joint_name="${joint_3}" type="continuous" parent="${link_2}" child="${link_3}" joint_axis_xyz="${joint_3_axis_xyz}" joint_origin_xyz="${joint_3_origin_xyz}" joint_origin_rpy="${joint_3_origin_rpy}"/>
-   <xacro:mico_link link_name="${link_4}"/>
-   <xacro:mico_joint joint_name="${joint_4}" type="continuous" parent="${link_3}" child="${link_4}" joint_axis_xyz="${joint_4_axis_xyz}" joint_origin_xyz="${joint_4_origin_xyz}" joint_origin_rpy="${joint_4_origin_rpy}"/>
-   <xacro:mico_link link_name="${link_5}"/>
-   <xacro:mico_joint joint_name="${joint_5}" type="continuous" parent="${link_4}" child="${link_5}" joint_axis_xyz="${joint_5_axis_xyz}" joint_origin_xyz="${joint_5_origin_xyz}" joint_origin_rpy="${joint_5_origin_rpy}"/>
-   <xacro:mico_link link_name="${link_hand}"/>
-   <xacro:mico_joint joint_name="${joint_6}" type="continuous" parent="${link_5}" child="${link_hand}" joint_axis_xyz="${joint_6_axis_xyz}" joint_origin_xyz="${joint_6_origin_xyz}" joint_origin_rpy="${joint_6_origin_rpy}"/>
-   <xacro:mico_link link_name="${link_finger_1}"/>
-   <xacro:mico_finger_joint joint_name="${joint_finger_1}" type="revolute" parent="${link_hand}" child="${link_finger_1}" joint_axis_xyz="${joint_finger_1_axis_xyz}" joint_origin_xyz="${joint_finger_1_origin_xyz}" joint_origin_rpy="${joint_finger_1_origin_rpy}" lower_limit="${joint_finger_1_lower_limit}" upper_limit="${joint_finger_1_upper_limit}"/>
-   <xacro:mico_link link_name="${link_finger_2}"/>
-   <xacro:mico_finger_joint joint_name="${joint_finger_2}" type="revolute" parent="${link_hand}" child="${link_finger_2}" joint_axis_xyz="${joint_finger_2_axis_xyz}" joint_origin_xyz="${joint_finger_2_origin_xyz}" joint_origin_rpy="${joint_finger_2_origin_rpy}" lower_limit="${joint_finger_2_lower_limit}" upper_limit="${joint_finger_2_upper_limit}"/>
-</xacro:macro>
+  <xacro:include filename="$(find jaco_model)/urdf/jaco_common.xacro" />
+  <xacro:macro name="mico_arm" params="parent">
+    <xacro:jaco_struct parent="${parent}" basename="mico"/>
+    <xacro:jaco_link link_name="${link_finger_1}"/>
+    <xacro:jaco_finger_joint joint_name="${joint_finger_1}" type="revolute" parent="${link_hand}" child="${link_finger_1}" joint_axis_xyz="${joint_finger_1_axis_xyz}" joint_origin_xyz="${joint_finger_1_origin_xyz}" joint_origin_rpy="${joint_finger_1_origin_rpy}" lower_limit="${joint_finger_1_lower_limit}" upper_limit="${joint_finger_1_upper_limit}"/>
+    <xacro:jaco_link link_name="${link_finger_2}"/>
+    <xacro:jaco_finger_joint joint_name="${joint_finger_2}" type="revolute" parent="${link_hand}" child="${link_finger_2}" joint_axis_xyz="${joint_finger_2_axis_xyz}" joint_origin_xyz="${joint_finger_2_origin_xyz}" joint_origin_rpy="${joint_finger_2_origin_rpy}" lower_limit="${joint_finger_2_lower_limit}" upper_limit="${joint_finger_2_upper_limit}"/>
+  </xacro:macro>
 </root>

Commit message: Publication of the end effector forces as a wrench. Still need to rotate in the proper frame, figure out torque format.

File: jaco_model/urdf/jaco_arm.xacro (robot description, xacro)
@@ -13,5 +13,5 @@
     xmlns:physics="http://playerstage.sourceforge.net/gazebo/xmlschema/#physics"
 	xmlns:xacro="http://ros.org/wiki/xacro">
-  <property name="J_PI" value="3.1415926535897931" />
+  <xacro:include filename="$(find jaco_model)/urdf/jaco_common.xacro" />
   <property name="link_base" value="jaco_link_base" />
   <property name="link_1" value="jaco_link_1" />
@@ -72,5 +72,6 @@
   <property name="joint_finger_3_lower_limit" value="0" />
   <property name="joint_finger_3_upper_limit" value="${J_PI/180*40}" />
-  <xacro:include filename="$(find jaco_model)/urdf/jaco_common.xacro" />
+  <property name="link_end_effector"   value="jaco_end_effector" />
+  <property name="end_effector_offset" value="0.1687" />
   <xacro:macro name="jaco_arm" params="parent">
     <xacro:jaco_struct parent="${parent}" basename="jaco"/>

File: jaco_model/urdf/jaco_common.xacro (robot description, xacro)
@@ -13,4 +13,5 @@
     xmlns:physics="http://playerstage.sourceforge.net/gazebo/xmlschema/#physics"
 	xmlns:xacro="http://ros.org/wiki/xacro">
+    <property name="J_PI" value="3.1415926535897931" />
     <xacro:macro name="jaco_link" params="link_name">
     <link name="${link_name}">
@@ -83,4 +84,10 @@
          -->
         </link>
+        <joint name="${link_hand}_to_end_effector" type="fixed">
+          <parent link="${link_hand}"/>
+          <child link="${link_end_effector}"/>
+          <origin xyz="0 0 -${end_effector_offset}" rpy="0 ${J_PI} 0" />
+        </joint>
+        <link name="${link_end_effector}" />
     </xacro:macro>
 </root>

File: jaco_model/urdf/mico_arm.xacro (robot description, xacro)
@@ -13,5 +13,5 @@
     xmlns:physics="http://playerstage.sourceforge.net/gazebo/xmlschema/#physics"
 	xmlns:xacro="http://ros.org/wiki/xacro">
-  <property name="J_PI" value="3.1415926535897931" />
+  <xacro:include filename="$(find jaco_model)/urdf/jaco_common.xacro" />
   <property name="link_base" value="mico_link_base" />
   <property name="link_1" value="mico_link_1" />
@@ -66,5 +66,6 @@
   <property name="joint_finger_2_lower_limit" value="0" />
   <property name="joint_finger_2_upper_limit" value="${J_PI/180*40}" />
-  <xacro:include filename="$(find jaco_model)/urdf/jaco_common.xacro" />
+  <property name="link_end_effector"   value="mico_end_effector" />
+  <property name="end_effector_offset" value="0.160" />
   <xacro:macro name="mico_arm" params="parent">
     <xacro:jaco_struct parent="${parent}" basename="mico"/>
