Commit message: Proper limits for jaco joints.

File: jaco_model/urdf/jaco_arm.xacro (robot description, xacro)
@@ -34,24 +34,36 @@
   <property name="joint_1_origin_xyz" value="0 0 0.1535" />
   <property name="joint_1_origin_rpy" value="${J_PI} 0 ${J_PI}" />
+  <property name="joint_1_lower_limit" value="${-2*J_PI}" />
+  <property name="joint_1_upper_limit" value="${2*J_PI}" />
   <property name="joint_2" value="jaco_joint_2" />
   <property name="joint_2_axis_xyz" value="0 0 1" />
   <property name="joint_2_origin_xyz" value="0 0 -0.1185" />
   <property name="joint_2_origin_rpy" value="-${J_PI/2} ${J_PI} 0" />
+  <property name="joint_2_lower_limit" value="${-J_PI}" />
+  <property name="joint_2_upper_limit" value="${0}" />
   <property name="joint_3" value="jaco_joint_3" />
   <property name="joint_3_axis_xyz" value="0 0 -1" />
   <property name="joint_3_origin_xyz" value="0.41 0 0" />
   <property name="joint_3_origin_rpy" value="${J_PI} 0 ${J_PI/2}" />
+  <property name="joint_3_lower_limit" value="${-5*J_PI/4}" />
+  <property name="joint_3_upper_limit" value="${1*J_PI/4}" />
   <property name="joint_4" value="jaco_joint_4" />
   <property name="joint_4_axis_xyz" value="0 0 -1" />
   <property name="joint_4_origin_xyz" value="0.207 0 -0.01125" />
   <property name="joint_4_origin_rpy" value="${J_PI} ${J_PI/2} 0" />
+  <property name="joint_4_lower_limit" value="${-2*J_PI}" />
+  <property name="joint_4_upper_limit" value="${2*J_PI}" />
   <property name="joint_5" value="jaco_joint_5" />
   <property name="joint_5_axis_xyz" value="0 0 -1" />
   <property name="joint_5_origin_xyz" value="0.0343 0 -0.06588" />
   <property name="joint_5_origin_rpy" value="0 -${J_PI/180*55} 0" />
+  <property name="joint_5_lower_limit" value="${-2*J_PI}" />
+  <property name="joint_5_upper_limit" value="${2*J_PI}" />
   <property name="joint_6" value="jaco_joint_6" />
   <property name="joint_6_axis_xyz" value="0 0 -1" />
   <property name="joint_6_origin_xyz" value="0.0343 0 -0.06588" />
   <property name="joint_6_origin_rpy" value="-${J_PI/180*55} 0 ${J_PI/2}" />
+  <property name="joint_6_lower_limit" value="${-2*J_PI}" />
+  <property name="joint_6_upper_limit" value="${2*J_PI}" />
   <property name="joint_finger_1" value="jaco_joint_finger_1" />
   <property name="joint_finger_1_axis_xyz" value="0 0 1" />

File: jaco_model/urdf/jaco_common.xacro (robot description, xacro)
@@ -33,10 +33,10 @@
     </link>
     </xacro:macro>
-    <xacro:macro name="jaco_joint" params="joint_name type parent child joint_axis_xyz joint_origin_xyz joint_origin_rpy">
+    <xacro:macro name="jaco_joint" params="joint_name type parent child joint_axis_xyz joint_origin_xyz joint_origin_rpy joint_lower_limit joint_upper_limit">
     <joint name="${joint_name}" type="${type}">
         <parent link="${parent}"/>
         <child link="${child}"/>
         <axis xyz="${joint_axis_xyz}"/>
-        <limit effort="30" velocity="0.35"/>
+        <limit effort="30" velocity="0.35" lower="${joint_lower_limit}" upper="${joint_upper_limit}"/>
         <origin xyz="${joint_origin_xyz}" rpy="${joint_origin_rpy}"/>
      </joint>
@@ -53,17 +53,17 @@
     <xacro:macro name="jaco_struct" params="parent basename">
         <xacro:jaco_link link_name="${link_base}"/>
-        <xacro:jaco_joint joint_name="${joint_base}" type="fixed" parent="${parent}" child="${link_base}" joint_axis_xyz="${joint_base_axis_xyz}" joint_origin_xyz="${joint_base_origin_xyz}" joint_origin_rpy="${joint_base_origin_rpy}"/>
+        <xacro:jaco_joint joint_name="${joint_base}" type="fixed" parent="${parent}" child="${link_base}" joint_axis_xyz="${joint_base_axis_xyz}" joint_origin_xyz="${joint_base_origin_xyz}" joint_origin_rpy="${joint_base_origin_rpy}" joint_lower_limit="0" joint_upper_limit="0"/>
         <xacro:jaco_link link_name="${link_1}"/>
-        <xacro:jaco_joint joint_name="${joint_1}" type="continuous" parent="${link_base}" child="${link_1}" joint_axis_xyz="${joint_1_axis_xyz}" joint_origin_xyz="${joint_1_origin_xyz}" joint_origin_rpy="${joint_1_origin_rpy}"/>
+        <xacro:jaco_joint joint_name="${joint_1}" type="continuous" parent="${link_base}" child="${link_1}" joint_axis_xyz="${joint_1_axis_xyz}" joint_origin_xyz="${joint_1_origin_xyz}" joint_origin_rpy="${joint_1_origin_rpy}" joint_lower_limit="${joint_1_lower_limit}" joint_upper_limit="${joint_1_upper_limit}"/>
         <xacro:jaco_link link_name="${link_2}"/>
-        <xacro:jaco_joint joint_name="${joint_2}" type="continuous" parent="${link_1}" child="${link_2}" joint_axis_xyz="${joint_2_axis_xyz}" joint_origin_xyz="${joint_2_origin_xyz}" joint_origin_rpy="${joint_2_origin_rpy}"/>
+        <xacro:jaco_joint joint_name="${joint_2}" type="revolute" parent="${link_1}" child="${link_2}" joint_axis_xyz="${joint_2_axis_xyz}" joint_origin_xyz="${joint_2_origin_xyz}" joint_origin_rpy="${joint_2_origin_rpy}" joint_lower_limit="${joint_2_lower_limit}" joint_upper_limit="${joint_2_upper_limit}"/>
         <xacro:jaco_link link_name="${link_3}"/>
-        <xacro:jaco_joint joint_name="${joint_3}" type="continuous" parent="${link_2}" child="${link_3}" joint_axis_xyz="${joint_3_axis_xyz}" joint_origin_xyz="${joint_3_origin_xyz}" joint_origin_rpy="${joint_3_origin_rpy}"/>
+        <xacro:jaco_joint joint_name="${joint_3}" type="revolute" parent="${link_2}" child="${link_3}" joint_axis_xyz="${joint_3_axis_xyz}" joint_origin_xyz="${joint_3_origin_xyz}" joint_origin_rpy="${joint_3_origin_rpy}" joint_lower_limit="${joint_3_lower_limit}" joint_upper_limit="${joint_3_upper_limit}"/>
         <xacro:jaco_link link_name="${link_4}"/>
-        <xacro:jaco_joint joint_name="${joint_4}" type="continuous" parent="${link_3}" child="${link_4}" joint_axis_xyz="${joint_4_axis_xyz}" joint_origin_xyz="${joint_4_origin_xyz}" joint_origin_rpy="${joint_4_origin_rpy}"/>
+        <xacro:jaco_joint joint_name="${joint_4}" type="continuous" parent="${link_3}" child="${link_4}" joint_axis_xyz="${joint_4_axis_xyz}" joint_origin_xyz="${joint_4_origin_xyz}" joint_origin_rpy="${joint_4_origin_rpy}" joint_lower_limit="${joint_4_lower_limit}" joint_upper_limit="${joint_4_upper_limit}"/>
         <xacro:jaco_link link_name="${link_5}"/>
-        <xacro:jaco_joint joint_name="${joint_5}" type="continuous" parent="${link_4}" child="${link_5}" joint_axis_xyz="${joint_5_axis_xyz}" joint_origin_xyz="${joint_5_origin_xyz}" joint_origin_rpy="${joint_5_origin_rpy}"/>
-        <xacro:jaco_link link_name="${link_hand}"/>
-        <xacro:jaco_joint joint_name="${joint_6}" type="continuous" parent="${link_5}" child="${link_hand}" joint_axis_xyz="${joint_6_axis_xyz}" joint_origin_xyz="${joint_6_origin_xyz}" joint_origin_rpy="${joint_6_origin_rpy}"/>
+        <xacro:jaco_joint joint_name="${joint_5}" type="continuous" parent="${link_4}" child="${link_5}" joint_axis_xyz="${joint_5_axis_xyz}" joint_origin_xyz="${joint_5_origin_xyz}" joint_origin_rpy="${joint_5_origin_rpy}" joint_lower_limit="${joint_5_lower_limit}" joint_upper_limit="${joint_5_upper_limit}"/>
+        <xacro:jaco_link link_name="${link_hand}" />
+        <xacro:jaco_joint joint_name="${joint_6}" type="continuous" parent="${link_5}" child="${link_hand}" joint_axis_xyz="${joint_6_axis_xyz}" joint_origin_xyz="${joint_6_origin_xyz}" joint_origin_rpy="${joint_6_origin_rpy}" joint_lower_limit="${joint_6_lower_limit}" joint_upper_limit="${joint_6_upper_limit}"/>
        <joint name="${link_base}_to_api_origin" type="fixed">
          <parent link="${link_base}"/>
