Commit message: Added missing velocity limits to jaco/mico joints in URDF.

File: jaco_model/urdf/jaco_common.xacro (robot description, xacro)
@@ -38,5 +38,6 @@
         <child link="${child}"/>
         <axis xyz="${joint_axis_xyz}"/>
-    <origin xyz="${joint_origin_xyz}" rpy="${joint_origin_rpy}"/>
+        <limits effort="30" velocity="0.35"/>
+        <origin xyz="${joint_origin_xyz}" rpy="${joint_origin_rpy}"/>
      </joint>
     </xacro:macro>
@@ -46,5 +47,5 @@
         <child link="${child}"/>
         <axis xyz="${joint_axis_xyz}"/>
-    <origin xyz="${joint_origin_xyz}" rpy="${joint_origin_rpy}"/>
+        <origin xyz="${joint_origin_xyz}" rpy="${joint_origin_rpy}"/>
         <limit lower="${lower_limit}" upper="${upper_limit}" effort="30" velocity="5"/>
      </joint>

Commit message: Fix a typo in 'limits' element of URDF joints.

File: jaco_model/urdf/jaco_common.xacro (robot description, xacro)
@@ -38,5 +38,5 @@
         <child link="${child}"/>
         <axis xyz="${joint_axis_xyz}"/>
-        <limits effort="30" velocity="0.35"/>
+        <limit effort="30" velocity="0.35"/>
         <origin xyz="${joint_origin_xyz}" rpy="${joint_origin_rpy}"/>
      </joint>

Commit message: Initial support for the finger limbs of the Mico robot. This includes:
+ Collada meshes of the finger limbs, exported from the STEP file.
+ Addition of the macro jaco_finger_tip_joint in the jaco_common.xacro
+ Updated micro_arm.xacro that includes proximal and distal finger limbs
+ The distal finger limb (smaller one) is modeled as a mimic of the proximal finger limb
+ The angular range of the fingers is updated and matches the actual robot
+ Launcher that starts mico robot description and visualization in rviz

File: jaco_model/urdf/jaco_common.xacro (robot description, xacro)
@@ -51,4 +51,14 @@
      </joint>
     </xacro:macro>
+   <xacro:macro name="jaco_finger_tip_joint" params="joint_name type parent child joint_axis_xyz joint_origin_xyz joint_origin_rpy lower_limit upper_limit mimic_joint mimic_multiplier mimic_offset">
+    <joint name="${joint_name}" type="${type}">
+        <parent link="${parent}"/>
+        <child link="${child}"/>
+        <axis xyz="${joint_axis_xyz}"/>
+        <origin xyz="${joint_origin_xyz}" rpy="${joint_origin_rpy}"/>
+        <limit lower="${lower_limit}" upper="${upper_limit}" effort="30" velocity="5"/>
+        <mimic joint="${mimic_joint}" multiplier="${mimic_multiplier}" offset="${mimic_offset}"/>
+     </joint>
+    </xacro:macro>
     <xacro:macro name="jaco_struct" params="parent basename">
         <xacro:jaco_link link_name="${link_base}"/>

File: jaco_model/urdf/mico_arm.xacro (robot description, xacro)
@@ -21,7 +21,9 @@
   <property name="link_5" value="mico_link_5" />
   <property name="link_hand" value="mico_link_hand" />
-  <property name="link_finger_1" value="mico_link_finger_1" />
-  <property name="link_finger_2" value="mico_link_finger_2" />
+  <property name="link_finger_1" value="finger_proximal_limb_1" /> <!-- proximal limb finger 1-->
+  <property name="link_finger_2" value="finger_proximal_limb_2" /> <!-- proximal limb finger 2-->
   <property name="link_finger_3" value="mico_link_finger_3" />
+  <property name="link_finger_tip_1" value="finger_distal_limb_1" /> <!-- distal limb finger 1 -->
+  <property name="link_finger_tip_2" value="finger_distal_limb_2" /> <!-- distal limb finger 2 -->
   <property name="api_offset" value="0.028" />
   <property name="api_origin" value="mico_api_origin" />
@@ -68,14 +70,32 @@
   <property name="joint_finger_1" value="mico_joint_finger_1" />
   <property name="joint_finger_1_axis_xyz" value="0 0 1" />
-  <property name="joint_finger_1_origin_xyz" value="-0.03978 0 -0.10071" />
-  <property name="joint_finger_1_origin_rpy" value="${-J_PI/2} 1.117 ${J_PI}" />
+  <property name="joint_finger_1_origin_xyz" value="-0.03095 -0.0025 -0.116" />
+  <property name="joint_finger_1_origin_rpy" value="${J_PI/2} ${J_PI/2} 0" />
   <property name="joint_finger_1_lower_limit" value="0" />
-  <property name="joint_finger_1_upper_limit" value="${J_PI/180*40}" />
+  <property name="joint_finger_1_upper_limit" value="${J_PI/180*60}" />
+  <property name="joint_finger_tip_1" value="mico_joint_finger_tip_1" />
+  <property name="joint_finger_tip_1_axis_xyz" value="0 0 1" />
+  <property name="joint_finger_tip_1_origin_xyz" value="0.035 -0.02595 -0.0025" />
+  <property name="joint_finger_tip_1_origin_rpy" value="0 0 0" />
+  <property name="joint_finger_tip_1_lower_limit" value="0" />
+  <property name="joint_finger_tip_1_upper_limit" value="${J_PI/180*40}" />
+  <property name="joint_finger_tip_1_mimic_joint" value="${J_PI/180*40}" />
+  <property name="joint_finger_tip_1_mimic_multiplier" value="0.0" />
+  <property name="joint_finger_tip_1_mimc_offset" value="0.0" />
   <property name="joint_finger_2" value="mico_joint_finger_2" />
   <property name="joint_finger_2_axis_xyz" value="0 0 1" />
-  <property name="joint_finger_2_origin_xyz" value="0.03569 0 -0.10071" />
-  <property name="joint_finger_2_origin_rpy" value="${J_PI/2} ${J_PI - 1.117} ${J_PI}" />
+  <property name="joint_finger_2_origin_xyz" value="0.03095 -0.0025 -0.116" />
+  <property name="joint_finger_2_origin_rpy" value="${-J_PI/2} ${J_PI/2} 0" />
   <property name="joint_finger_2_lower_limit" value="0" />
-  <property name="joint_finger_2_upper_limit" value="${J_PI/180*40}" />
+  <property name="joint_finger_2_upper_limit" value="${J_PI/180*60}" />
+  <property name="joint_finger_tip_2" value="mico_joint_finger_tip_2" />
+  <property name="joint_finger_tip_2_axis_xyz" value="0 0 1" />
+  <property name="joint_finger_tip_2_origin_xyz" value="0.035 -0.02595 -0.0025" />
+  <property name="joint_finger_tip_2_origin_rpy" value="0 0 0" />
+  <property name="joint_finger_tip_2_lower_limit" value="0" />
+  <property name="joint_finger_tip_2_upper_limit" value="${J_PI/180*40}" />
+  <property name="joint_finger_tip_2_mimic_joint" value="${J_PI/180*40}" />
+  <property name="joint_finger_tip_2_mimic_multiplier" value="0.0" />
+  <property name="joint_finger_tip_2_mimc_offset" value="0.0" />
   <property name="link_end_effector"   value="mico_end_effector" />
   <property name="end_effector_offset" value="0.160" />
@@ -84,6 +104,10 @@
     <xacro:jaco_link link_name="${link_finger_1}"/>
     <xacro:jaco_finger_joint joint_name="${joint_finger_1}" type="revolute" parent="${link_hand}" child="${link_finger_1}" joint_axis_xyz="${joint_finger_1_axis_xyz}" joint_origin_xyz="${joint_finger_1_origin_xyz}" joint_origin_rpy="${joint_finger_1_origin_rpy}" lower_limit="${joint_finger_1_lower_limit}" upper_limit="${joint_finger_1_upper_limit}"/>
+    <xacro:jaco_link link_name="${link_finger_tip_1}"/>
+    <xacro:jaco_finger_tip_joint joint_name="${joint_finger_tip_1}" type="revolute" parent="${link_finger_1}" child="${link_finger_tip_1}" joint_axis_xyz="${joint_finger_tip_1_axis_xyz}" joint_origin_xyz="${joint_finger_tip_1_origin_xyz}" joint_origin_rpy="${joint_finger_tip_1_origin_rpy}" lower_limit="${joint_finger_tip_1_lower_limit}" upper_limit="${joint_finger_tip_1_upper_limit}" mimic_joint="${joint_finger_1}" mimic_multiplier="${joint_finger_tip_1_mimic_multiplier}" mimic_offset="${joint_finger_tip_1_mimc_offset}"/>
     <xacro:jaco_link link_name="${link_finger_2}"/>
     <xacro:jaco_finger_joint joint_name="${joint_finger_2}" type="revolute" parent="${link_hand}" child="${link_finger_2}" joint_axis_xyz="${joint_finger_2_axis_xyz}" joint_origin_xyz="${joint_finger_2_origin_xyz}" joint_origin_rpy="${joint_finger_2_origin_rpy}" lower_limit="${joint_finger_2_lower_limit}" upper_limit="${joint_finger_2_upper_limit}"/>
+    <xacro:jaco_link link_name="${link_finger_tip_2}"/>
+    <xacro:jaco_finger_tip_joint joint_name="${joint_finger_tip_2}" type="revolute" parent="${link_finger_2}" child="${link_finger_tip_2}" joint_axis_xyz="${joint_finger_tip_2_axis_xyz}" joint_origin_xyz="${joint_finger_tip_2_origin_xyz}" joint_origin_rpy="${joint_finger_tip_2_origin_rpy}" lower_limit="${joint_finger_tip_2_lower_limit}" upper_limit="${joint_finger_tip_2_upper_limit}" mimic_joint="${joint_finger_2}" mimic_multiplier="${joint_finger_tip_2_mimic_multiplier}" mimic_offset="${joint_finger_tip_2_mimc_offset}"/>
   </xacro:macro>
 </root>

Commit message: * Added support for gazebo * Added FollowJointTrajectory action for integration with moveit * Tested gazebo-moveIt motion planning

File: jaco_model/urdf/jaco_common.xacro (robot description, xacro)
@@ -16,4 +16,9 @@
     <xacro:macro name="jaco_link" params="link_name">
     <link name="${link_name}">
+	S<inertial>
+                <mass value="0.25"/>
+                <inertia ixx="0.01" ixy="0" ixz="0" iyy="0.01" iyz="0" izz="0.01"/>
+                <origin/>
+            </inertial>
           <visual>
                      <geometry>

File: jaco_model/urdf/mico_arm.xacro (robot description, xacro)
@@ -14,4 +14,5 @@
 	xmlns:xacro="http://ros.org/wiki/xacro">
   <xacro:include filename="$(find jaco_model)/urdf/jaco_common.xacro" />
+  <xacro:include filename="$(find jaco_model)/urdf/jaco_transmission_friction.xacro" />
   <property name="link_base" value="mico_link_base" />
   <property name="link_1" value="mico_link_1" />
@@ -100,5 +101,36 @@
   <property name="link_end_effector"   value="mico_end_effector" />
   <property name="end_effector_offset" value="0.160" />
+  <xacro:property name="mu1_default" value="0.2" />
+  <xacro:property name="mu2_default" value="0.2" />
+  <xacro:property name="kp_default" value="1000.0" />
+  <xacro:property name="kd_default" value="1.0" />
   <xacro:macro name="mico_arm" params="parent">
+	<gazebo>
+	    <plugin name="gazebo_ros_controller_manager" filename="libgazebo_ros_control.so">
+		<robotNamespace>/mico_arm</robotNamespace>
+		<robotParam>robot_description</robotParam>
+	    </plugin>
+	</gazebo>
+	<gazebo>
+	    <plugin name="gazebo_ros_joint_trajectory" filename="libgazebo_ros_joint_pose_trajectory.so">
+		<robotNamespace>/mico_arm</robotNamespace>
+		<alwaysOn>true</alwaysOn>
+		<updateRate>100.0</updateRate>
+	    </plugin>
+	</gazebo>
+	<gazebo>
+		<plugin name="mimic_plugin" filename="libgazebo_mimic_plugin.so">
+			<joint>${joint_finger_1}</joint>
+			<mimicJoint>${joint_finger_tip_1}</mimicJoint>
+			<multiplier>${joint_finger_tip_1_mimic_multiplier}</multiplier>
+		</plugin>
+	</gazebo>
+	<gazebo>
+		<plugin name="mimic_plugin" filename="libgazebo_mimic_plugin.so">
+			<joint>${joint_finger_2}</joint>
+			<mimicJoint>${joint_finger_tip_2}</mimicJoint>
+			<multiplier>${joint_finger_tip_2_mimic_multiplier}</multiplier>
+		</plugin>
+	</gazebo>
     <xacro:jaco_struct parent="${parent}" basename="mico"/>
     <xacro:jaco_link link_name="${link_finger_1}"/>
@@ -110,4 +142,5 @@
     <xacro:jaco_link link_name="${link_finger_tip_2}"/>
     <xacro:jaco_finger_tip_joint joint_name="${joint_finger_tip_2}" type="revolute" parent="${link_finger_2}" child="${link_finger_tip_2}" joint_axis_xyz="${joint_finger_tip_2_axis_xyz}" joint_origin_xyz="${joint_finger_tip_2_origin_xyz}" joint_origin_rpy="${joint_finger_tip_2_origin_rpy}" lower_limit="${joint_finger_tip_2_lower_limit}" upper_limit="${joint_finger_tip_2_upper_limit}" mimic_joint="${joint_finger_2}" mimic_multiplier="${joint_finger_tip_2_mimic_multiplier}" mimic_offset="${joint_finger_tip_2_mimc_offset}"/>
+  <xacro:jaco_transmission_friction_gazebo/>
   </xacro:macro>
 </root>

Commit message: * Joint trajectory controllers from the gazebo ros interface disabled in the launcher * Set masses and inertias to default values that gurantee stability of the ros controllers * Configuration tested on moveIt for both jaco and mico models

File: jaco_model/urdf/jaco_common.xacro (robot description, xacro)
@@ -17,6 +17,6 @@
     <link name="${link_name}">
 	<inertial>
-                <mass value="0.25"/>
-                <inertia ixx="0.01" ixy="0" ixz="0" iyy="0.01" iyz="0" izz="0.01"/>
+                <mass value="0.01"/>
+                <inertia ixx="0.001" ixy="0" ixz="0" iyy="0.001" iyz="0" izz="0.001"/>
                 <origin/>
             </inertial>
@@ -50,4 +50,5 @@
         <limit effort="30" velocity="0.35" lower="${joint_lower_limit}" upper="${joint_upper_limit}"/>
         <origin xyz="${joint_origin_xyz}" rpy="${joint_origin_rpy}"/>
+        <dynamics damping="0.0"/>
      </joint>
     </xacro:macro>
@@ -58,5 +59,6 @@
         <axis xyz="${joint_axis_xyz}"/>
         <origin xyz="${joint_origin_xyz}" rpy="${joint_origin_rpy}"/>
-        <limit lower="${lower_limit}" upper="${upper_limit}" effort="30" velocity="5"/>
+        <limit lower="${lower_limit}" upper="${upper_limit}" effort="30" velocity="0.3"/>
+        <dynamics damping="0.0"/>
      </joint>
     </xacro:macro>

File: jaco_model/urdf/jaco_transmission_friction.xacro (robot description, xacro)
@@ -35,7 +35,7 @@
 		<kd value="${kd}" />
 		<kp value="${kp}" />
-		<stopCfm value="${kp}" />
+		<!--<stopCfm value="${kp}" />
 		<stopErp value="${kd}" />
-		<fudgeFactor value="1.0" />
+		<fudgeFactor value="1.0" />-->
 	</gazebo>
 </xacro:macro>

File: jaco_model/urdf/mico_arm.xacro (robot description, xacro)
@@ -101,4 +101,8 @@
   <property name="link_end_effector"   value="mico_end_effector" />
   <property name="end_effector_offset" value="0.160" />
+  <!--<xacro:property name="mu1_default" value="0.0" />
+  <xacro:property name="mu2_default" value="0.0" />
+  <xacro:property name="kp_default" value="0.0" />
+  <xacro:property name="kd_default" value="0.0" />-->
   <xacro:property name="mu1_default" value="0.2" />
   <xacro:property name="mu2_default" value="0.2" />
@@ -123,5 +127,6 @@
 		<robotNamespace>/mico_arm</robotNamespace>
 		<alwaysOn>true</alwaysOn>
-		<updateRate>100.0</updateRate>
+		<updateRate>1000.0</updateRate>
+		<disablePhysicsUpdates>true</disablePhysicsUpdates>
 	    </plugin>
 	</gazebo>
