Commit message: added sensors file for the kinect example

File: jaco_model/urdf/mico_on_table_gazebo.xacro (robot description, xacro)
@@ -33,5 +33,5 @@
 	    <parent link="world"/>
 	    <child link="root"/>
-	    <origin xyz="0.0 -0.95 1.01" rpy="0.0 0.0 0.0" />
+	    <origin xyz="0.0 -0.95 1.03" rpy="0.0 0.0 0.0" />
 	</joint>
 <xacro:mico_arm  parent="root"/>
