Commit message: Renaming jaco_model to kinova_description.

File: kinova_description/urdf/jaco_arm.xacro (robot description, xacro)
@@ -13,5 +13,5 @@
     xmlns:physics="http://playerstage.sourceforge.net/gazebo/xmlschema/#physics"
 	xmlns:xacro="http://ros.org/wiki/xacro">
-  <xacro:include filename="$(find jaco_model)/urdf/jaco_common.xacro" />
+  <xacro:include filename="$(find kinova_description)/urdf/jaco_common.xacro" />
   <property name="link_base" value="jaco_link_base" />
   <property name="link_1" value="jaco_link_1" />

File: kinova_description/urdf/jaco_common.xacro (robot description, xacro)
@@ -15,21 +15,21 @@
     <property name="J_PI" value="3.1415926535897931" />
     <xacro:macro name="jaco_link" params="link_name">
-    <link name="${link_name}">
-          <visual>
-                     <geometry>
-                             <mesh
-              filename="package://jaco_model/meshes/${link_name}.dae"/>
-                    </geometry>
-                    <material name="carbon_fiber">
-                <color rgba="0.792156862745098 0.819607843137255 0.933333333333333 1" />
-                    </material>
+        <link name="${link_name}">
+            <visual>
+                <geometry>
+                    <mesh
+                        filename="package://kinova_description/meshes/${link_name}.dae"/>
+                </geometry>
+                <material name="carbon_fiber">
+                    <color rgba="0.792156862745098 0.819607843137255 0.933333333333333 1" />
+                </material>
             </visual>
             <collision>
-                    <geometry>
-                             <mesh
-              filename="package://jaco_model/meshes/${link_name}.dae"/>
-                    </geometry>
+                <geometry>
+                    <mesh
+                        filename="package://kinova_description/meshes/${link_name}.dae"/>
+                </geometry>
             </collision>
-    </link>
+        </link>
     </xacro:macro>
     <xacro:macro name="jaco_joint" params="joint_name type parent child joint_axis_xyz joint_origin_xyz joint_origin_rpy joint_lower_limit joint_upper_limit">

File: kinova_description/urdf/mico_arm.xacro (robot description, xacro)
@@ -13,5 +13,5 @@
     xmlns:physics="http://playerstage.sourceforge.net/gazebo/xmlschema/#physics"
 	xmlns:xacro="http://ros.org/wiki/xacro">
-  <xacro:include filename="$(find jaco_model)/urdf/jaco_common.xacro" />
+  <xacro:include filename="$(find kinova_description)/urdf/jaco_common.xacro" />
   <property name="link_base" value="mico_link_base" />
   <property name="link_1" value="mico_link_1" />

File: kinova_description/urdf/standalone_jaco.xacro (robot description, xacro)
@@ -12,6 +12,6 @@
     xmlns:renderable="http://playerstage.sourceforge.net/gazebo/xmlschema/#renderable"
     xmlns:physics="http://playerstage.sourceforge.net/gazebo/xmlschema/#physics"
-	xmlns:xacro="http://ros.org/wiki/xacro" name="mico">
-  <xacro:include filename="$(find jaco_model)/urdf/mico_arm.xacro" />
+	xmlns:xacro="http://ros.org/wiki/xacro" name="jaco">
+  <xacro:include filename="$(find kinova_description)/urdf/jaco_arm.xacro" />
 <link name="root">
       <visual>
@@ -29,4 +29,4 @@
       </collision>
     </link>
-<xacro:mico_arm  parent="root"/>
+<xacro:jaco_arm  parent="root"/>
 </robot>

File: kinova_description/urdf/standalone_mico.xacro (robot description, xacro)
@@ -12,6 +12,6 @@
     xmlns:renderable="http://playerstage.sourceforge.net/gazebo/xmlschema/#renderable"
     xmlns:physics="http://playerstage.sourceforge.net/gazebo/xmlschema/#physics"
-	xmlns:xacro="http://ros.org/wiki/xacro" name="jaco">
-  <xacro:include filename="$(find jaco_model)/urdf/jaco_arm.xacro" />
+	xmlns:xacro="http://ros.org/wiki/xacro" name="mico">
+  <xacro:include filename="$(find kinova_description)/urdf/mico_arm.xacro" />
 <link name="root">
       <visual>
@@ -29,4 +29,4 @@
       </collision>
     </link>
-<xacro:jaco_arm  parent="root"/>
+<xacro:mico_arm  parent="root"/>
 </robot>

Commit message: Working Gazebo config with follow_joint_trajectory, missing fingers.

File: kinova_description/urdf/jaco_arm.xacro (robot description, xacro)
@@ -15,10 +15,66 @@
   <xacro:include filename="$(find kinova_description)/urdf/jaco_common.xacro" />
   <property name="link_base" value="jaco_link_base" />
+  <property name="link_base_cog"  value="0 0 0" />
+  <property name="link_base_mass" value="0.100" />
+  <property name="link_base_ixx"  value="0.100" />
+  <property name="link_base_ixy"  value="0.000" />
+  <property name="link_base_ixz"  value="0.000" />
+  <property name="link_base_iyy"  value="0.100" />
+  <property name="link_base_iyz"  value="0.000" />
+  <property name="link_base_izz"  value="0.100" />
   <property name="link_1" value="jaco_link_1" />
+  <property name="link_1_cog"  value="0.0692 0.0001 -0.0103" />
+  <property name="link_1_mass" value="0.748" />
+  <property name="link_1_ixx"  value="1.02e-2" />
+  <property name="link_1_ixy"  value="-5.21e-7" />
+  <property name="link_1_ixz"  value="-2.12e-3" />
+  <property name="link_1_iyy"  value="3.25e-2" />
+  <property name="link_1_iyz"  value="-4.14e-7" />
+  <property name="link_1_izz"  value="3.54e-2" />
   <property name="link_2" value="jaco_link_2" />
+  <property name="link_2_cog"  value="0.2052 0.0000 0.0223" />
+  <property name="link_2_mass" value="1.011" />
+  <property name="link_2_ixx"  value="3.79e-1" />
+  <property name="link_2_ixy"  value="0.000" />
+  <property name="link_2_ixz"  value="0.000" />
+  <property name="link_2_iyy"  value="3.73e-1" />
+  <property name="link_2_iyz"  value="-5.90e-6" />
+  <property name="link_2_izz"  value="6.98e-3" />
   <property name="link_3" value="jaco_link_3" />
+  <property name="link_3_cog"  value="0.0196 0.0000 0.0644" />
+  <property name="link_3_mass" value="0.568" />
+  <property name="link_3_ixx"  value="5.11e-2" />
+  <property name="link_3_ixy"  value="1.92e-7" />
+  <property name="link_3_ixz"  value="-2.67e-7" />
+  <property name="link_3_iyy"  value="1.44e-1" />
+  <property name="link_3_iyz"  value="-9.59e-5" />
+  <property name="link_3_izz"  value="1.29e-2" />
   <property name="link_4" value="jaco_link_4" />
+  <property name="link_4_cog"  value="0.0086 0.0000 -0.0374" />
+  <property name="link_4_mass" value="0.427" />
+  <property name="link_4_ixx"  value="2.46e-3" />
+  <property name="link_4_ixy"  value="8.33e-4" />
+  <property name="link_4_ixz"  value="3.35e-8" />
+  <property name="link_4_iyy"  value="3.42e-3" />
+  <property name="link_4_iyz"  value="3.40e-8" />
+  <property name="link_4_izz"  value="3.63e-3" />
   <property name="link_5" value="jaco_link_5" />
+  <property name="link_5_cog"  value="0.0086 0.0000 -0.0374" />
+  <property name="link_5_mass" value="0.427" />
+  <property name="link_5_ixx"  value="2.46e-3" />
+  <property name="link_5_ixy"  value="8.33e-4" />
+  <property name="link_5_ixz"  value="3.35e-8" />
+  <property name="link_5_iyy"  value="3.42e-3" />
+  <property name="link_5_iyz"  value="3.40e-8" />
+  <property name="link_5_izz"  value="3.63e-3" />
   <property name="link_hand" value="jaco_link_hand" />
+  <property name="link_hand_cog"  value="0.0068 0.0000 -0.0822" />
+  <property name="link_hand_mass" value="0.727" />
+  <property name="link_hand_ixx"  value="4.66e-3" />
+  <property name="link_hand_ixy"  value="4.13e-4" />
+  <property name="link_hand_ixz"  value="-1.05e-5" />
+  <property name="link_hand_iyy"  value="2.65e-3" />
+  <property name="link_hand_iyz"  value="-3.24e-6" />
+  <property name="link_hand_izz"  value="5.25e-3" />
   <property name="link_finger_1" value="jaco_link_finger_1" />
   <property name="link_finger_2" value="jaco_link_finger_2" />
@@ -88,9 +144,9 @@
   <xacro:macro name="jaco_arm" params="parent">
     <xacro:jaco_struct parent="${parent}" basename="jaco"/>
-    <xacro:jaco_link link_name="${link_finger_1}"/>
+    <xacro:jaco_finger_link link_name="${link_finger_1}"/>
     <xacro:jaco_finger_joint joint_name="${joint_finger_1}" type="revolute" parent="${link_hand}" child="${link_finger_1}" joint_axis_xyz="${joint_finger_1_axis_xyz}" joint_origin_xyz="${joint_finger_1_origin_xyz}" joint_origin_rpy="${joint_finger_1_origin_rpy}" lower_limit="${joint_finger_1_lower_limit}" upper_limit="${joint_finger_1_upper_limit}"/>
-    <xacro:jaco_link link_name="${link_finger_2}"/>
+    <xacro:jaco_finger_link link_name="${link_finger_2}"/>
     <xacro:jaco_finger_joint joint_name="${joint_finger_2}" type="revolute" parent="${link_hand}" child="${link_finger_2}" joint_axis_xyz="${joint_finger_2_axis_xyz}" joint_origin_xyz="${joint_finger_2_origin_xyz}" joint_origin_rpy="${joint_finger_2_origin_rpy}" lower_limit="${joint_finger_2_lower_limit}" upper_limit="${joint_finger_2_upper_limit}"/>
-    <xacro:jaco_link link_name="${link_finger_3}"/>
+    <xacro:jaco_finger_link link_name="${link_finger_3}"/>
     <xacro:jaco_finger_joint joint_name="${joint_finger_3}" type="revolute" parent="${link_hand}" child="${link_finger_3}" joint_axis_xyz="${joint_finger_3_axis_xyz}" joint_origin_xyz="${joint_finger_3_origin_xyz}" joint_origin_rpy="${joint_finger_3_origin_rpy}" lower_limit="${joint_finger_3_lower_limit}" upper_limit="${joint_finger_3_upper_limit}"/>
   </xacro:macro>

File: kinova_description/urdf/jaco_common.xacro (robot description, xacro)
@@ -14,16 +14,15 @@
 	xmlns:xacro="http://ros.org/wiki/xacro">
     <property name="J_PI" value="3.1415926535897931" />
-    <xacro:macro name="jaco_link" params="link_name">
+    <xacro:macro name="jaco_link" params="link_name link_mass link_cog link_ixx link_ixy link_ixz link_iyy link_iyz link_izz">
         <link name="${link_name}">
             <inertial>
-                <!-- TODO: Proper mass and inertia values! -->
-                <origin xyz="0 0 0" rpy="0 0 0"/>
-                <mass value="1"/>
-                <inertia ixx="0.1"
-                         ixy="0.0"
-                         ixz="0.0"
-                         iyy="0.1"
-                         iyz="0.0"
-                         izz="0.1"/>
+                <origin xyz="${link_cog}" rpy="0 0 0"/>
+                <mass value="${link_mass}"/>
+                <inertia ixx="${link_ixx}"
+                         ixy="${link_ixy}"
+                         ixz="${link_ixz}"
+                         iyy="${link_iyy}"
+                         iyz="${link_iyz}"
+                         izz="${link_izz}"/>
             </inertial>
             <visual>
@@ -62,4 +61,34 @@
     </transmission>
     </xacro:macro>
+    <xacro:macro name="jaco_finger_link" params="link_name">
+        <link name="${link_name}">
+            <!-- Inertia included in the hand link -->
+            <inertial>
+                <origin xyz="0 0 0" rpy="0 0 0"/>
+                <mass value="0.010"/>
+                <inertia ixx="0.010"
+                         ixy="0"
+                         ixz="0"
+                         iyy="0.010"
+                         iyz="0"
+                         izz="0.010"/>
+            </inertial>
+            <visual>
+                <geometry>
+                    <mesh
+                        filename="package://kinova_description/meshes/${link_name}.dae"/>
+                </geometry>
+                <material name="carbon_fiber">
+                    <color rgba="0.792156862745098 0.819607843137255 0.933333333333333 1" />
+                </material>
+            </visual>
+            <collision>
+                <geometry>
+                    <mesh
+                        filename="package://kinova_description/meshes/${link_name}.dae"/>
+                </geometry>
+            </collision>
+        </link>
+    </xacro:macro>
     <xacro:macro name="jaco_finger_joint" params="joint_name type parent child joint_axis_xyz joint_origin_xyz joint_origin_rpy lower_limit upper_limit">
     <joint name="${joint_name}" type="${type}">
@@ -70,7 +99,16 @@
         <limit lower="${lower_limit}" upper="${upper_limit}" effort="30" velocity="5"/>
      </joint>
+     <transmission name="${joint_name}_trans">
+        <type>transmission_interface/SimpleTransmission</type>
+        <joint name="${joint_name}">
+            <hardwareInterface>EffortJointInterface</hardwareInterface>
+        </joint>
+        <actuator name="${joint_name}_motor">
+            <mechanicalReduction>1.0</mechanicalReduction>
+        </actuator>
+    </transmission>
     </xacro:macro>
     <xacro:macro name="jaco_struct" params="parent basename">
-        <xacro:jaco_link link_name="${link_base}"/>
+        <xacro:jaco_link link_name="${link_base}" link_mass="${link_base_mass}" link_cog="${link_base_cog}" link_ixx="${link_base_ixx}" link_ixy="${link_base_ixy}" link_ixz="${link_base_ixz}" link_iyy="${link_base_iyy}" link_iyz="${link_base_iyz}" link_izz="${link_base_izz}"/>
         <!-- Separate joint definition for base to avoid creating a transmission
              on fixed joint.
@@ -82,15 +120,15 @@
             <origin xyz="${joint_base_origin_xyz}" rpy="${joint_base_origin_rpy}"/>
         </joint>
-        <xacro:jaco_link link_name="${link_1}"/>
+        <xacro:jaco_link link_name="${link_1}" link_mass="${link_1_mass}" link_cog="${link_1_cog}" link_ixx="${link_1_ixx}" link_ixy="${link_1_ixy}" link_ixz="${link_1_ixz}" link_iyy="${link_1_iyy}" link_iyz="${link_1_iyz}" link_izz="${link_1_izz}"/>
         <xacro:jaco_joint joint_name="${joint_1}" type="continuous" parent="${link_base}" child="${link_1}" joint_axis_xyz="${joint_1_axis_xyz}" joint_origin_xyz="${joint_1_origin_xyz}" joint_origin_rpy="${joint_1_origin_rpy}" joint_lower_limit="${joint_1_lower_limit}" joint_upper_limit="${joint_1_upper_limit}"/>
-        <xacro:jaco_link link_name="${link_2}"/>
+        <xacro:jaco_link link_name="${link_2}" link_mass="${link_2_mass}" link_cog="${link_2_cog}" link_ixx="${link_2_ixx}" link_ixy="${link_2_ixy}" link_ixz="${link_2_ixz}" link_iyy="${link_2_iyy}" link_iyz="${link_2_iyz}" link_izz="${link_2_izz}"/>
         <xacro:jaco_joint joint_name="${joint_2}" type="revolute" parent="${link_1}" child="${link_2}" joint_axis_xyz="${joint_2_axis_xyz}" joint_origin_xyz="${joint_2_origin_xyz}" joint_origin_rpy="${joint_2_origin_rpy}" joint_lower_limit="${joint_2_lower_limit}" joint_upper_limit="${joint_2_upper_limit}"/>
-        <xacro:jaco_link link_name="${link_3}"/>
+        <xacro:jaco_link link_name="${link_3}" link_mass="${link_3_mass}" link_cog="${link_3_cog}" link_ixx="${link_3_ixx}" link_ixy="${link_3_ixy}" link_ixz="${link_3_ixz}" link_iyy="${link_3_iyy}" link_iyz="${link_3_iyz}" link_izz="${link_3_izz}"/>
         <xacro:jaco_joint joint_name="${joint_3}" type="revolute" parent="${link_2}" child="${link_3}" joint_axis_xyz="${joint_3_axis_xyz}" joint_origin_xyz="${joint_3_origin_xyz}" joint_origin_rpy="${joint_3_origin_rpy}" joint_lower_limit="${joint_3_lower_limit}" joint_upper_limit="${joint_3_upper_limit}"/>
-        <xacro:jaco_link link_name="${link_4}"/>
+        <xacro:jaco_link link_name="${link_4}" link_mass="${link_4_mass}" link_cog="${link_4_cog}" link_ixx="${link_4_ixx}" link_ixy="${link_4_ixy}" link_ixz="${link_4_ixz}" link_iyy="${link_4_iyy}" link_iyz="${link_4_iyz}" link_izz="${link_4_izz}"/>
         <xacro:jaco_joint joint_name="${joint_4}" type="continuous" parent="${link_3}" child="${link_4}" joint_axis_xyz="${joint_4_axis_xyz}" joint_origin_xyz="${joint_4_origin_xyz}" joint_origin_rpy="${joint_4_origin_rpy}" joint_lower_limit="${joint_4_lower_limit}" joint_upper_limit="${joint_4_upper_limit}"/>
-        <xacro:jaco_link link_name="${link_5}"/>
+        <xacro:jaco_link link_name="${link_5}" link_mass="${link_5_mass}" link_cog="${link_5_cog}" link_ixx="${link_5_ixx}" link_ixy="${link_5_ixy}" link_ixz="${link_5_ixz}" link_iyy="${link_5_iyy}" link_iyz="${link_5_iyz}" link_izz="${link_5_izz}"/>
         <xacro:jaco_joint joint_name="${joint_5}" type="continuous" parent="${link_4}" child="${link_5}" joint_axis_xyz="${joint_5_axis_xyz}" joint_origin_xyz="${joint_5_origin_xyz}" joint_origin_rpy="${joint_5_origin_rpy}" joint_lower_limit="${joint_5_lower_limit}" joint_upper_limit="${joint_5_upper_limit}"/>
-        <xacro:jaco_link link_name="${link_hand}" />
+        <xacro:jaco_link link_name="${link_hand}" link_mass="${link_hand_mass}" link_cog="${link_hand_cog}" link_ixx="${link_hand_ixx}" link_ixy="${link_hand_ixy}" link_ixz="${link_hand_ixz}" link_iyy="${link_hand_iyy}" link_iyz="${link_hand_iyz}" link_izz="${link_hand_izz}" />
         <xacro:jaco_joint joint_name="${joint_6}" type="continuous" parent="${link_5}" child="${link_hand}" joint_axis_xyz="${joint_6_axis_xyz}" joint_origin_xyz="${joint_6_origin_xyz}" joint_origin_rpy="${joint_6_origin_rpy}" joint_lower_limit="${joint_6_lower_limit}" joint_upper_limit="${joint_6_upper_limit}"/>
        <joint name="${link_base}_to_api_origin" type="fixed">
