Commit message: Working launch files for Jaco2, Mico Gazebo config, plus fixes to URDF for Gazebo.

File: kinova_description/urdf/jaco2_arm.xacro (robot description, xacro)
@@ -110,5 +110,5 @@
   <property name="joint_4_lower_limit" value="${-2*J_PI}" />
   <property name="joint_4_upper_limit" value="${2*J_PI}" />
-  <property name="joint_5" value="jaco_joint_5" />
+  <property name="joint_5" value="jaco2_joint_5" />
   <property name="joint_5_axis_xyz" value="0 0 -1" />
   <property name="joint_5_origin_xyz" value="0.03700 0 -0.06408" />
@@ -116,5 +116,5 @@
   <property name="joint_5_lower_limit" value="${-2*J_PI}" />
   <property name="joint_5_upper_limit" value="${2*J_PI}" />
-  <property name="joint_6" value="jaco_joint_6" />
+  <property name="joint_6" value="jaco2_joint_6" />
   <property name="joint_6_axis_xyz" value="0 0 -1" />
   <property name="joint_6_origin_xyz" value="0.03700 0 -0.06408" />
@@ -144,9 +144,9 @@
   <xacro:macro name="jaco2_arm" params="parent">
     <xacro:jaco_struct parent="${parent}" basename="jaco2"/>
-    <xacro:jaco_link link_name="${link_finger_1}"/>
+    <xacro:jaco_finger_link link_name="${link_finger_1}"/>
     <xacro:jaco_finger_joint joint_name="${joint_finger_1}" type="revolute" parent="${link_hand}" child="${link_finger_1}" joint_axis_xyz="${joint_finger_1_axis_xyz}" joint_origin_xyz="${joint_finger_1_origin_xyz}" joint_origin_rpy="${joint_finger_1_origin_rpy}" lower_limit="${joint_finger_1_lower_limit}" upper_limit="${joint_finger_1_upper_limit}"/>
-    <xacro:jaco_link link_name="${link_finger_2}"/>
+    <xacro:jaco_finger_link link_name="${link_finger_2}"/>
     <xacro:jaco_finger_joint joint_name="${joint_finger_2}" type="revolute" parent="${link_hand}" child="${link_finger_2}" joint_axis_xyz="${joint_finger_2_axis_xyz}" joint_origin_xyz="${joint_finger_2_origin_xyz}" joint_origin_rpy="${joint_finger_2_origin_rpy}" lower_limit="${joint_finger_2_lower_limit}" upper_limit="${joint_finger_2_upper_limit}"/>
-    <xacro:jaco_link link_name="${link_finger_3}"/>
+    <xacro:jaco_finger_link link_name="${link_finger_3}"/>
     <xacro:jaco_finger_joint joint_name="${joint_finger_3}" type="revolute" parent="${link_hand}" child="${link_finger_3}" joint_axis_xyz="${joint_finger_3_axis_xyz}" joint_origin_xyz="${joint_finger_3_origin_xyz}" joint_origin_rpy="${joint_finger_3_origin_rpy}" lower_limit="${joint_finger_3_lower_limit}" upper_limit="${joint_finger_3_upper_limit}"/>
   </xacro:macro>

File: kinova_description/urdf/mico_arm.xacro (robot description, xacro)
@@ -138,7 +138,7 @@
   <xacro:macro name="mico_arm" params="parent">
     <xacro:jaco_struct parent="${parent}" basename="mico"/>
-    <xacro:jaco_link link_name="${link_finger_1}"/>
+    <xacro:jaco_finger_link link_name="${link_finger_1}"/>
     <xacro:jaco_finger_joint joint_name="${joint_finger_1}" type="revolute" parent="${link_hand}" child="${link_finger_1}" joint_axis_xyz="${joint_finger_1_axis_xyz}" joint_origin_xyz="${joint_finger_1_origin_xyz}" joint_origin_rpy="${joint_finger_1_origin_rpy}" lower_limit="${joint_finger_1_lower_limit}" upper_limit="${joint_finger_1_upper_limit}"/>
-    <xacro:jaco_link link_name="${link_finger_2}"/>
+    <xacro:jaco_finger_link link_name="${link_finger_2}"/>
     <xacro:jaco_finger_joint joint_name="${joint_finger_2}" type="revolute" parent="${link_hand}" child="${link_finger_2}" joint_axis_xyz="${joint_finger_2_axis_xyz}" joint_origin_xyz="${joint_finger_2_origin_xyz}" joint_origin_rpy="${joint_finger_2_origin_rpy}" lower_limit="${joint_finger_2_lower_limit}" upper_limit="${joint_finger_2_upper_limit}"/>
   </xacro:macro>

File: kinova_description/urdf/standalone_jaco2.xacro (robot description, xacro)
@@ -30,3 +30,9 @@
     </link>
 <xacro:jaco2_arm  parent="root"/>
+<!-- Used to fix the model to the ground in Gazebo. -->
+<link name="world"/>
+<joint name="world_2_root_fixed" type="fixed">
+    <parent link="world"/>
+    <child  link="root"/>
+</joint>
 </robot>

File: kinova_description/urdf/standalone_mico.xacro (robot description, xacro)
@@ -30,3 +30,9 @@
     </link>
 <xacro:mico_arm  parent="root"/>
+<!-- Used to fix the model to the ground in Gazebo. -->
+<link name="world"/>
+<joint name="world_2_root_fixed" type="fixed">
+    <parent link="world"/>
+    <child  link="root"/>
+</joint>
 </robot>
