Commit message: j2_7s_3_standalone pass xacro generation
parameters value have to be in the same file with macros. Seperate j2_7s_config and j2_7s_structure doesn't work.

File: kinova_description/urdf/j2_7s_3_all.xacro (robot description, xacro)
@@ -15,64 +15,64 @@
     xmlns:xacro="http://ros.org/wiki/xacro">
     <xacro:include filename="$(find kinova_description)/urdf/kinova_common.xacro" />
-    <property name="link_base" value="j2_7s_3_link_base" />
-    <property name="link_1" value="j2_7s_3_link_1" />
-    <property name="link_2" value="j2_7s_3_link_2" />
-    <property name="link_3" value="j2_7s_3_link_3" />
-    <property name="link_4" value="j2_7s_3_link_4" />
-    <property name="link_5" value="j2_7s_3_link_5" />
-    <property name="link_6" value="j2_7s_3_link_6" />
-    <property name="link_7" value="j2_7s_3_link_7" />
-    <property name="link_end_effector" value="j2_7s_3_end_effector" />
-    <property name="joint_base" value="j2_7s_3_joint_base" />
-    <property name="joint_base_axis_xyz" value="0 0 0" />
-    <property name="joint_base_origin_xyz" value="0 0 0" />
-    <property name="joint_base_origin_rpy" value="0 0 0" />
-    <property name="joint_1" value="j2_7s_3_joint_1" />
-    <property name="joint_1_axis_xyz" value="0 0 1" />
-    <property name="joint_1_origin_xyz" value="0 0 0.15675" />
-    <property name="joint_1_origin_rpy" value="0 0 0" />
-    <property name="joint_1_lower_limit" value="${-2*J_PI}" />
-    <property name="joint_1_upper_limit" value="${2*J_PI}" />
-    <property name="joint_2" value="j2_7s_3_joint_2" />
-    <property name="joint_2_axis_xyz" value="0 0 1" />
-    <property name="joint_2_origin_xyz" value="0 0.0016 -0.11875" />
-    <property name="joint_2_origin_rpy" value="${-J_PI/2} 0 ${J_PI}" />
-    <property name="joint_2_lower_limit" value="${-J_PI}" />
-    <property name="joint_2_upper_limit" value="${0}" />
-    <property name="joint_3" value="j2_7s_3_joint_3" />
-    <property name="joint_3_axis_xyz" value="0 0 1" />
-    <property name="joint_3_origin_xyz" value="0 -0.205 0" />
-    <property name="joint_3_origin_rpy" value="${J_PI} 0 ${J_PI}" />
-    <property name="joint_3_lower_limit" value="${-5*J_PI/4}" />
-    <property name="joint_3_upper_limit" value="${1*J_PI/4}" />
-    <property name="joint_4" value="j2_7s_3_joint_4" />
-    <property name="joint_4_axis_xyz" value="0 0 1" />
-    <property name="joint_4_origin_xyz" value="0 0 -0.205" />
-    <property name="joint_4_origin_rpy" value="${J_PI/2} ${J_PI/2} 0" />
-    <property name="joint_4_lower_limit" value="${-2*J_PI}" />
-    <property name="joint_4_upper_limit" value="${2*J_PI}" />
-    <property name="joint_5" value="j2_7s_3_joint_5" />
-    <property name="joint_5_axis_xyz" value="0 0 1" />
-    <property name="joint_5_origin_xyz" value="0 0.2073 -0.0114" />
-    <property name="joint_5_origin_rpy" value="${-J_PI/3} 0 0" />
-    <property name="joint_5_lower_limit" value="${-2*J_PI}" />
-    <property name="joint_5_upper_limit" value="${2*J_PI}" />
-    <property name="joint_6" value="j2_7s_3_joint_6" />
-    <property name="joint_6_axis_xyz" value="0 0 1" />
-    <property name="joint_6_origin_xyz" value="0 -0.03703 -0.06414" />
-    <property name="joint_6_origin_rpy" value="${-J_PI/3} 0 0" />
-    <property name="joint_6_lower_limit" value="${-2*J_PI}" />
-    <property name="joint_6_upper_limit" value="${2*J_PI}" />
-    <property name="joint_7" value="j2_7s_3_joint_7" />
-    <property name="joint_7_axis_xyz" value="0 0 1" />
-    <property name="joint_7_origin_xyz" value="0 -0.03703 -0.06414" />
-    <property name="joint_7_origin_rpy" value="${-J_PI/3} 0 0" />
-    <property name="joint_7_lower_limit" value="${-2*J_PI}" />
-    <property name="joint_7_upper_limit" value="${2*J_PI}" />
-    <property name="joint_end_effector" value="j2_7s_3_end_effector_offset" />
-    <property name="joint_end_effector_axis_xyz" value="0 0 0" />
-    <property name="joint_end_effector_origin_xyz" value="0 0 -0.1600" />
-    <property name="joint_end_effector_origin_rpy" value="0 0 0" />
-    <xacro:macro name="j2_7s_3" params="base_parent">
+        <property name="link_base" value="j2_7s_3_link_base" />
+        <property name="link_1" value="j2_7s_3_link_1" />
+        <property name="link_2" value="j2_7s_3_link_2" />
+        <property name="link_3" value="j2_7s_3_link_3" />
+        <property name="link_4" value="j2_7s_3_link_4" />
+        <property name="link_5" value="j2_7s_3_link_5" />
+        <property name="link_6" value="j2_7s_3_link_6" />
+        <property name="link_7" value="j2_7s_3_link_7" />
+        <property name="link_end_effector" value="j2_7s_3_end_effector" />
+        <property name="joint_base" value="j2_7s_3_joint_base" />
+        <property name="joint_base_axis_xyz" value="0 0 0" />
+        <property name="joint_base_origin_xyz" value="0 0 0" />
+        <property name="joint_base_origin_rpy" value="0 0 0" />
+        <property name="joint_1" value="j2_7s_3_joint_1" />
+        <property name="joint_1_axis_xyz" value="0 0 1" />
+        <property name="joint_1_origin_xyz" value="0 0 0.15675" />
+        <property name="joint_1_origin_rpy" value="0 0 0" />
+        <property name="joint_1_lower_limit" value="${-2*J_PI}" />
+        <property name="joint_1_upper_limit" value="${2*J_PI}" />
+        <property name="joint_2" value="j2_7s_3_joint_2" />
+        <property name="joint_2_axis_xyz" value="0 0 1" />
+        <property name="joint_2_origin_xyz" value="0 0.0016 -0.11875" />
+        <property name="joint_2_origin_rpy" value="${-J_PI/2} 0 ${J_PI}" />
+        <property name="joint_2_lower_limit" value="${-J_PI}" />
+        <property name="joint_2_upper_limit" value="${0}" />
+        <property name="joint_3" value="j2_7s_3_joint_3" />
+        <property name="joint_3_axis_xyz" value="0 0 1" />
+        <property name="joint_3_origin_xyz" value="0 -0.205 0" />
+        <property name="joint_3_origin_rpy" value="${J_PI} 0 ${J_PI}" />
+        <property name="joint_3_lower_limit" value="${-5*J_PI/4}" />
+        <property name="joint_3_upper_limit" value="${1*J_PI/4}" />
+        <property name="joint_4" value="j2_7s_3_joint_4" />
+        <property name="joint_4_axis_xyz" value="0 0 1" />
+        <property name="joint_4_origin_xyz" value="0 0 -0.205" />
+        <property name="joint_4_origin_rpy" value="${J_PI/2} ${J_PI/2} 0" />
+        <property name="joint_4_lower_limit" value="${-2*J_PI}" />
+        <property name="joint_4_upper_limit" value="${2*J_PI}" />
+        <property name="joint_5" value="j2_7s_3_joint_5" />
+        <property name="joint_5_axis_xyz" value="0 0 1" />
+        <property name="joint_5_origin_xyz" value="0 0.2073 -0.0114" />
+        <property name="joint_5_origin_rpy" value="${-J_PI/3} 0 0" />
+        <property name="joint_5_lower_limit" value="${-2*J_PI}" />
+        <property name="joint_5_upper_limit" value="${2*J_PI}" />
+        <property name="joint_6" value="j2_7s_3_joint_6" />
+        <property name="joint_6_axis_xyz" value="0 0 1" />
+        <property name="joint_6_origin_xyz" value="0 -0.03703 -0.06414" />
+        <property name="joint_6_origin_rpy" value="${-J_PI/3} 0 0" />
+        <property name="joint_6_lower_limit" value="${-2*J_PI}" />
+        <property name="joint_6_upper_limit" value="${2*J_PI}" />
+        <property name="joint_7" value="j2_7s_3_joint_7" />
+        <property name="joint_7_axis_xyz" value="0 0 1" />
+        <property name="joint_7_origin_xyz" value="0 -0.03703 -0.06414" />
+        <property name="joint_7_origin_rpy" value="${-J_PI/3} 0 0" />
+        <property name="joint_7_lower_limit" value="${-2*J_PI}" />
+        <property name="joint_7_upper_limit" value="${2*J_PI}" />
+        <property name="joint_end_effector" value="j2_7s_3_end_effector_offset" />
+        <property name="joint_end_effector_axis_xyz" value="0 0 0" />
+        <property name="joint_end_effector_origin_xyz" value="0 0 -0.1600" />
+        <property name="joint_end_effector_origin_rpy" value="0 0 0" />
+    <xacro:macro name="j2_7s_3_all" params="base_parent">
         <xacro:kinova_armlink link_name="${link_base}"/>
         <xacro:kinova_armjoint joint_name="${joint_base}" type="fixed" parent="${base_parent}" child="${link_base}" joint_axis_xyz="${joint_base_axis_xyz}" joint_origin_xyz="${joint_base_origin_xyz}" joint_origin_rpy="${joint_base_origin_rpy}" joint_lower_limit="0" joint_upper_limit="0"/>

File: kinova_description/urdf/j2_7s_config.xacro (robot description, xacro)
@@ -23,5 +23,5 @@
     <property name="link_6" value="${prefix}_link_6" />
     <property name="link_7" value="${prefix}_link_7" />
-    <property name="link_end_effector"   value="${prefix}_end_effector" />
+    <property name="link_end_effector" value="${prefix}_end_effector" />
     <property name="joint_base" value="${prefix}_joint_base" />
     <property name="joint_base_axis_xyz" value="0 0 0" />
@@ -64,10 +64,10 @@
     <property name="joint_6_lower_limit" value="${-2*J_PI}" />
     <property name="joint_6_upper_limit" value="${2*J_PI}" />
-    <property name="joint_6" value="${prefix}_joint_6" />
-    <property name="joint_6_axis_xyz" value="0 0 1" />
-    <property name="joint_6_origin_xyz" value="0 -0.03703 -0.06414" />
-    <property name="joint_6_origin_rpy" value="${-J_PI/3} 0 0" />
-    <property name="joint_6_lower_limit" value="${-2*J_PI}" />
-    <property name="joint_6_upper_limit" value="${2*J_PI}" />
+    <property name="joint_7" value="${prefix}_joint_7" />
+    <property name="joint_7_axis_xyz" value="0 0 1" />
+    <property name="joint_7_origin_xyz" value="0 -0.03703 -0.06414" />
+    <property name="joint_7_origin_rpy" value="${-J_PI/3} 0 0" />
+    <property name="joint_7_lower_limit" value="${-2*J_PI}" />
+    <property name="joint_7_upper_limit" value="${2*J_PI}" />
     <property name="joint_end_effector" value="${prefix}_end_effector_offset" />
     <property name="joint_end_effector_axis_xyz" value="0 0 0" />

File: kinova_description/urdf/j2_7s_structure.xacro (robot description, xacro)
@@ -15,5 +15,7 @@
 	xmlns:xacro="http://ros.org/wiki/xacro">
   <xacro:include filename="$(find kinova_description)/urdf/kinova_common.xacro" />
-  <xacro:macro name="j2_7s_structure" params="base_parent">
+  <xacro:include filename="$(find kinova_description)/urdf/j2_7s_config.xacro" />
+  <xacro:j2_7s_config prefix="prefix"/>
+  <xacro:macro name="j2_7s_structure" params="prefix base_parent">
     <xacro:kinova_armlink link_name="${link_base}"/>
     <xacro:kinova_armjoint joint_name="${joint_base}" type="fixed" parent="${base_parent}" child="${link_base}" joint_axis_xyz="${joint_base_axis_xyz}" joint_origin_xyz="${joint_base_origin_xyz}" joint_origin_rpy="${joint_base_origin_rpy}" joint_lower_limit="0" joint_upper_limit="0"/>

File: kinova_description/urdf/jaco2_arm.xacro (robot description, xacro)
@@ -13,5 +13,6 @@
     xmlns:physics="http://playerstage.sourceforge.net/gazebo/xmlschema/#physics"
 	xmlns:xacro="http://ros.org/wiki/xacro">
-  <xacro:include filename="$(find kinova_description)/urdf/jaco_common.xacro" />
+  <xacro:include filename="$(find kinova_description)/urdf/kinova_6DOF.xacro" />
+  <xacro:include filename="$(find kinova_description)/urdf/kinova_3fingers.xacro"/>
   <property name="link_base" value="jaco2_link_base" />
   <property name="link_1" value="jaco2_link_1" />
@@ -20,8 +21,11 @@
   <property name="link_4" value="jaco2_link_4" />
   <property name="link_5" value="jaco2_link_5" />
-  <property name="link_hand" value="jaco2_link_hand" />
+  <property name="link_6" value="jaco2_link_6" />
   <property name="link_finger_1" value="jaco2_link_finger_1" />
   <property name="link_finger_2" value="jaco2_link_finger_2" />
   <property name="link_finger_3" value="jaco2_link_finger_3" />
+  <property name="link_finger_tip_1" value="jaco2_link_finger_tip_1" />
+  <property name="link_finger_tip_2" value="jaco2_link_finger_tip_2" />
+  <property name="link_finger_tip_3" value="jaco2_link_finger_tip_3" />
   <property name="api_offset" value="0.028" />
   <property name="api_origin" value="jaco2_api_origin" />
@@ -31,45 +35,54 @@
   <property name="joint_base_origin_rpy" value="0 0 0" />
   <property name="joint_1" value="jaco2_joint_1" />
-  <property name="joint_1_axis_xyz" value="0 0 -1" />
+  <property name="joint_1_axis_xyz" value="0 0 1" />
   <property name="joint_1_origin_xyz" value="0 0 0.1535" />
-  <property name="joint_1_origin_rpy" value="${J_PI} 0 ${J_PI}" />
+  <property name="joint_1_origin_rpy" value="0 0 0" />
   <property name="joint_1_lower_limit" value="${-2*J_PI}" />
   <property name="joint_1_upper_limit" value="${2*J_PI}" />
   <property name="joint_2" value="jaco2_joint_2" />
   <property name="joint_2_axis_xyz" value="0 0 1" />
-  <property name="joint_2_origin_xyz" value="0 0 -0.1185" />
-  <property name="joint_2_origin_rpy" value="-${J_PI/2} ${J_PI} 0" />
+  <property name="joint_2_origin_xyz" value="0 0 0.1185" />
+  <property name="joint_2_origin_rpy" value="${-J_PI/2} 0 ${J_PI}" />
   <property name="joint_2_lower_limit" value="${-J_PI}" />
   <property name="joint_2_upper_limit" value="${0}" />
   <property name="joint_3" value="jaco2_joint_3" />
-  <property name="joint_3_axis_xyz" value="0 0 -1" />
-  <property name="joint_3_origin_xyz" value="0.41 0 0" />
-  <property name="joint_3_origin_rpy" value="${J_PI} 0 ${J_PI/2}" />
+  <property name="joint_3_axis_xyz" value="0 0 1" />
+  <property name="joint_3_origin_xyz" value="0 0.41 0" />
+  <property name="joint_3_origin_rpy" value="${J_PI} 0 ${J_PI}" />
   <property name="joint_3_lower_limit" value="${-5*J_PI/4}" />
   <property name="joint_3_upper_limit" value="${1*J_PI/4}" />
   <property name="joint_4" value="jaco2_joint_4" />
-  <property name="joint_4_axis_xyz" value="0 0 -1" />
-  <property name="joint_4_origin_xyz" value="0.207 0 -0.01125" />
-  <property name="joint_4_origin_rpy" value="${J_PI} ${J_PI/2} 0" />
+  <property name="joint_4_axis_xyz" value="0 0 1" />
+  <property name="joint_4_origin_xyz" value="0 -0.207 0.01125" />
+  <property name="joint_4_origin_rpy" value="${J_PI/2} ${J_PI/2} 0" />
   <property name="joint_4_lower_limit" value="${-2*J_PI}" />
   <property name="joint_4_upper_limit" value="${2*J_PI}" />
-  <property name="joint_5" value="jaco_joint_5" />
-  <property name="joint_5_axis_xyz" value="0 0 -1" />
-  <property name="joint_5_origin_xyz" value="0.03700 0 -0.06408" />
-  <property name="joint_5_origin_rpy" value="0 -${J_PI/180*60} 0" />
+  <property name="joint_5" value="jaco2_joint_5" />
+  <property name="joint_5_axis_xyz" value="0 0 1" />
+  <property name="joint_5_origin_xyz" value="0 0.03700 0.06408" />
+  <property name="joint_5_origin_rpy" value="${-J_PI/3} 0 0" />
   <property name="joint_5_lower_limit" value="${-2*J_PI}" />
   <property name="joint_5_upper_limit" value="${2*J_PI}" />
-  <property name="joint_6" value="jaco_joint_6" />
-  <property name="joint_6_axis_xyz" value="0 0 -1" />
-  <property name="joint_6_origin_xyz" value="0.03700 0 -0.06408" />
-  <property name="joint_6_origin_rpy" value="-${J_PI/180*60} 0 ${J_PI/2}" />
+  <property name="joint_6" value="jaco2_joint_6" />
+  <property name="joint_6_axis_xyz" value="0 0 1" />
+  <property name="joint_6_origin_xyz" value="0 0.03700 0.06408" />
+  <property name="joint_6_origin_rpy" value="${-J_PI/3} 0 0" />
   <property name="joint_6_lower_limit" value="${-2*J_PI}" />
   <property name="joint_6_upper_limit" value="${2*J_PI}" />
   <property name="joint_finger_1" value="jaco2_joint_finger_1" />
   <property name="joint_finger_1_axis_xyz" value="0 0 1" />
-  <property name="joint_finger_1_origin_xyz" value="-0.03978 0 -0.10071" />
-  <property name="joint_finger_1_origin_rpy" value="-1.7983 1.117 3.1416" />
+  <property name="joint_finger_1_origin_xyz" value="0 -0.03978 0.10071" />
+  <property name="joint_finger_1_origin_rpy" value="1.117 0 0" />
   <property name="joint_finger_1_lower_limit" value="0" />
   <property name="joint_finger_1_upper_limit" value="${J_PI/180*40}" />
+  <property name="joint_finger_tip_1" value="jaco2_joint_finger_tip_1" />
+  <property name="joint_finger_tip_1_axis_xyz" value="0 0 1" />
+  <property name="joint_finger_tip_1_origin_xyz" value="0.035 -0.02595 -0.0025" />
+  <property name="joint_finger_tip_1_origin_rpy" value="0 0 0" />
+  <property name="joint_finger_tip_1_lower_limit" value="0" />
+  <property name="joint_finger_tip_1_upper_limit" value="${J_PI/180*40}" />
+  <property name="joint_finger_tip_1_mimic_joint" value="${J_PI/180*40}" />
+  <property name="joint_finger_tip_1_mimic_multiplier" value="0.0" />
+  <property name="joint_finger_tip_1_mimc_offset" value="0.0" />
   <property name="joint_finger_2" value="jaco2_joint_finger_2" />
   <property name="joint_finger_2_axis_xyz" value="0 0 1" />
@@ -78,4 +91,13 @@
   <property name="joint_finger_2_lower_limit" value="0" />
   <property name="joint_finger_2_upper_limit" value="${J_PI/180*40}" />
+  <property name="joint_finger_tip_2" value="jaco2_joint_finger_tip_2" />
+  <property name="joint_finger_tip_2_axis_xyz" value="0 0 1" />
+  <property name="joint_finger_tip_2_origin_xyz" value="0.035 -0.02595 -0.0025" />
+  <property name="joint_finger_tip_2_origin_rpy" value="0 0 0" />
+  <property name="joint_finger_tip_2_lower_limit" value="0" />
+  <property name="joint_finger_tip_2_upper_limit" value="${J_PI/180*40}" />
+  <property name="joint_finger_tip_2_mimic_joint" value="${J_PI/180*40}" />
+  <property name="joint_finger_tip_2_mimic_multiplier" value="0.0" />
+  <property name="joint_finger_tip_2_mimc_offset" value="0.0" />
   <property name="joint_finger_3" value="jaco2_joint_finger_3" />
   <property name="joint_finger_3_axis_xyz" value="0 0 1" />
@@ -84,14 +106,24 @@
   <property name="joint_finger_3_lower_limit" value="0" />
   <property name="joint_finger_3_upper_limit" value="${J_PI/180*40}" />
+  <property name="joint_finger_tip_3" value="jaco3_joint_finger_tip_3" />
+  <property name="joint_finger_tip_3_axis_xyz" value="0 0 1" />
+  <property name="joint_finger_tip_3_origin_xyz" value="0.035 -0.02595 -0.0025" />
+  <property name="joint_finger_tip_3_origin_rpy" value="0 0 0" />
+  <property name="joint_finger_tip_3_lower_limit" value="0" />
+  <property name="joint_finger_tip_3_upper_limit" value="${J_PI/180*40}" />
+  <property name="joint_finger_tip_3_mimic_joint" value="${J_PI/180*40}" />
+  <property name="joint_finger_tip_3_mimic_multiplier" value="0.0" />
+  <property name="joint_finger_tip_3_mimc_offset" value="0.0" />
   <property name="link_end_effector"   value="jaco2_end_effector" />
   <property name="end_effector_offset" value="0.1687" />
   <xacro:macro name="jaco2_arm" params="parent">
-    <xacro:jaco_struct parent="${parent}" basename="jaco2"/>
-    <xacro:jaco_link link_name="${link_finger_1}"/>
-    <xacro:jaco_finger_joint joint_name="${joint_finger_1}" type="revolute" parent="${link_hand}" child="${link_finger_1}" joint_axis_xyz="${joint_finger_1_axis_xyz}" joint_origin_xyz="${joint_finger_1_origin_xyz}" joint_origin_rpy="${joint_finger_1_origin_rpy}" lower_limit="${joint_finger_1_lower_limit}" upper_limit="${joint_finger_1_upper_limit}"/>
-    <xacro:jaco_link link_name="${link_finger_2}"/>
-    <xacro:jaco_finger_joint joint_name="${joint_finger_2}" type="revolute" parent="${link_hand}" child="${link_finger_2}" joint_axis_xyz="${joint_finger_2_axis_xyz}" joint_origin_xyz="${joint_finger_2_origin_xyz}" joint_origin_rpy="${joint_finger_2_origin_rpy}" lower_limit="${joint_finger_2_lower_limit}" upper_limit="${joint_finger_2_upper_limit}"/>
-    <xacro:jaco_link link_name="${link_finger_3}"/>
-    <xacro:jaco_finger_joint joint_name="${joint_finger_3}" type="revolute" parent="${link_hand}" child="${link_finger_3}" joint_axis_xyz="${joint_finger_3_axis_xyz}" joint_origin_xyz="${joint_finger_3_origin_xyz}" joint_origin_rpy="${joint_finger_3_origin_rpy}" lower_limit="${joint_finger_3_lower_limit}" upper_limit="${joint_finger_3_upper_limit}"/>
+    <xacro:kinova_6DOF base_parent="${parent}"/>
+    <link name="${link_end_effector}" />
+    <joint name="${link_6}_to_end_effector" type="fixed">
+      <parent link="${link_6}"/>
+      <child link="${link_end_effector}"/>
+      <origin xyz="0 0 -${end_effector_offset}" rpy="0 ${J_PI} 0" />
+    </joint>
+    <xacro:kinova_3fingers link_hand="${link_6}"/>
   </xacro:macro>
 </root>

File: kinova_description/urdf/kinova_common.xacro (robot description, xacro)
@@ -42,22 +42,22 @@
      </joint>
     </xacro:macro>
-    <xacro:macro name="kinova_fingerjoint" params="joint_name type parent child joint_axis_xyz joint_origin_xyz joint_origin_rpy lower_limit upper_limit">
-    <joint name="${joint_name}" type="${type}">
-        <parent link="${parent}"/>
-        <child link="${child}"/>
-        <axis xyz="${joint_axis_xyz}"/>
-        <origin xyz="${joint_origin_xyz}" rpy="${joint_origin_rpy}"/>
-        <limit lower="${lower_limit}" upper="${upper_limit}" effort="30" velocity="5"/>
-     </joint>
-    </xacro:macro>
-   <xacro:macro name="kinova_fingertipjoint" params="joint_name type parent child joint_axis_xyz joint_origin_xyz joint_origin_rpy lower_limit upper_limit mimic_joint mimic_multiplier mimic_offset">
-    <joint name="${joint_name}" type="${type}">
-        <parent link="${parent}"/>
-        <child link="${child}"/>
-        <axis xyz="${joint_axis_xyz}"/>
-        <origin xyz="${joint_origin_xyz}" rpy="${joint_origin_rpy}"/>
-        <limit lower="${lower_limit}" upper="${upper_limit}" effort="30" velocity="5"/>
-        <mimic joint="${mimic_joint}" multiplier="${mimic_multiplier}" offset="${mimic_offset}"/>
-     </joint>
+    <xacro:macro name="kinova_finger" params="joint_name type parent joint_axis_xyz joint_origin_xyz joint_origin_rpy lower_limit upper_limit lower_limit_tip upper_limit_tip mimic_joint mimic_multiplier mimic_offset">
+        <LINK />
+        <joint name="${joint_name}" type="${type}">
+            <parent link="${parent}"/>
+            <child link="${child}"/>
+            <axis xyz="${joint_axis_xyz}"/>
+            <origin xyz="${joint_origin_xyz}" rpy="${joint_origin_rpy}"/>
+            <limit lower="${lower_limit}" upper="${upper_limit}" effort="30" velocity="5"/>
+        </joint>
+        <LINK />
+        <joint name="${joint_name}" type="${type}">
+            <parent link="${parent}"/>
+            <child link="${child}"/>
+            <axis xyz="${joint_axis_xyz}"/>
+            <origin xyz="${joint_origin_xyz}" rpy="${joint_origin_rpy}"/>
+            <limit lower="${lower_limit_tip}" upper="${upper_limit_tip}" effort="30" velocity="5"/>
+            <mimic joint="${mimic_joint}" multiplier="${mimic_multiplier}" offset="${mimic_offset}"/>
+        </joint>
     </xacro:macro>
 </root>
