Commit message: add mesh to j2_7s_3

File: kinova_description/urdf/j2_7s_3.xacro (robot description, xacro)
@@ -24,4 +24,12 @@
     <property name="link_7" value="j2_7s_3_link_7" />
     <property name="link_end_effector" value="j2_7s_3_end_effector" />
+    <property name="link_base_mesh" value="base" />
+    <property name="link_1_mesh" value="shoulder" />
+    <property name="link_2_mesh" value="arm_half_1" />
+    <property name="link_3_mesh" value="arm_half_2" />
+    <property name="link_4_mesh" value="forearm" />
+    <property name="link_5_mesh" value="wrist_spherical_1" />
+    <property name="link_6_mesh" value="wrist_spherical_2" />
+    <property name="link_7_mesh" value="hand_3finger" />
     <property name="joint_base" value="j2_7s_3_joint_base" />
     <property name="joint_base_axis_xyz" value="0 0 0" />
@@ -75,19 +83,19 @@
     <property name="joint_end_effector_origin_rpy" value="0 0 0" />
     <xacro:macro name="j2_7s_3" params="base_parent">
-        <xacro:kinova_armlink link_name="${link_base}"/>
+        <xacro:kinova_armlink link_name="${link_base}" link_mesh="${link_base_mesh}"/>
         <xacro:kinova_armjoint joint_name="${joint_base}" type="fixed" parent="${base_parent}" child="${link_base}" joint_axis_xyz="${joint_base_axis_xyz}" joint_origin_xyz="${joint_base_origin_xyz}" joint_origin_rpy="${joint_base_origin_rpy}" joint_lower_limit="0" joint_upper_limit="0"/>
-        <xacro:kinova_armlink link_name="${link_1}"/>
+        <xacro:kinova_armlink link_name="${link_1}" link_mesh="${link_1_mesh}"/>
         <xacro:kinova_armjoint joint_name="${joint_1}" type="continuous" parent="${link_base}" child="${link_1}" joint_axis_xyz="${joint_1_axis_xyz}" joint_origin_xyz="${joint_1_origin_xyz}" joint_origin_rpy="${joint_1_origin_rpy}" joint_lower_limit="${joint_1_lower_limit}" joint_upper_limit="${joint_1_upper_limit}"/>
-        <xacro:kinova_armlink link_name="${link_2}"/>
+        <xacro:kinova_armlink link_name="${link_2}" link_mesh="${link_2_mesh}"/>
         <xacro:kinova_armjoint joint_name="${joint_2}" type="revolute" parent="${link_1}" child="${link_2}" joint_axis_xyz="${joint_2_axis_xyz}" joint_origin_xyz="${joint_2_origin_xyz}" joint_origin_rpy="${joint_2_origin_rpy}" joint_lower_limit="${joint_2_lower_limit}" joint_upper_limit="${joint_2_upper_limit}"/>
-        <xacro:kinova_armlink link_name="${link_3}"/>
+        <xacro:kinova_armlink link_name="${link_3}" link_mesh="${link_3_mesh}"/>
         <xacro:kinova_armjoint joint_name="${joint_3}" type="continuous" parent="${link_2}" child="${link_3}" joint_axis_xyz="${joint_3_axis_xyz}" joint_origin_xyz="${joint_3_origin_xyz}" joint_origin_rpy="${joint_3_origin_rpy}" joint_lower_limit="${joint_3_lower_limit}" joint_upper_limit="${joint_3_upper_limit}"/>
-        <xacro:kinova_armlink link_name="${link_4}"/>
+        <xacro:kinova_armlink link_name="${link_4}" link_mesh="${link_4_mesh}"/>
         <xacro:kinova_armjoint joint_name="${joint_4}" type="revolute" parent="${link_3}" child="${link_4}" joint_axis_xyz="${joint_4_axis_xyz}" joint_origin_xyz="${joint_4_origin_xyz}" joint_origin_rpy="${joint_4_origin_rpy}" joint_lower_limit="${joint_4_lower_limit}" joint_upper_limit="${joint_4_upper_limit}"/>
-        <xacro:kinova_armlink link_name="${link_5}"/>
+        <xacro:kinova_armlink link_name="${link_5}" link_mesh="${link_5_mesh}"/>
         <xacro:kinova_armjoint joint_name="${joint_5}" type="continuous" parent="${link_4}" child="${link_5}" joint_axis_xyz="${joint_5_axis_xyz}" joint_origin_xyz="${joint_5_origin_xyz}" joint_origin_rpy="${joint_5_origin_rpy}" joint_lower_limit="${joint_5_lower_limit}" joint_upper_limit="${joint_5_upper_limit}"/>
-        <xacro:kinova_armlink link_name="${link_6}" />
+        <xacro:kinova_armlink link_name="${link_6}" link_mesh="${link_6_mesh}"/>
         <xacro:kinova_armjoint joint_name="${joint_6}" type="revolute" parent="${link_5}" child="${link_6}" joint_axis_xyz="${joint_6_axis_xyz}" joint_origin_xyz="${joint_6_origin_xyz}" joint_origin_rpy="${joint_6_origin_rpy}" joint_lower_limit="${joint_6_lower_limit}" joint_upper_limit="${joint_6_upper_limit}"/>
-        <xacro:kinova_armlink link_name="${link_7}" />
+        <xacro:kinova_armlink link_name="${link_7}" link_mesh="${link_7_mesh}"/>
         <xacro:kinova_armjoint joint_name="${joint_7}" type="continuous" parent="${link_6}" child="${link_7}" joint_axis_xyz="${joint_7_axis_xyz}" joint_origin_xyz="${joint_7_origin_xyz}" joint_origin_rpy="${joint_7_origin_rpy}" joint_lower_limit="${joint_7_lower_limit}" joint_upper_limit="${joint_7_upper_limit}"/>
         <xacro:kinova_armlink link_name="${link_end_effector}" />

File: kinova_description/urdf/kinova_common.xacro (robot description, xacro)
@@ -14,10 +14,10 @@
 	xmlns:xacro="http://ros.org/wiki/xacro">
     <property name="J_PI" value="3.1415926535897931" />
-    <xacro:macro name="kinova_armlink" params="link_name">
+    <xacro:macro name="kinova_armlink" params="link_name link_mesh">
         <link name="${link_name}">
             <visual>
                 <geometry>
                     <mesh
-                        filename="package://kinova_description/meshes/${link_name}.dae"/>
+                        filename="package://kinova_description/meshes/${link_mesh}.dae"/>
                 </geometry>
                 <material name="carbon_fiber">
@@ -28,5 +28,5 @@
                 <geometry>
                     <mesh
-                        filename="package://kinova_description/meshes/${link_name}.dae"/>
+                        filename="package://kinova_description/meshes/${link_mesh}.dae"/>
                 </geometry>
             </collision>

Commit message: 3finger: first finger OK

File: kinova_description/urdf/j2_7s_3.xacro (robot description, xacro)
@@ -15,4 +15,6 @@
     xmlns:xacro="http://ros.org/wiki/xacro">
     <xacro:include filename="$(find kinova_description)/urdf/kinova_common.xacro" />
+    <xacro:include filename="$(find kinova_description)/urdf/kinova_3fingers.xacro" />
+    <property name="prefix" value="j2_7s_3" />
     <property name="link_base" value="j2_7s_3_link_base" />
     <property name="link_1" value="j2_7s_3_link_1" />
@@ -111,3 +113,4 @@
         <xacro:kinova_virtual_joint joint_name="${joint_end_effector}" type="${joint_end_effector_type}" parent="${link_7}" child="${link_end_effector}" joint_axis_xyz="${joint_end_effector_axis_xyz}" joint_origin_xyz="${joint_end_effector_origin_xyz}" joint_origin_rpy="${joint_end_effector_origin_rpy}" joint_lower_limit="0" joint_upper_limit="0"/>
     </xacro:macro>
+    <xacro:kinova_3fingers link_hand="${link_7}" />
 </root>

File: kinova_description/urdf/kinova_3fingers.xacro (robot description, xacro)
@@ -1,29 +1,23 @@
 <?xml version="1.0"?>
+<!-- j2_7s refers to jaco v2 7DOF spherical -->
 <root xmlns:xi="http://www.w3.org/2001/XInclude"
-	xmlns:gazebo="http://playerstage.sourceforge.net/gazebo/xmlschema/#gz"
+    xmlns:gazebo="http://playerstage.sourceforge.net/gazebo/xmlschema/#gz"
     xmlns:model="http://playerstage.sourceforge.net/gazebo/xmlschema/#model"
-	xmlns:sensor="http://playerstage.sourceforge.net/gazebo/xmlschema/#sensor"
-	xmlns:body="http://playerstage.sourceforge.net/gazebo/xmlschema/#body"
+    xmlns:sensor="http://playerstage.sourceforge.net/gazebo/xmlschema/#sensor"
+    xmlns:body="http://playerstage.sourceforge.net/gazebo/xmlschema/#body"
     xmlns:geom="http://playerstage.sourceforge.net/gazebo/xmlschema/#geom"
     xmlns:joint="http://playerstage.sourceforge.net/gazebo/xmlschema/#joint"
-	xmlns:controller="http://playerstage.sourceforge.net/gazebo/xmlschema/#controller"
-	xmlns:interface="http://playerstage.sourceforge.net/gazebo/xmlschema/#interface"
-	xmlns:rendering="http://playerstage.sourceforge.net/gazebo/xmlschema/#rendering"
+    xmlns:controller="http://playerstage.sourceforge.net/gazebo/xmlschema/#controller"
+    xmlns:interface="http://playerstage.sourceforge.net/gazebo/xmlschema/#interface"
+    xmlns:rendering="http://playerstage.sourceforge.net/gazebo/xmlschema/#rendering"
     xmlns:renderable="http://playerstage.sourceforge.net/gazebo/xmlschema/#renderable"
     xmlns:physics="http://playerstage.sourceforge.net/gazebo/xmlschema/#physics"
-	xmlns:xacro="http://ros.org/wiki/xacro">
-  <xacro:macro name="kinova_3fingers" params="link_hand">
-    <xacro:kinova_armlink link_name="${link_finger_1}"/>
-    <xacro:kinova_fingerjoint joint_name="${joint_finger_1}" type="revolute" parent="${link_hand}" child="${link_finger_1}" joint_axis_xyz="${joint_finger_1_axis_xyz}" joint_origin_xyz="${joint_finger_1_origin_xyz}" joint_origin_rpy="${joint_finger_1_origin_rpy}" lower_limit="${joint_finger_1_lower_limit}" upper_limit="${joint_finger_1_upper_limit}"/>
-    <xacro:kinova_armlink link_name="${link_finger_tip_1}"/>
-    <xacro:kinova_fingertipjoint joint_name="${joint_finger_tip_1}" type="revolute" parent="${link_finger_1}" child="${link_finger_tip_1}" joint_axis_xyz="${joint_finger_tip_1_axis_xyz}" joint_origin_xyz="${joint_finger_tip_1_origin_xyz}" joint_origin_rpy="${joint_finger_tip_1_origin_rpy}" lower_limit="${joint_finger_tip_1_lower_limit}" upper_limit="${joint_finger_tip_1_upper_limit}" mimic_joint="${joint_finger_1}" mimic_multiplier="${joint_finger_tip_1_mimic_multiplier}" mimic_offset="${joint_finger_tip_1_mimc_offset}"/>
-    <xacro:kinova_armlink link_name="${link_finger_2}"/>
-    <xacro:kinova_fingerjoint joint_name="${joint_finger_2}" type="revolute" parent="${link_hand}" child="${link_finger_2}" joint_axis_xyz="${joint_finger_2_axis_xyz}" joint_origin_xyz="${joint_finger_2_origin_xyz}" joint_origin_rpy="${joint_finger_2_origin_rpy}" lower_limit="${joint_finger_2_lower_limit}" upper_limit="${joint_finger_2_upper_limit}"/>
-    <xacro:kinova_armlink link_name="${link_finger_tip_2}"/>
-    <xacro:kinova_fingertipjoint joint_name="${joint_finger_tip_2}" type="revolute" parent="${link_finger_2}" child="${link_finger_tip_2}" joint_axis_xyz="${joint_finger_tip_2_axis_xyz}" joint_origin_xyz="${joint_finger_tip_2_origin_xyz}" joint_origin_rpy="${joint_finger_tip_2_origin_rpy}" lower_limit="${joint_finger_tip_2_lower_limit}" upper_limit="${joint_finger_tip_2_upper_limit}" mimic_joint="${joint_finger_2}" mimic_multiplier="${joint_finger_tip_2_mimic_multiplier}" mimic_offset="${joint_finger_tip_2_mimc_offset}"/>
-    <xacro:kinova_armlink link_name="${link_finger_3}"/>
-    <xacro:kinova_fingerjoint joint_name="${joint_finger_3}" type="revolute" parent="${link_hand}" child="${link_finger_3}" joint_axis_xyz="${joint_finger_3_axis_xyz}" joint_origin_xyz="${joint_finger_3_origin_xyz}" joint_origin_rpy="${joint_finger_3_origin_rpy}" lower_limit="${joint_finger_3_lower_limit}" upper_limit="${joint_finger_3_upper_limit}"/>
-    <xacro:kinova_armlink link_name="${link_finger_tip_3}"/>
-    <xacro:kinova_fingertipjoint joint_name="${joint_finger_tip_3}" type="revolute" parent="${link_finger_3}" child="${link_finger_tip_3}" joint_axis_xyz="${joint_finger_tip_3_axis_xyz}" joint_origin_xyz="${joint_finger_tip_3_origin_xyz}" joint_origin_rpy="${joint_finger_tip_3_origin_rpy}" lower_limit="${joint_finger_tip_3_lower_limit}" upper_limit="${joint_finger_tip_3_upper_limit}" mimic_joint="${joint_finger_3}" mimic_multiplier="${joint_finger_tip_3_mimic_multiplier}" mimic_offset="${joint_finger_tip_3_mimc_offset}"/>
-  </xacro:macro>
+    xmlns:xacro="http://ros.org/wiki/xacro">
+    <xacro:include filename="$(find kinova_description)/urdf/kinova_common.xacro" />
+    <xacro:macro name="kinova_3fingers" params="link_hand">
+<!-- 1.310949945 1.150615015 1.149100618 -->
+        <xacro:kinova_finger prefix="test" finger_number="1" hand="${link_hand}" finger_origin_xyz="0.00279 0.03126 -0.11467" finger_origin_rpy="-1.830642709 1.150615015 1.149100618"/>
+        <xacro:kinova_finger prefix="test" finger_number="2" hand="${link_hand}" finger_origin_xyz="-0.02226 -0.02707 -0.11482" finger_origin_rpy="1.570796327 0.1256637062 1.386140492"/>
+        <xacro:kinova_finger prefix="test" finger_number="3" hand="${link_hand}" finger_origin_xyz="0.02226 -0.02707 -0.11482" finger_origin_rpy="0 0 0"/>
+    </xacro:macro>
 </root>

File: kinova_description/urdf/test.xacro (robot description, xacro)
@@ -1,5 +1,5 @@
 <?xml version="1.0"?>
 <!-- j2_7s refers to jaco v2 7DOF spherical -->
-<root xmlns:xi="http://www.w3.org/2001/XInclude"
+<robot xmlns:xi="http://www.w3.org/2001/XInclude"
     xmlns:gazebo="http://playerstage.sourceforge.net/gazebo/xmlschema/#gz"
     xmlns:model="http://playerstage.sourceforge.net/gazebo/xmlschema/#model"
@@ -13,16 +13,25 @@
     xmlns:renderable="http://playerstage.sourceforge.net/gazebo/xmlschema/#renderable"
     xmlns:physics="http://playerstage.sourceforge.net/gazebo/xmlschema/#physics"
-    xmlns:xacro="http://ros.org/wiki/xacro">
-  <xacro:include filename="$(find kinova_description)/urdf/kinova_common.xacro" />
-    <property name="link_base" value="jaco2_link_base" />
-    <property name="link_1" value="jaco2_link_1" />
-	<property name="base_parent" value="root" />
-  <xacro:macro name="test">
-    <property name="joint_base" value="jaco2_joint_base" />
-    <property name="joint_base_axis_xyz" value="0 0 0" />
-    <property name="joint_base_origin_xyz" value="0 0 0" />
-    <property name="joint_base_origin_rpy" value="0 0 0" />
-    <!-- <xacro:kinova_armlink link_name="${link_base}"/> -->
-    <xacro:kinova_armjoint joint_name="${joint_base}" type="fixed" parent="${base_parent}" child="${link_base}" joint_axis_xyz="${joint_base_axis_xyz}" joint_origin_xyz="${joint_base_origin_xyz}" joint_origin_rpy="${joint_base_origin_rpy}" joint_lower_limit="0" joint_upper_limit="0"/>
-  </xacro:macro>
-</root>
+    xmlns:xacro="http://ros.org/wiki/xacro" name="test">
+    <xacro:include filename="$(find kinova_description)/urdf/kinova_common.xacro" />
+<xacro:include filename="$(find kinova_description)/urdf/kinova_3fingers.xacro" />
+    <property name="prefix" value="j2_7s_3" />
+  <link name="robotbase">
+    <visual>
+      <origin xyz="0 0 0" rpy="0 0 0" />
+      <geometry>
+        <box size = "0 0 0"/>
+      </geometry>
+    <!--<material name="Black" /> -->
+    </visual>
+    <collision>
+      <origin xyz="0 0 0" rpy="0 0 0" />
+      <geometry>
+        <box size = "0 0 0"/>
+      </geometry>
+    </collision>
+  </link>
+  <property name="link_hand" value="robotbase" />
+    <!-- <xacro:kinova_finger prefix="test" finger_number="1" hand="${link_hand}" finger_origin_xyz="0 0 0" finger_origin_rpy="0 0 0"/> -->
+    <xacro:kinova_3fingers link_hand="${link_hand}" />
+</robot>

Commit message: 3 fingers working

File: kinova_description/urdf/j2_7s_3.xacro (robot description, xacro)
@@ -113,4 +113,4 @@
         <xacro:kinova_virtual_joint joint_name="${joint_end_effector}" type="${joint_end_effector_type}" parent="${link_7}" child="${link_end_effector}" joint_axis_xyz="${joint_end_effector_axis_xyz}" joint_origin_xyz="${joint_end_effector_origin_xyz}" joint_origin_rpy="${joint_end_effector_origin_rpy}" joint_lower_limit="0" joint_upper_limit="0"/>
     </xacro:macro>
-    <xacro:kinova_3fingers link_hand="${link_7}" />
+    <xacro:kinova_3fingers link_hand="${link_7}" prefix="${prefix}"/>
 </root>

File: kinova_description/urdf/kinova_3fingers.xacro (robot description, xacro)
@@ -15,9 +15,17 @@
     xmlns:xacro="http://ros.org/wiki/xacro">
     <xacro:include filename="$(find kinova_description)/urdf/kinova_common.xacro" />
-    <xacro:macro name="kinova_3fingers" params="link_hand">
-<!-- 1.310949945 1.150615015 1.149100618 -->
-        <xacro:kinova_finger prefix="test" finger_number="1" hand="${link_hand}" finger_origin_xyz="0.00279 0.03126 -0.11467" finger_origin_rpy="-1.830642709 1.150615015 1.149100618"/>
-        <xacro:kinova_finger prefix="test" finger_number="2" hand="${link_hand}" finger_origin_xyz="-0.02226 -0.02707 -0.11482" finger_origin_rpy="1.570796327 0.1256637062 1.386140492"/>
-        <xacro:kinova_finger prefix="test" finger_number="3" hand="${link_hand}" finger_origin_xyz="0.02226 -0.02707 -0.11482" finger_origin_rpy="0 0 0"/>
+    <xacro:macro name="kinova_3fingers" params="link_hand prefix">
+        <!-- finger1 Rot := Ry((1/2)*Pi) . Rx(12.1*((1/180)*Pi)+Pi) . Rz(-52.8*((1/180)*Pi)) -->
+        <xacro:kinova_finger prefix="_${prefix}" finger_number="1" hand="${link_hand}" finger_origin_xyz="0.00279 0.03126 -0.11467" finger_origin_rpy="-1.570796327 .649262481663582 1.35961148639407"/>
+        <!-- finger2 Rot := Ry((1/2)*Pi) . Rx(10.58*((1/180)*Pi)) . Rz(-52.8*((1/180)*Pi)) -->
+        <xacro:kinova_finger prefix="_${prefix}" finger_number="2" hand="${link_hand}" finger_origin_xyz="-0.02226 -0.02707 -0.11482" finger_origin_rpy="-1.570796327 .649262481663582 -1.75545216211587"/>
+        <!-- finger3 Rot := Ry((1/2)*Pi) . Rx(-10.58*((1/180)*Pi)) . Rz(-52.8*((1/180)*Pi)) -->
+        <xacro:kinova_finger prefix="_${prefix}" finger_number="3" hand="${link_hand}" finger_origin_xyz="0.02226 -0.02707 -0.11482" finger_origin_rpy="-1.570796327 .649262481663582 -1.38614049188413"/>
+    </xacro:macro>
+    <xacro:macro name="kinova_2fingers" params="link_hand">
+        <!-- finger1 Rot := Ry((1/2)*Pi) . Rx(12.1*((1/180)*Pi)+Pi) . Rz(-52.8*((1/180)*Pi)) -->
+        <xacro:kinova_finger prefix="_${prefix}" finger_number="1" hand="${link_hand}" finger_origin_xyz="0.00279 0.03126 -0.11467" finger_origin_rpy="-1.570796327 .649262481663582 1.35961148639407"/>
+        <!-- finger2 Rot := Ry((1/2)*Pi) . Rx(10.58*((1/180)*Pi)) . Rz(-52.8*((1/180)*Pi)) -->
+        <xacro:kinova_finger prefix="_${prefix}" finger_number="2" hand="${link_hand}" finger_origin_xyz="-0.02226 -0.02707 -0.11482" finger_origin_rpy="-1.570796327 .649262481663582 -1.75545216211587"/>
     </xacro:macro>
 </root>
