Commit message: Add finger set to all robots

File: kinova_description/urdf/j2_4n_3.xacro (robot description, xacro)
@@ -15,4 +15,6 @@
     xmlns:xacro="http://ros.org/wiki/xacro">
     <xacro:include filename="$(find kinova_description)/urdf/kinova_common.xacro" />
+    <xacro:include filename="$(find kinova_description)/urdf/kinova_finger_set.xacro" />
+    <property name="prefix" value="j2_4n_3" />
     <property name="link_base" value="j2_4n_3_link_base" />
     <property name="link_1" value="j2_4n_3_link_1" />
@@ -23,5 +25,5 @@
     <property name="link_base_mesh" value="base" />
     <property name="link_1_mesh" value="shoulder" />
-    <property name="link_2_mesh" value="arm_mico" />
+    <property name="link_2_mesh" value="arm" />
     <property name="link_3_mesh" value="forearm" />
     <property name="link_4_mesh" value="hand_3finger" />
@@ -78,3 +80,4 @@
         <xacro:kinova_virtual_joint joint_name="${joint_end_effector}" type="${joint_end_effector_type}" parent="${link_4}" child="${link_end_effector}" joint_axis_xyz="${joint_end_effector_axis_xyz}" joint_origin_xyz="${joint_end_effector_origin_xyz}" joint_origin_rpy="${joint_end_effector_origin_rpy}" joint_lower_limit="0" joint_upper_limit="0"/>
     </xacro:macro>
+    <xacro:kinova_3fingers link_hand="${link_4}" prefix="${prefix}"/>
 </root>

File: kinova_description/urdf/j2_6n_3.xacro (robot description, xacro)
@@ -15,4 +15,6 @@
     xmlns:xacro="http://ros.org/wiki/xacro">
     <xacro:include filename="$(find kinova_description)/urdf/kinova_common.xacro" />
+    <xacro:include filename="$(find kinova_description)/urdf/kinova_finger_set.xacro" />
+    <property name="prefix" value="j2_6n_3" />
     <property name="link_base" value="j2_6n_3_link_base" />
     <property name="link_1" value="j2_6n_3_link_1" />
@@ -100,3 +102,4 @@
         <xacro:kinova_virtual_joint joint_name="${joint_end_effector}" type="${joint_end_effector_type}" parent="${link_6}" child="${link_end_effector}" joint_axis_xyz="${joint_end_effector_axis_xyz}" joint_origin_xyz="${joint_end_effector_origin_xyz}" joint_origin_rpy="${joint_end_effector_origin_rpy}" joint_lower_limit="0" joint_upper_limit="0"/>
     </xacro:macro>
+    <xacro:kinova_3fingers link_hand="${link_6}" prefix="${prefix}"/>
 </root>

File: kinova_description/urdf/j2_6s_3.xacro (robot description, xacro)
@@ -15,4 +15,6 @@
     xmlns:xacro="http://ros.org/wiki/xacro">
     <xacro:include filename="$(find kinova_description)/urdf/kinova_common.xacro" />
+    <xacro:include filename="$(find kinova_description)/urdf/kinova_finger_set.xacro" />
+    <property name="prefix" value="j2_6s_3" />
     <property name="link_base" value="j2_6s_3_link_base" />
     <property name="link_1" value="j2_6s_3_link_1" />
@@ -100,3 +102,4 @@
         <xacro:kinova_virtual_joint joint_name="${joint_end_effector}" type="${joint_end_effector_type}" parent="${link_6}" child="${link_end_effector}" joint_axis_xyz="${joint_end_effector_axis_xyz}" joint_origin_xyz="${joint_end_effector_origin_xyz}" joint_origin_rpy="${joint_end_effector_origin_rpy}" joint_lower_limit="0" joint_upper_limit="0"/>
     </xacro:macro>
+    <xacro:kinova_3fingers link_hand="${link_6}" prefix="${prefix}"/>
 </root>

File: kinova_description/urdf/j2_7n_3.xacro (robot description, xacro)
@@ -15,4 +15,6 @@
     xmlns:xacro="http://ros.org/wiki/xacro">
     <xacro:include filename="$(find kinova_description)/urdf/kinova_common.xacro" />
+    <xacro:include filename="$(find kinova_description)/urdf/kinova_finger_set.xacro" />
+    <property name="prefix" value="j2_7n_3" />
     <property name="link_base" value="j2_7n_3_link_base" />
     <property name="link_1" value="j2_7n_3_link_1" />
@@ -111,3 +113,4 @@
         <xacro:kinova_virtual_joint joint_name="${joint_end_effector}" type="${joint_end_effector_type}" parent="${link_7}" child="${link_end_effector}" joint_axis_xyz="${joint_end_effector_axis_xyz}" joint_origin_xyz="${joint_end_effector_origin_xyz}" joint_origin_rpy="${joint_end_effector_origin_rpy}" joint_lower_limit="0" joint_upper_limit="0"/>
     </xacro:macro>
+    <xacro:kinova_3fingers link_hand="${link_7}" prefix="${prefix}"/>
 </root>

File: kinova_description/urdf/j2_7s_3.xacro (robot description, xacro)
@@ -15,5 +15,5 @@
     xmlns:xacro="http://ros.org/wiki/xacro">
     <xacro:include filename="$(find kinova_description)/urdf/kinova_common.xacro" />
-    <xacro:include filename="$(find kinova_description)/urdf/kinova_3fingers.xacro" />
+    <xacro:include filename="$(find kinova_description)/urdf/kinova_finger_set.xacro" />
     <property name="prefix" value="j2_7s_3" />
     <property name="link_base" value="j2_7s_3_link_base" />

File: kinova_description/urdf/jaco2_arm.xacro (robot description, xacro)
@@ -14,5 +14,5 @@
 	xmlns:xacro="http://ros.org/wiki/xacro">
   <xacro:include filename="$(find kinova_description)/urdf/kinova_6DOF.xacro" />
-  <xacro:include filename="$(find kinova_description)/urdf/kinova_3fingers.xacro"/>
+  <xacro:include filename="$(find kinova_description)/urdf/kinova_finger.xacro"/>
   <property name="link_base" value="jaco2_link_base" />
   <property name="link_1" value="jaco2_link_1" />

File: kinova_description/urdf/kinova_finger_set.xacro (robot description, xacro)
@@ -1,4 +1,4 @@
 <?xml version="1.0"?>
-<!-- j2_7s refers to jaco v2 7DOF spherical -->
+<!-- for 3finger_hand and 2finger_hand -->
 <root xmlns:xi="http://www.w3.org/2001/XInclude"
     xmlns:gazebo="http://playerstage.sourceforge.net/gazebo/xmlschema/#gz"
@@ -23,9 +23,9 @@
         <xacro:kinova_finger prefix="_${prefix}" finger_number="3" hand="${link_hand}" finger_origin_xyz="0.02226 -0.02707 -0.11482" finger_origin_rpy="-1.570796327 .649262481663582 -1.38614049188413"/>
     </xacro:macro>
-    <xacro:macro name="kinova_2fingers" params="link_hand">
-        <!-- finger1 Rot := Ry((1/2)*Pi) . Rx(12.1*((1/180)*Pi)+Pi) . Rz(-52.8*((1/180)*Pi)) -->
-        <xacro:kinova_finger prefix="_${prefix}" finger_number="1" hand="${link_hand}" finger_origin_xyz="0.00279 0.03126 -0.11467" finger_origin_rpy="-1.570796327 .649262481663582 1.35961148639407"/>
-        <!-- finger2 Rot := Ry((1/2)*Pi) . Rx(10.58*((1/180)*Pi)) . Rz(-52.8*((1/180)*Pi)) -->
-        <xacro:kinova_finger prefix="_${prefix}" finger_number="2" hand="${link_hand}" finger_origin_xyz="-0.02226 -0.02707 -0.11482" finger_origin_rpy="-1.570796327 .649262481663582 -1.75545216211587"/>
+    <xacro:macro name="kinova_2fingers" params="link_hand prefix">
+        <!-- finger1 Rot := Ry((1/2)*Pi) . Rx(Pi) . Rz(-52.8*((1/180)*Pi)) -->
+        <xacro:kinova_finger prefix="_${prefix}" finger_number="1" hand="${link_hand}" finger_origin_xyz="-0.0025 0.03095 -0.11482" finger_origin_rpy="-1.570796327 .649262481663582 1.57079632679490"/>
+        <!-- finger2 Rot := Ry((1/2)*Pi) . Rz(-52.8*((1/180)*Pi))  -->
+        <xacro:kinova_finger prefix="_${prefix}" finger_number="2" hand="${link_hand}" finger_origin_xyz="-0.0025 -0.03095 -0.11482" finger_origin_rpy="-1.570796327 .649262481663582 -1.57079632679490"/>
     </xacro:macro>
 </root>

File: kinova_description/urdf/m1_4n_2.xacro (robot description, xacro)
@@ -15,4 +15,6 @@
     xmlns:xacro="http://ros.org/wiki/xacro">
     <xacro:include filename="$(find kinova_description)/urdf/kinova_common.xacro" />
+    <xacro:include filename="$(find kinova_description)/urdf/kinova_finger_set.xacro" />
+    <property name="prefix" value="m1_4n_2" />
     <property name="link_base" value="m1_4n_2_link_base" />
     <property name="link_1" value="m1_4n_2_link_1" />
@@ -78,3 +80,4 @@
         <xacro:kinova_virtual_joint joint_name="${joint_end_effector}" type="${joint_end_effector_type}" parent="${link_4}" child="${link_end_effector}" joint_axis_xyz="${joint_end_effector_axis_xyz}" joint_origin_xyz="${joint_end_effector_origin_xyz}" joint_origin_rpy="${joint_end_effector_origin_rpy}" joint_lower_limit="0" joint_upper_limit="0"/>
     </xacro:macro>
+    <xacro:kinova_2fingers link_hand="${link_4}" prefix="${prefix}"/>
 </root>

File: kinova_description/urdf/m1_6n_2.xacro (robot description, xacro)
@@ -15,5 +15,5 @@
     xmlns:xacro="http://ros.org/wiki/xacro">
     <xacro:include filename="$(find kinova_description)/urdf/kinova_common.xacro" />
-    <xacro:include filename="$(find kinova_description)/urdf/kinova_3fingers.xacro" />
+    <xacro:include filename="$(find kinova_description)/urdf/kinova_finger_set.xacro" />
     <property name="prefix" value="m1_6n_2" />
     <property name="link_base" value="m1_6n_2_link_base" />
