Commit message: display j2n4, m1n4 and m1n6

File: kinova_description/urdf/j2n4a300.xacro (robot description, xacro)
@@ -1,4 +1,4 @@
 <?xml version="1.0"?>
-<!-- m1_4n refers to mico v1 6DOF non-spherical -->
+<!-- j2_4n refers to jaco v2 4DOF non-spherical -->
 <root xmlns:xi="http://www.w3.org/2001/XInclude"
     xmlns:gazebo="http://playerstage.sourceforge.net/gazebo/xmlschema/#gz"
@@ -16,5 +16,5 @@
     <xacro:include filename="$(find kinova_description)/urdf/kinova_common.xacro" />
     <xacro:include filename="$(find kinova_description)/urdf/kinova_finger_set.xacro" />
-    <property name="prefix" value="m1n4a200" />
+    <property name="prefix" value="j2n4a300" />
     <property name="link_base" value="${prefix}_link_base" />
     <property name="link_1" value="${prefix}_link_1" />
@@ -25,7 +25,7 @@
     <property name="link_base_mesh" value="base" />
     <property name="link_1_mesh" value="shoulder" />
-    <property name="link_2_mesh" value="arm_mico" />
+    <property name="link_2_mesh" value="arm" />
     <property name="link_3_mesh" value="forearm" />
-    <property name="link_4_mesh" value="hand_2finger" />
+    <property name="link_4_mesh" value="hand_3finger" />
     <property name="joint_base" value="${prefix}_joint_base" />
     <property name="joint_base_type" value="fixed" />
@@ -45,13 +45,13 @@
     <property name="joint_2_origin_xyz" value="0 0.0016 -0.11875" />
     <property name="joint_2_origin_rpy" value="${-J_PI/2} 0 ${J_PI}" />
-    <property name="joint_2_lower_limit" value="-2.35" />
-    <property name="joint_2_upper_limit" value="2.35" />
+    <property name="joint_2_lower_limit" value="-2.3" />
+    <property name="joint_2_upper_limit" value="2.3" />
     <property name="joint_3" value="${prefix}_joint_3" />
     <property name="joint_3_type" value="continuous" />
     <property name="joint_3_axis_xyz" value="0 0 1" />
-    <property name="joint_3_origin_xyz" value="0 -0.290 0" />
+    <property name="joint_3_origin_xyz" value="0 -0.410 0" />
     <property name="joint_3_origin_rpy" value="0 ${J_PI} 0" />
-    <property name="joint_3_lower_limit" value="-2.86" />
-    <property name="joint_3_upper_limit" value="2.86" />
+    <property name="joint_3_lower_limit" value="-2.8" />
+    <property name="joint_3_upper_limit" value="2.8" />
     <property name="joint_4" value="${prefix}_joint_4" />
     <property name="joint_4_type" value="continuous" />
@@ -66,5 +66,5 @@
     <property name="joint_end_effector_origin_xyz" value="0 0 -0.1600" />
     <property name="joint_end_effector_origin_rpy" value="${J_PI} 0 0" />
-    <xacro:macro name="m1n4a200" params="base_parent">
+    <xacro:macro name="j2n4a300" params="base_parent">
         <xacro:kinova_armlink link_name="${link_base}" link_mesh="${link_base_mesh}"/>
         <xacro:kinova_armjoint joint_name="${joint_base}" type="${joint_base_type}" parent="${base_parent}" child="${link_base}" joint_axis_xyz="${joint_base_axis_xyz}" joint_origin_xyz="${joint_base_origin_xyz}" joint_origin_rpy="${joint_base_origin_rpy}" joint_lower_limit="0" joint_upper_limit="0"/>
@@ -80,4 +80,4 @@
         <xacro:kinova_virtual_joint joint_name="${joint_end_effector}" type="${joint_end_effector_type}" parent="${link_4}" child="${link_end_effector}" joint_axis_xyz="${joint_end_effector_axis_xyz}" joint_origin_xyz="${joint_end_effector_origin_xyz}" joint_origin_rpy="${joint_end_effector_origin_rpy}" joint_lower_limit="0" joint_upper_limit="0"/>
     </xacro:macro>
-    <xacro:kinova_2fingers link_hand="${link_4}" prefix="${prefix}"/>
+    <xacro:kinova_3fingers link_hand="${link_4}" prefix="${prefix}"/>
 </root>

File: kinova_description/urdf/j2n4s300.xacro (robot description, xacro)
@@ -1,4 +1,4 @@
 <?xml version="1.0"?>
-<!-- m1_4n refers to mico v1 6DOF non-spherical -->
+<!-- j2_4n refers to jaco v2 4DOF non-spherical -->
 <root xmlns:xi="http://www.w3.org/2001/XInclude"
     xmlns:gazebo="http://playerstage.sourceforge.net/gazebo/xmlschema/#gz"
@@ -16,5 +16,5 @@
     <xacro:include filename="$(find kinova_description)/urdf/kinova_common.xacro" />
     <xacro:include filename="$(find kinova_description)/urdf/kinova_finger_set.xacro" />
-    <property name="prefix" value="m1n4a200" />
+    <property name="prefix" value="j2n4s300" />
     <property name="link_base" value="${prefix}_link_base" />
     <property name="link_1" value="${prefix}_link_1" />
@@ -25,7 +25,7 @@
     <property name="link_base_mesh" value="base" />
     <property name="link_1_mesh" value="shoulder" />
-    <property name="link_2_mesh" value="arm_mico" />
+    <property name="link_2_mesh" value="arm" />
     <property name="link_3_mesh" value="forearm" />
-    <property name="link_4_mesh" value="hand_2finger" />
+    <property name="link_4_mesh" value="hand_3finger" />
     <property name="joint_base" value="${prefix}_joint_base" />
     <property name="joint_base_type" value="fixed" />
@@ -45,13 +45,13 @@
     <property name="joint_2_origin_xyz" value="0 0.0016 -0.11875" />
     <property name="joint_2_origin_rpy" value="${-J_PI/2} 0 ${J_PI}" />
-    <property name="joint_2_lower_limit" value="-2.35" />
-    <property name="joint_2_upper_limit" value="2.35" />
+    <property name="joint_2_lower_limit" value="-2.3" />
+    <property name="joint_2_upper_limit" value="2.3" />
     <property name="joint_3" value="${prefix}_joint_3" />
     <property name="joint_3_type" value="continuous" />
     <property name="joint_3_axis_xyz" value="0 0 1" />
-    <property name="joint_3_origin_xyz" value="0 -0.290 0" />
+    <property name="joint_3_origin_xyz" value="0 -0.410 0" />
     <property name="joint_3_origin_rpy" value="0 ${J_PI} 0" />
-    <property name="joint_3_lower_limit" value="-2.86" />
-    <property name="joint_3_upper_limit" value="2.86" />
+    <property name="joint_3_lower_limit" value="-2.8" />
+    <property name="joint_3_upper_limit" value="2.8" />
     <property name="joint_4" value="${prefix}_joint_4" />
     <property name="joint_4_type" value="continuous" />
@@ -66,5 +66,5 @@
     <property name="joint_end_effector_origin_xyz" value="0 0 -0.1600" />
     <property name="joint_end_effector_origin_rpy" value="${J_PI} 0 0" />
-    <xacro:macro name="m1n4a200" params="base_parent">
+    <xacro:macro name="j2n4s300" params="base_parent">
         <xacro:kinova_armlink link_name="${link_base}" link_mesh="${link_base_mesh}"/>
         <xacro:kinova_armjoint joint_name="${joint_base}" type="${joint_base_type}" parent="${base_parent}" child="${link_base}" joint_axis_xyz="${joint_base_axis_xyz}" joint_origin_xyz="${joint_base_origin_xyz}" joint_origin_rpy="${joint_base_origin_rpy}" joint_lower_limit="0" joint_upper_limit="0"/>
@@ -80,4 +80,4 @@
         <xacro:kinova_virtual_joint joint_name="${joint_end_effector}" type="${joint_end_effector_type}" parent="${link_4}" child="${link_end_effector}" joint_axis_xyz="${joint_end_effector_axis_xyz}" joint_origin_xyz="${joint_end_effector_origin_xyz}" joint_origin_rpy="${joint_end_effector_origin_rpy}" joint_lower_limit="0" joint_upper_limit="0"/>
     </xacro:macro>
-    <xacro:kinova_2fingers link_hand="${link_4}" prefix="${prefix}"/>
+    <xacro:kinova_3fingers link_hand="${link_4}" prefix="${prefix}"/>
 </root>

File: kinova_description/urdf/m1n4a200_standalone.xacro (robot description, xacro)
@@ -1,4 +1,4 @@
 <?xml version="1.0"?>
-<!-- j2n4_3 refers to jaco v2 6DOF non-spherical 3fingers -->
+<!-- m1n4_2 refers to mico v1 6DOF non-spherical 2fingers -->
 <robot xmlns:xi="http://www.w3.org/2001/XInclude"
 	xmlns:gazebo="http://playerstage.sourceforge.net/gazebo/xmlschema/#gz"
@@ -13,6 +13,6 @@
     xmlns:renderable="http://playerstage.sourceforge.net/gazebo/xmlschema/#renderable"
     xmlns:physics="http://playerstage.sourceforge.net/gazebo/xmlschema/#physics"
-	xmlns:xacro="http://ros.org/wiki/xacro" name="j2n4_3">
-  <xacro:include filename="$(find kinova_description)/urdf/j2n4_3.xacro"/>
+	xmlns:xacro="http://ros.org/wiki/xacro" name="m1n4a200">
+  <xacro:include filename="$(find kinova_description)/urdf/m1n4a200.xacro"/>
   <link name="root">
     <visual>
@@ -31,4 +31,4 @@
   </link>
   <property name="robot_root" value="root" />
-  <xacro:j2n4_3  base_parent="${robot_root}"/>
+  <xacro:m1n4a200  base_parent="${robot_root}"/>
 </robot>

File: kinova_description/urdf/m1n4s200.xacro (robot description, xacro)
@@ -16,5 +16,5 @@
     <xacro:include filename="$(find kinova_description)/urdf/kinova_common.xacro" />
     <xacro:include filename="$(find kinova_description)/urdf/kinova_finger_set.xacro" />
-    <property name="prefix" value="m1n4a200" />
+    <property name="prefix" value="m1n4s200" />
     <property name="link_base" value="${prefix}_link_base" />
     <property name="link_1" value="${prefix}_link_1" />
@@ -66,5 +66,5 @@
     <property name="joint_end_effector_origin_xyz" value="0 0 -0.1600" />
     <property name="joint_end_effector_origin_rpy" value="${J_PI} 0 0" />
-    <xacro:macro name="m1n4a200" params="base_parent">
+    <xacro:macro name="m1n4s200" params="base_parent">
         <xacro:kinova_armlink link_name="${link_base}" link_mesh="${link_base_mesh}"/>
         <xacro:kinova_armjoint joint_name="${joint_base}" type="${joint_base_type}" parent="${base_parent}" child="${link_base}" joint_axis_xyz="${joint_base_axis_xyz}" joint_origin_xyz="${joint_base_origin_xyz}" joint_origin_rpy="${joint_base_origin_rpy}" joint_lower_limit="0" joint_upper_limit="0"/>

File: kinova_description/urdf/m1n6a200.xacro (robot description, xacro)
@@ -1,4 +1,4 @@
 <?xml version="1.0"?>
-<!-- m1_4n refers to mico v1 6DOF non-spherical -->
+<!-- m1_6n refers to mico v1 6DOF non-spherical -->
 <root xmlns:xi="http://www.w3.org/2001/XInclude"
     xmlns:gazebo="http://playerstage.sourceforge.net/gazebo/xmlschema/#gz"
@@ -16,5 +16,5 @@
     <xacro:include filename="$(find kinova_description)/urdf/kinova_common.xacro" />
     <xacro:include filename="$(find kinova_description)/urdf/kinova_finger_set.xacro" />
-    <property name="prefix" value="m1n4a200" />
+    <property name="prefix" value="m1n6a200" />
     <property name="link_base" value="${prefix}_link_base" />
     <property name="link_1" value="${prefix}_link_1" />
@@ -22,4 +22,6 @@
     <property name="link_3" value="${prefix}_link_3" />
     <property name="link_4" value="${prefix}_link_4" />
+    <property name="link_5" value="${prefix}_link_5" />
+    <property name="link_6" value="${prefix}_link_6" />
     <property name="link_end_effector" value="${prefix}_end_effector" />
     <property name="link_base_mesh" value="base" />
@@ -27,5 +29,7 @@
     <property name="link_2_mesh" value="arm_mico" />
     <property name="link_3_mesh" value="forearm" />
-    <property name="link_4_mesh" value="hand_2finger" />
+    <property name="link_4_mesh" value="wrist" />
+    <property name="link_5_mesh" value="wrist" />
+    <property name="link_6_mesh" value="hand_2finger" />
     <property name="joint_base" value="${prefix}_joint_base" />
     <property name="joint_base_type" value="fixed" />
@@ -61,4 +65,18 @@
     <property name="joint_4_lower_limit" value="${-2*J_PI}" />
     <property name="joint_4_upper_limit" value="${2*J_PI}" />
+    <property name="joint_5" value="${prefix}_joint_5" />
+    <property name="joint_5_type" value="continuous" />
+    <property name="joint_5_axis_xyz" value="0 0 1" />
+    <property name="joint_5_origin_xyz" value="0 -0.03703 -0.06414" />
+    <property name="joint_5_origin_rpy" value="${J_PI/3} 0 ${J_PI}" />
+    <property name="joint_5_lower_limit" value="${-2*J_PI}" />
+    <property name="joint_5_upper_limit" value="${2*J_PI}" />
+    <property name="joint_6" value="${prefix}_joint_6" />
+    <property name="joint_6_type" value="continuous" />
+    <property name="joint_6_axis_xyz" value="0 0 1" />
+    <property name="joint_6_origin_xyz" value="0 -0.03703 -0.06414" />
+    <property name="joint_6_origin_rpy" value="${J_PI/3} 0 ${J_PI}" />
+    <property name="joint_6_lower_limit" value="${-2*J_PI}" />
+    <property name="joint_6_upper_limit" value="${2*J_PI}" />
     <property name="joint_end_effector" value="${prefix}_end_effector_offset" />
     <property name="joint_end_effector_type" value="fixed" />
@@ -66,5 +84,5 @@
     <property name="joint_end_effector_origin_xyz" value="0 0 -0.1600" />
     <property name="joint_end_effector_origin_rpy" value="${J_PI} 0 0" />
-    <xacro:macro name="m1n4a200" params="base_parent">
+    <xacro:macro name="m1n6a200" params="base_parent">
         <xacro:kinova_armlink link_name="${link_base}" link_mesh="${link_base_mesh}"/>
         <xacro:kinova_armjoint joint_name="${joint_base}" type="${joint_base_type}" parent="${base_parent}" child="${link_base}" joint_axis_xyz="${joint_base_axis_xyz}" joint_origin_xyz="${joint_base_origin_xyz}" joint_origin_rpy="${joint_base_origin_rpy}" joint_lower_limit="0" joint_upper_limit="0"/>
@@ -77,7 +95,11 @@
         <xacro:kinova_armlink link_name="${link_4}" link_mesh="${link_4_mesh}"/>
         <xacro:kinova_armjoint joint_name="${joint_4}" type="${joint_4_type}" parent="${link_3}" child="${link_4}" joint_axis_xyz="${joint_4_axis_xyz}" joint_origin_xyz="${joint_4_origin_xyz}" joint_origin_rpy="${joint_4_origin_rpy}" joint_lower_limit="${joint_4_lower_limit}" joint_upper_limit="${joint_4_upper_limit}"/>
+        <xacro:kinova_armlink link_name="${link_5}" link_mesh="${link_5_mesh}"/>
+        <xacro:kinova_armjoint joint_name="${joint_5}" type="${joint_5_type}" parent="${link_4}" child="${link_5}" joint_axis_xyz="${joint_5_axis_xyz}" joint_origin_xyz="${joint_5_origin_xyz}" joint_origin_rpy="${joint_5_origin_rpy}" joint_lower_limit="${joint_5_lower_limit}" joint_upper_limit="${joint_5_upper_limit}"/>
+        <xacro:kinova_armlink link_name="${link_6}" link_mesh="${link_6_mesh}"/>
+        <xacro:kinova_armjoint joint_name="${joint_6}" type="${joint_6_type}" parent="${link_5}" child="${link_6}" joint_axis_xyz="${joint_6_axis_xyz}" joint_origin_xyz="${joint_6_origin_xyz}" joint_origin_rpy="${joint_6_origin_rpy}" joint_lower_limit="${joint_6_lower_limit}" joint_upper_limit="${joint_6_upper_limit}"/>
         <xacro:kinova_virtual_link link_name="${link_end_effector}"/>
-        <xacro:kinova_virtual_joint joint_name="${joint_end_effector}" type="${joint_end_effector_type}" parent="${link_4}" child="${link_end_effector}" joint_axis_xyz="${joint_end_effector_axis_xyz}" joint_origin_xyz="${joint_end_effector_origin_xyz}" joint_origin_rpy="${joint_end_effector_origin_rpy}" joint_lower_limit="0" joint_upper_limit="0"/>
+        <xacro:kinova_virtual_joint joint_name="${joint_end_effector}" type="${joint_end_effector_type}" parent="${link_6}" child="${link_end_effector}" joint_axis_xyz="${joint_end_effector_axis_xyz}" joint_origin_xyz="${joint_end_effector_origin_xyz}" joint_origin_rpy="${joint_end_effector_origin_rpy}" joint_lower_limit="0" joint_upper_limit="0"/>
     </xacro:macro>
-    <xacro:kinova_2fingers link_hand="${link_4}" prefix="${prefix}"/>
+    <xacro:kinova_2fingers link_hand="${link_6}" prefix="${prefix}"/>
 </root>

File: kinova_description/urdf/m1n6s200.xacro (robot description, xacro)
@@ -1,4 +1,4 @@
 <?xml version="1.0"?>
-<!-- m1_4n refers to mico v1 6DOF non-spherical -->
+<!-- m1_6n refers to mico v1 6DOF non-spherical -->
 <root xmlns:xi="http://www.w3.org/2001/XInclude"
     xmlns:gazebo="http://playerstage.sourceforge.net/gazebo/xmlschema/#gz"
@@ -16,5 +16,5 @@
     <xacro:include filename="$(find kinova_description)/urdf/kinova_common.xacro" />
     <xacro:include filename="$(find kinova_description)/urdf/kinova_finger_set.xacro" />
-    <property name="prefix" value="m1n4a200" />
+    <property name="prefix" value="m1n6s200" />
     <property name="link_base" value="${prefix}_link_base" />
     <property name="link_1" value="${prefix}_link_1" />
@@ -22,4 +22,6 @@
     <property name="link_3" value="${prefix}_link_3" />
     <property name="link_4" value="${prefix}_link_4" />
+    <property name="link_5" value="${prefix}_link_5" />
+    <property name="link_6" value="${prefix}_link_6" />
     <property name="link_end_effector" value="${prefix}_end_effector" />
     <property name="link_base_mesh" value="base" />
@@ -27,5 +29,7 @@
     <property name="link_2_mesh" value="arm_mico" />
     <property name="link_3_mesh" value="forearm" />
-    <property name="link_4_mesh" value="hand_2finger" />
+    <property name="link_4_mesh" value="wrist" />
+    <property name="link_5_mesh" value="wrist" />
+    <property name="link_6_mesh" value="hand_2finger" />
     <property name="joint_base" value="${prefix}_joint_base" />
     <property name="joint_base_type" value="fixed" />
@@ -61,4 +65,18 @@
     <property name="joint_4_lower_limit" value="${-2*J_PI}" />
     <property name="joint_4_upper_limit" value="${2*J_PI}" />
+    <property name="joint_5" value="${prefix}_joint_5" />
+    <property name="joint_5_type" value="continuous" />
+    <property name="joint_5_axis_xyz" value="0 0 1" />
+    <property name="joint_5_origin_xyz" value="0 -0.03703 -0.06414" />
+    <property name="joint_5_origin_rpy" value="${J_PI/3} 0 ${J_PI}" />
+    <property name="joint_5_lower_limit" value="${-2*J_PI}" />
+    <property name="joint_5_upper_limit" value="${2*J_PI}" />
+    <property name="joint_6" value="${prefix}_joint_6" />
+    <property name="joint_6_type" value="continuous" />
+    <property name="joint_6_axis_xyz" value="0 0 1" />
+    <property name="joint_6_origin_xyz" value="0 -0.03703 -0.06414" />
+    <property name="joint_6_origin_rpy" value="${J_PI/3} 0 ${J_PI}" />
+    <property name="joint_6_lower_limit" value="${-2*J_PI}" />
+    <property name="joint_6_upper_limit" value="${2*J_PI}" />
     <property name="joint_end_effector" value="${prefix}_end_effector_offset" />
     <property name="joint_end_effector_type" value="fixed" />
@@ -66,5 +84,5 @@
     <property name="joint_end_effector_origin_xyz" value="0 0 -0.1600" />
     <property name="joint_end_effector_origin_rpy" value="${J_PI} 0 0" />
-    <xacro:macro name="m1n4a200" params="base_parent">
+    <xacro:macro name="m1n6s200" params="base_parent">
         <xacro:kinova_armlink link_name="${link_base}" link_mesh="${link_base_mesh}"/>
         <xacro:kinova_armjoint joint_name="${joint_base}" type="${joint_base_type}" parent="${base_parent}" child="${link_base}" joint_axis_xyz="${joint_base_axis_xyz}" joint_origin_xyz="${joint_base_origin_xyz}" joint_origin_rpy="${joint_base_origin_rpy}" joint_lower_limit="0" joint_upper_limit="0"/>
@@ -77,7 +95,11 @@
         <xacro:kinova_armlink link_name="${link_4}" link_mesh="${link_4_mesh}"/>
         <xacro:kinova_armjoint joint_name="${joint_4}" type="${joint_4_type}" parent="${link_3}" child="${link_4}" joint_axis_xyz="${joint_4_axis_xyz}" joint_origin_xyz="${joint_4_origin_xyz}" joint_origin_rpy="${joint_4_origin_rpy}" joint_lower_limit="${joint_4_lower_limit}" joint_upper_limit="${joint_4_upper_limit}"/>
+        <xacro:kinova_armlink link_name="${link_5}" link_mesh="${link_5_mesh}"/>
+        <xacro:kinova_armjoint joint_name="${joint_5}" type="${joint_5_type}" parent="${link_4}" child="${link_5}" joint_axis_xyz="${joint_5_axis_xyz}" joint_origin_xyz="${joint_5_origin_xyz}" joint_origin_rpy="${joint_5_origin_rpy}" joint_lower_limit="${joint_5_lower_limit}" joint_upper_limit="${joint_5_upper_limit}"/>
+        <xacro:kinova_armlink link_name="${link_6}" link_mesh="${link_6_mesh}"/>
+        <xacro:kinova_armjoint joint_name="${joint_6}" type="${joint_6_type}" parent="${link_5}" child="${link_6}" joint_axis_xyz="${joint_6_axis_xyz}" joint_origin_xyz="${joint_6_origin_xyz}" joint_origin_rpy="${joint_6_origin_rpy}" joint_lower_limit="${joint_6_lower_limit}" joint_upper_limit="${joint_6_upper_limit}"/>
         <xacro:kinova_virtual_link link_name="${link_end_effector}"/>
-        <xacro:kinova_virtual_joint joint_name="${joint_end_effector}" type="${joint_end_effector_type}" parent="${link_4}" child="${link_end_effector}" joint_axis_xyz="${joint_end_effector_axis_xyz}" joint_origin_xyz="${joint_end_effector_origin_xyz}" joint_origin_rpy="${joint_end_effector_origin_rpy}" joint_lower_limit="0" joint_upper_limit="0"/>
+        <xacro:kinova_virtual_joint joint_name="${joint_end_effector}" type="${joint_end_effector_type}" parent="${link_6}" child="${link_end_effector}" joint_axis_xyz="${joint_end_effector_axis_xyz}" joint_origin_xyz="${joint_end_effector_origin_xyz}" joint_origin_rpy="${joint_end_effector_origin_rpy}" joint_lower_limit="0" joint_upper_limit="0"/>
     </xacro:macro>
-    <xacro:kinova_2fingers link_hand="${link_4}" prefix="${prefix}"/>
+    <xacro:kinova_2fingers link_hand="${link_6}" prefix="${prefix}"/>
 </root>
