Commit message: Correct typo for "j2s6a300" and "j2s6s300"

File: kinova_description/urdf/j2s6s300.xacro (robot description, xacro)
@@ -16,5 +16,5 @@
     <xacro:include filename="$(find kinova_description)/urdf/kinova_common.xacro" />
     <xacro:include filename="$(find kinova_description)/urdf/kinova_finger_set.xacro" />
-    <property name="prefix" value="j2s6a300" />
+    <property name="prefix" value="j2s6s300" />
     <property name="link_base" value="${prefix}_link_base" />
     <property name="link_1" value="${prefix}_link_1" />
@@ -84,5 +84,5 @@
     <property name="joint_end_effector_origin_xyz" value="0 0 -0.1600" />
     <property name="joint_end_effector_origin_rpy" value="${J_PI} 0 0" />
-    <xacro:macro name="j2s6a300" params="base_parent">
+    <xacro:macro name="j2s6s300" params="base_parent">
         <xacro:kinova_armlink link_name="${link_base}" link_mesh="${link_base_mesh}"/>
         <xacro:kinova_armjoint joint_name="${joint_base}" type="${joint_base_type}" parent="${base_parent}" child="${link_base}" joint_axis_xyz="${joint_base_axis_xyz}" joint_origin_xyz="${joint_base_origin_xyz}" joint_origin_rpy="${joint_base_origin_rpy}" joint_lower_limit="0" joint_upper_limit="0"/>
