Commit message: Test 	modified:   kinova_description/urdf/kinova_common.xacro 	modified:   kinova_description/urdf/kinova_inertial.xacro

File: kinova_description/urdf/j2n6s300_standalone.xacro (robot description, xacro)
@@ -15,19 +15,19 @@
 	xmlns:xacro="http://ros.org/wiki/xacro" name="j2n6s300">
   <xacro:include filename="$(find kinova_description)/urdf/j2n6s300.xacro"/>
-  <link name="root">
-    <visual>
-      <origin xyz="0 0 0" rpy="0 0 0" />
-      <geometry>
-        <box size = "0 0 0"/>
-      </geometry>
-    <!--<material name="Black" /> -->
-    </visual>
-    <collision>
-      <origin xyz="0 0 0" rpy="0 0 0" />
-      <geometry>
-        <box size = "0 0 0"/>
-      </geometry>
-    </collision>
-  </link>
+ <link name="root">
+   <visual>
+     <origin xyz="0 0 0" rpy="0 0 0" />
+     <geometry>
+       <box size = "0.00001 0.00001 0.00001"/>
+     </geometry>
+   <!--<material name="Black" /> -->
+   </visual>
+   <collision>
+     <origin xyz="0 0 0" rpy="0 0 0" />
+     <geometry>
+       <box size = "0.00001 0.00001 0.00001"/>
+     </geometry>
+   </collision>
+ </link>
   <!-- for gazebo -->
   <link name="world"/>

File: kinova_description/urdf/kinova_common.xacro (robot description, xacro)
@@ -54,12 +54,62 @@
      </joint>
    <xacro:unless value="${fixed}">
-     <transmission name="${joint_name}_trans">
+     <transmission name="${prefix}_joint_1_trans">
         <type>transmission_interface/SimpleTransmission</type>
-        <joint name="${joint_name}">
+        <joint name="${prefix}_joint_1">
           <hardwareInterface>EffortJointInterface</hardwareInterface>
         </joint>
-        <actuator name="${joint_name}_actuator">
+        <actuator name="${prefix}_joint_1_actuator">
           <hardwareInterface>EffortJointInterface</hardwareInterface>
         <mechanicalReduction>160</mechanicalReduction>
+        </actuator>
+     </transmission>
+     <transmission name="${prefix}_joint_2_trans">
+        <type>transmission_interface/SimpleTransmission</type>
+        <joint name="${prefix}_joint_2">
+          <hardwareInterface>EffortJointInterface</hardwareInterface>
+        </joint>
+        <actuator name="${prefix}_joint_2_actuator">
+          <hardwareInterface>EffortJointInterface</hardwareInterface>
+        <mechanicalReduction>160</mechanicalReduction>
+        </actuator>
+     </transmission>
+     <transmission name="${prefix}_joint_3_trans">
+        <type>transmission_interface/SimpleTransmission</type>
+        <joint name="${prefix}_joint_3">
+          <hardwareInterface>EffortJointInterface</hardwareInterface>
+        </joint>
+        <actuator name="${prefix}_joint_3_actuator">
+          <hardwareInterface>EffortJointInterface</hardwareInterface>
+        <mechanicalReduction>160</mechanicalReduction>
+        </actuator>
+     </transmission>
+     <transmission name="${prefix}_joint_4_trans">
+        <type>transmission_interface/SimpleTransmission</type>
+        <joint name="${prefix}_joint_4">
+          <hardwareInterface>EffortJointInterface</hardwareInterface>
+        </joint>
+        <actuator name="${prefix}_joint_4_actuator">
+          <hardwareInterface>EffortJointInterface</hardwareInterface>
+        <mechanicalReduction>110</mechanicalReduction>
+        </actuator>
+     </transmission>
+     <transmission name="${prefix}_joint_5_trans">
+        <type>transmission_interface/SimpleTransmission</type>
+        <joint name="${prefix}_joint_5">
+          <hardwareInterface>EffortJointInterface</hardwareInterface>
+        </joint>
+        <actuator name="${prefix}_joint_5_actuator">
+          <hardwareInterface>EffortJointInterface</hardwareInterface>
+        <mechanicalReduction>110</mechanicalReduction>
+        </actuator>
+     </transmission>
+     <transmission name="${prefix}_joint_6_trans">
+        <type>transmission_interface/SimpleTransmission</type>
+        <joint name="${prefix}_joint_6">
+          <hardwareInterface>EffortJointInterface</hardwareInterface>
+        </joint>
+        <actuator name="${prefix}_joint_6_actuator">
+          <hardwareInterface>EffortJointInterface</hardwareInterface>
+        <mechanicalReduction>110</mechanicalReduction>
         </actuator>
      </transmission>
@@ -70,10 +120,10 @@
             <visual>
                 <geometry>
-                    <box size = "0 0 0"/>
+                    <box size = "0.00001 0.00001 0.00001"/>
                 </geometry>
             </visual>
             <collision>
                 <geometry>
-                    <box size = "0 0 0"/>
+                    <box size = "0.00001 0.00001 0.00001"/>
                 </geometry>
             </collision>

File: kinova_description/urdf/kinova_inertial.xacro (robot description, xacro)
@@ -61,5 +61,5 @@
   <xacro:unless value="${mesh_no-1}">
     <inertial>
-        <mass value="0.7477" />
+        <mass value="0.76" />
         <origin xyz="0 -0.002 -0.0605" />
         <xacro:inertia_cylinder height="0.14"  radius = "0.04" mass="0.7477"/>
@@ -69,5 +69,5 @@
   <xacro:unless value="${mesh_no-2}">
     <inertial>
-        <mass value="0.99" />
+        <mass value="0.9907" />
         <origin xyz="0 -0.2065 -0.01" />
         <xacro:inertia_cylinder height="0.35"  radius = "0.04" mass="0.99" axis="1"/>
@@ -77,5 +77,5 @@
   <xacro:unless value="${mesh_no-3}">
     <inertial>
-        <mass value="0.6763" />
+        <mass value="0.6685" />
         <origin xyz="0 0.081 -0.0086" />
         <xacro:inertia_cylinder height="0.15"  radius = "0.03" mass="0.6763" axis="1"/>
@@ -85,5 +85,5 @@
   <xacro:unless value="${mesh_no-4}">
     <inertial>
-        <mass value="0.1785" />
+        <mass value="0.4104" />
         <origin xyz="0 -0.037 -0.0642" />
         <xacro:inertia_cylinder height="0.02"  radius = "0.04" mass="0.1785"/>
@@ -141,5 +141,5 @@
   <xacro:unless value="${mesh_no - 55}">
     <inertial>
-        <mass value="0.727" />
+        <mass value="0.8977" />
         <origin xyz="0 0 -0.06" />
         <xacro:inertia_cylinder height="0.03"  radius = "0.04" mass="0.727"/>

Commit message: This reverts commit 0f6e8b3e74b2f614a2236156b0f52c91cc4c9119.

File: kinova_description/urdf/j2n6s300_standalone.xacro (robot description, xacro)
@@ -15,19 +15,19 @@
 	xmlns:xacro="http://ros.org/wiki/xacro" name="j2n6s300">
   <xacro:include filename="$(find kinova_description)/urdf/j2n6s300.xacro"/>
- <link name="root">
-   <visual>
-     <origin xyz="0 0 0" rpy="0 0 0" />
-     <geometry>
-       <box size = "0.00001 0.00001 0.00001"/>
-     </geometry>
-   <!--<material name="Black" /> -->
-   </visual>
-   <collision>
-     <origin xyz="0 0 0" rpy="0 0 0" />
-     <geometry>
-       <box size = "0.00001 0.00001 0.00001"/>
-     </geometry>
-   </collision>
- </link>
+  <link name="root">
+    <visual>
+      <origin xyz="0 0 0" rpy="0 0 0" />
+      <geometry>
+        <box size = "0 0 0"/>
+      </geometry>
+    <!--<material name="Black" /> -->
+    </visual>
+    <collision>
+      <origin xyz="0 0 0" rpy="0 0 0" />
+      <geometry>
+        <box size = "0 0 0"/>
+      </geometry>
+    </collision>
+  </link>
   <!-- for gazebo -->
   <link name="world"/>

File: kinova_description/urdf/kinova_common.xacro (robot description, xacro)
@@ -54,62 +54,12 @@
      </joint>
    <xacro:unless value="${fixed}">
-     <transmission name="${prefix}_joint_1_trans">
+     <transmission name="${joint_name}_trans">
         <type>transmission_interface/SimpleTransmission</type>
-        <joint name="${prefix}_joint_1">
+        <joint name="${joint_name}">
           <hardwareInterface>EffortJointInterface</hardwareInterface>
         </joint>
-        <actuator name="${prefix}_joint_1_actuator">
+        <actuator name="${joint_name}_actuator">
           <hardwareInterface>EffortJointInterface</hardwareInterface>
         <mechanicalReduction>160</mechanicalReduction>
-        </actuator>
-     </transmission>
-     <transmission name="${prefix}_joint_2_trans">
-        <type>transmission_interface/SimpleTransmission</type>
-        <joint name="${prefix}_joint_2">
-          <hardwareInterface>EffortJointInterface</hardwareInterface>
-        </joint>
-        <actuator name="${prefix}_joint_2_actuator">
-          <hardwareInterface>EffortJointInterface</hardwareInterface>
-        <mechanicalReduction>160</mechanicalReduction>
-        </actuator>
-     </transmission>
-     <transmission name="${prefix}_joint_3_trans">
-        <type>transmission_interface/SimpleTransmission</type>
-        <joint name="${prefix}_joint_3">
-          <hardwareInterface>EffortJointInterface</hardwareInterface>
-        </joint>
-        <actuator name="${prefix}_joint_3_actuator">
-          <hardwareInterface>EffortJointInterface</hardwareInterface>
-        <mechanicalReduction>160</mechanicalReduction>
-        </actuator>
-     </transmission>
-     <transmission name="${prefix}_joint_4_trans">
-        <type>transmission_interface/SimpleTransmission</type>
-        <joint name="${prefix}_joint_4">
-          <hardwareInterface>EffortJointInterface</hardwareInterface>
-        </joint>
-        <actuator name="${prefix}_joint_4_actuator">
-          <hardwareInterface>EffortJointInterface</hardwareInterface>
-        <mechanicalReduction>110</mechanicalReduction>
-        </actuator>
-     </transmission>
-     <transmission name="${prefix}_joint_5_trans">
-        <type>transmission_interface/SimpleTransmission</type>
-        <joint name="${prefix}_joint_5">
-          <hardwareInterface>EffortJointInterface</hardwareInterface>
-        </joint>
-        <actuator name="${prefix}_joint_5_actuator">
-          <hardwareInterface>EffortJointInterface</hardwareInterface>
-        <mechanicalReduction>110</mechanicalReduction>
-        </actuator>
-     </transmission>
-     <transmission name="${prefix}_joint_6_trans">
-        <type>transmission_interface/SimpleTransmission</type>
-        <joint name="${prefix}_joint_6">
-          <hardwareInterface>EffortJointInterface</hardwareInterface>
-        </joint>
-        <actuator name="${prefix}_joint_6_actuator">
-          <hardwareInterface>EffortJointInterface</hardwareInterface>
-        <mechanicalReduction>110</mechanicalReduction>
         </actuator>
      </transmission>
@@ -120,10 +70,10 @@
             <visual>
                 <geometry>
-                    <box size = "0.00001 0.00001 0.00001"/>
+                    <box size = "0 0 0"/>
                 </geometry>
             </visual>
             <collision>
                 <geometry>
-                    <box size = "0.00001 0.00001 0.00001"/>
+                    <box size = "0 0 0"/>
                 </geometry>
             </collision>

File: kinova_description/urdf/kinova_inertial.xacro (robot description, xacro)
@@ -61,5 +61,5 @@
   <xacro:unless value="${mesh_no-1}">
     <inertial>
-        <mass value="0.76" />
+        <mass value="0.7477" />
         <origin xyz="0 -0.002 -0.0605" />
         <xacro:inertia_cylinder height="0.14"  radius = "0.04" mass="0.7477"/>
@@ -69,5 +69,5 @@
   <xacro:unless value="${mesh_no-2}">
     <inertial>
-        <mass value="0.9907" />
+        <mass value="0.99" />
         <origin xyz="0 -0.2065 -0.01" />
         <xacro:inertia_cylinder height="0.35"  radius = "0.04" mass="0.99" axis="1"/>
@@ -77,5 +77,5 @@
   <xacro:unless value="${mesh_no-3}">
     <inertial>
-        <mass value="0.6685" />
+        <mass value="0.6763" />
         <origin xyz="0 0.081 -0.0086" />
         <xacro:inertia_cylinder height="0.15"  radius = "0.03" mass="0.6763" axis="1"/>
@@ -85,5 +85,5 @@
   <xacro:unless value="${mesh_no-4}">
     <inertial>
-        <mass value="0.4104" />
+        <mass value="0.1785" />
         <origin xyz="0 -0.037 -0.0642" />
         <xacro:inertia_cylinder height="0.02"  radius = "0.04" mass="0.1785"/>
@@ -141,5 +141,5 @@
   <xacro:unless value="${mesh_no - 55}">
     <inertial>
-        <mass value="0.8977" />
+        <mass value="0.727" />
         <origin xyz="0 0 -0.06" />
         <xacro:inertia_cylinder height="0.03"  radius = "0.04" mass="0.727"/>

Commit message: fix boost::shared_ptr error and gazebo7

File: kinova_description/urdf/j2n6s300_standalone.xacro (robot description, xacro)
@@ -19,5 +19,5 @@
       <origin xyz="0 0 0" rpy="0 0 0" />
       <geometry>
-        <box size = "0 0 0"/>
+        <box size = "0.001 0.001 0.001"/>
       </geometry>
     <!--<material name="Black" /> -->
@@ -26,5 +26,5 @@
       <origin xyz="0 0 0" rpy="0 0 0" />
       <geometry>
-        <box size = "0 0 0"/>
+        <box size = "0.001 0.001 0.001"/>
       </geometry>
     </collision>

File: kinova_description/urdf/kinova_common.xacro (robot description, xacro)
@@ -70,10 +70,10 @@
             <visual>
                 <geometry>
-                    <box size = "0 0 0"/>
+                    <box size = "0.001 0.001 0.001"/>
                 </geometry>
             </visual>
             <collision>
                 <geometry>
-                    <box size = "0 0 0"/>
+                    <box size = "0.001 0.001 0.001"/>
                 </geometry>
             </collision>
