Commit message: updates velocities and efforts

File: kinova_description/urdf/j2s6s200_standalone.urdf (robot description, URDF)
Before this commit: robot j2s6s200, 13 links, 12 joints
Joints:
- joint j2s6s200_joint_1: limit lower=-6.28318530718 upper=6.28318530718 effort=30.5 velocity=2 -> lower=-6.28318530718 upper=6.28318530718 effort=30.5 velocity=0.984365697
- joint j2s6s200_joint_2: limit lower=0.820304748437 upper=5.46288055874 effort=30.5 velocity=2 -> lower=0.820304748437 upper=5.46288055874 effort=30.5 velocity=0.984365697
- joint j2s6s200_joint_3: limit lower=0.331612557879 upper=5.9515727493 effort=30.5 velocity=2 -> lower=0.331612557879 upper=5.9515727493 effort=30.5 velocity=0.984365697
- joint j2s6s200_joint_4: limit lower=-6.28318530718 upper=6.28318530718 effort=6.8 velocity=2 -> lower=-6.28318530718 upper=6.28318530718 effort=6.8 velocity=1.570796326
- joint j2s6s200_joint_5: limit lower=0.523598775598 upper=5.75958653158 effort=6.8 velocity=2 -> lower=0.523598775598 upper=5.75958653158 effort=6.8 velocity=1.570796326
- joint j2s6s200_joint_6: limit lower=-6.28318530718 upper=6.28318530718 effort=6.8 velocity=2 -> lower=-6.28318530718 upper=6.28318530718 effort=6.8 velocity=1.570796326
- joint j2s6s200_joint_finger_1: limit lower=0 upper=2 effort=2000 velocity=1 -> lower=0 upper=2 effort=25 velocity=1
- joint j2s6s200_joint_finger_2: limit lower=0 upper=2 effort=2000 velocity=1 -> lower=0 upper=2 effort=25 velocity=1
