Commit message: Added world frame to urdf for gazebo
Added world frame to urdf for gazebo

File: kinova_description/urdf/j2n4s300_standalone.xacro (robot description, xacro)
@@ -30,4 +30,11 @@
     </collision>
   </link>
+  <!-- for gazebo -->
+  <link name="world"/>
+  <joint name="connect_root_and_world" type="fixed">
+    <child link="root" />
+    <parent link="world" />
+    <origin xyz="0 0 0" rpy="0 0 0" />
+  </joint>
   <property name="robot_root" value="root" />
   <xacro:j2n4s300  base_parent="${robot_root}"/>

File: kinova_description/urdf/j2n7s300_standalone.xacro (robot description, xacro)
@@ -30,4 +30,11 @@
     </collision>
   </link>
+  <!-- for gazebo -->
+  <link name="world"/>
+  <joint name="connect_root_and_world" type="fixed">
+    <child link="root" />
+    <parent link="world" />
+    <origin xyz="0 0 0" rpy="0 0 0" />
+  </joint>
   <property name="robot_root" value="root" />
   <xacro:j2n7s300  base_parent="${robot_root}"/>

File: kinova_description/urdf/j2s6s300_standalone.xacro (robot description, xacro)
@@ -30,4 +30,11 @@
     </collision>
   </link>
+  <!-- for gazebo -->
+  <link name="world"/>
+  <joint name="connect_root_and_world" type="fixed">
+    <child link="root" />
+    <parent link="world" />
+    <origin xyz="0 0 0" rpy="0 0 0" />
+  </joint>
   <property name="robot_root" value="root" />
   <xacro:j2s6s300  base_parent="${robot_root}"/>

File: kinova_description/urdf/m1n4s200_standalone.xacro (robot description, xacro)
@@ -30,4 +30,11 @@
     </collision>
   </link>
+  <!-- for gazebo -->
+  <link name="world"/>
+  <joint name="connect_root_and_world" type="fixed">
+    <child link="root" />
+    <parent link="world" />
+    <origin xyz="0 0 0" rpy="0 0 0" />
+  </joint>
   <property name="robot_root" value="root" />
   <xacro:m1n4s200  base_parent="${robot_root}"/>

File: kinova_description/urdf/m1n6s300_standalone.xacro (robot description, xacro)
@@ -30,4 +30,11 @@
     </collision>
   </link>
+  <!-- for gazebo -->
+  <link name="world"/>
+  <joint name="connect_root_and_world" type="fixed">
+    <child link="root" />
+    <parent link="world" />
+    <origin xyz="0 0 0" rpy="0 0 0" />
+  </joint>
   <property name="robot_root" value="root" />
   <xacro:m1n6s300  base_parent="${robot_root}"/>
