Commit message: remove visual from root frame

File: kinova_description/urdf/j2n4s300_standalone.xacro (robot description, xacro)
@@ -15,19 +15,5 @@
 	xmlns:xacro="http://ros.org/wiki/xacro" name="j2n4s300">
   <xacro:include filename="$(find kinova_description)/urdf/j2n4s300.xacro"/>
-  <link name="root">
-    <visual>
-      <origin xyz="0 0 0" rpy="0 0 0" />
-      <geometry>
-        <box size = "0 0 0"/>
-      </geometry>
-    <!--<material name="Black" /> -->
-    </visual>
-    <collision>
-      <origin xyz="0 0 0" rpy="0 0 0" />
-      <geometry>
-        <box size = "0 0 0"/>
-      </geometry>
-    </collision>
-  </link>
+  <link name="root" />
   <!-- for gazebo -->
   <link name="world"/>

File: kinova_description/urdf/j2n6s200_standalone.xacro (robot description, xacro)
@@ -15,19 +15,5 @@
 	xmlns:xacro="http://ros.org/wiki/xacro" name="j2n6s200">
   <xacro:include filename="$(find kinova_description)/urdf/j2n6s200.xacro"/>
-  <link name="root">
-    <visual>
-      <origin xyz="0 0 0" rpy="0 0 0" />
-      <geometry>
-        <box size = "0 0 0"/>
-      </geometry>
-    <!--<material name="Black" /> -->
-    </visual>
-    <collision>
-      <origin xyz="0 0 0" rpy="0 0 0" />
-      <geometry>
-        <box size = "0 0 0"/>
-      </geometry>
-    </collision>
-  </link>
+  <link name="root"/>
   <!-- for gazebo -->
   <link name="world"/>

File: kinova_description/urdf/j2n6s300_standalone.xacro (robot description, xacro)
@@ -15,19 +15,5 @@
 	xmlns:xacro="http://ros.org/wiki/xacro" name="j2n6s300">
   <xacro:include filename="$(find kinova_description)/urdf/j2n6s300.xacro"/>
-  <link name="root">
-    <visual>
-      <origin xyz="0 0 0" rpy="0 0 0" />
-      <geometry>
-        <box size = "0 0 0"/>
-      </geometry>
-    <!--<material name="Black" /> -->
-    </visual>
-    <collision>
-      <origin xyz="0 0 0" rpy="0 0 0" />
-      <geometry>
-        <box size = "0 0 0"/>
-      </geometry>
-    </collision>
-  </link>
+  <link name="root"/>
   <!-- for gazebo -->
   <link name="world"/>

File: kinova_description/urdf/j2n7s300_standalone.xacro (robot description, xacro)
@@ -15,19 +15,5 @@
 	xmlns:xacro="http://ros.org/wiki/xacro" name="j2n7s300">
   <xacro:include filename="$(find kinova_description)/urdf/j2n7s300.xacro"/>
-  <link name="root">
-    <visual>
-      <origin xyz="0 0 0" rpy="0 0 0" />
-      <geometry>
-        <box size = "0 0 0"/>
-      </geometry>
-    <!--<material name="Black" /> -->
-    </visual>
-    <collision>
-      <origin xyz="0 0 0" rpy="0 0 0" />
-      <geometry>
-        <box size = "0 0 0"/>
-      </geometry>
-    </collision>
-  </link>
+  <link name="root"/>
   <!-- for gazebo -->
   <link name="world"/>

File: kinova_description/urdf/j2s6s300_standalone.xacro (robot description, xacro)
@@ -15,19 +15,5 @@
 	xmlns:xacro="http://ros.org/wiki/xacro" name="j2s6s300">
   <xacro:include filename="$(find kinova_description)/urdf/j2s6s300.xacro"/>
-  <link name="root">
-    <visual>
-      <origin xyz="0 0 0" rpy="0 0 0" />
-      <geometry>
-        <box size = "0 0 0"/>
-      </geometry>
-    <!--<material name="Black" /> -->
-    </visual>
-    <collision>
-      <origin xyz="0 0 0" rpy="0 0 0" />
-      <geometry>
-        <box size = "0 0 0"/>
-      </geometry>
-    </collision>
-  </link>
+  <link name="root"/>
   <!-- for gazebo -->
   <link name="world"/>

File: kinova_description/urdf/j2s7s300_standalone.xacro (robot description, xacro)
@@ -15,19 +15,5 @@
 	xmlns:xacro="http://ros.org/wiki/xacro" name="j2s7s300">
   <xacro:include filename="$(find kinova_description)/urdf/j2s7s300.xacro"/>
-  <link name="root">
-    <visual>
-      <origin xyz="0 0 0" rpy="0 0 0" />
-      <geometry>
-        <box size = "0 0 0"/>
-      </geometry>
-    <!--<material name="Black" /> -->
-    </visual>
-    <collision>
-      <origin xyz="0 0 0" rpy="0 0 0" />
-      <geometry>
-        <box size = "0 0 0"/>
-      </geometry>
-    </collision>
-  </link>
+  <link name="root"/>
   <!-- for gazebo -->
   <link name="world"/>

File: kinova_description/urdf/m1n4s200_standalone.xacro (robot description, xacro)
@@ -15,19 +15,5 @@
 	xmlns:xacro="http://ros.org/wiki/xacro" name="m1n4s200">
   <xacro:include filename="$(find kinova_description)/urdf/m1n4s200.xacro"/>
-  <link name="root">
-    <visual>
-      <origin xyz="0 0 0" rpy="0 0 0" />
-      <geometry>
-        <box size = "0 0 0"/>
-      </geometry>
-    <!--<material name="Black" /> -->
-    </visual>
-    <collision>
-      <origin xyz="0 0 0" rpy="0 0 0" />
-      <geometry>
-        <box size = "0 0 0"/>
-      </geometry>
-    </collision>
-  </link>
+  <link name="root"/>
   <!-- for gazebo -->
   <link name="world"/>

File: kinova_description/urdf/m1n6s200_standalone.xacro (robot description, xacro)
@@ -15,19 +15,5 @@
 	xmlns:xacro="http://ros.org/wiki/xacro" name="m1n6s200">
   <xacro:include filename="$(find kinova_description)/urdf/m1n6s200.xacro"/>
-  <link name="root">
-    <visual>
-      <origin xyz="0 0 0" rpy="0 0 0" />
-      <geometry>
-        <box size = "0 0 0"/>
-      </geometry>
-    <!--<material name="Black" /> -->
-    </visual>
-    <collision>
-      <origin xyz="0 0 0" rpy="0 0 0" />
-      <geometry>
-        <box size = "0 0 0"/>
-      </geometry>
-    </collision>
-  </link>
+  <link name="root"/>
   <!-- for gazebo -->
   <link name="world"/>

File: kinova_description/urdf/m1n6s300_standalone.xacro (robot description, xacro)
@@ -15,19 +15,5 @@
 	xmlns:xacro="http://ros.org/wiki/xacro" name="m1n6s300">
   <xacro:include filename="$(find kinova_description)/urdf/m1n6s300.xacro"/>
-  <link name="root">
-    <visual>
-      <origin xyz="0 0 0" rpy="0 0 0" />
-      <geometry>
-        <box size = "0 0 0"/>
-      </geometry>
-    <!--<material name="Black" /> -->
-    </visual>
-    <collision>
-      <origin xyz="0 0 0" rpy="0 0 0" />
-      <geometry>
-        <box size = "0 0 0"/>
-      </geometry>
-    </collision>
-  </link>
+  <link name="root"/>
   <!-- for gazebo -->
   <link name="world"/>

Commit message: remove world frame

File: kinova_description/urdf/j2n4s300_standalone.xacro (robot description, xacro)
@@ -16,11 +16,4 @@
   <xacro:include filename="$(find kinova_description)/urdf/j2n4s300.xacro"/>
   <link name="root" />
-  <!-- for gazebo -->
-  <link name="world"/>
-  <joint name="connect_root_and_world" type="fixed">
-    <child link="root" />
-    <parent link="world" />
-    <origin xyz="0 0 0" rpy="0 0 0" />
-  </joint>
   <xacro:property name="robot_root" value="root" />
   <xacro:j2n4s300  base_parent="${robot_root}"/>

File: kinova_description/urdf/j2n6s200_standalone.xacro (robot description, xacro)
@@ -16,11 +16,4 @@
   <xacro:include filename="$(find kinova_description)/urdf/j2n6s200.xacro"/>
   <link name="root"/>
-  <!-- for gazebo -->
-  <link name="world"/>
-  <joint name="connect_root_and_world" type="fixed">
-    <child link="root" />
-    <parent link="world" />
-    <origin xyz="0 0 0" rpy="0 0 0" />
-  </joint>
   <xacro:property name="robot_root" value="root" />
   <xacro:j2n6s200  base_parent="${robot_root}"/>

File: kinova_description/urdf/j2n6s300_standalone.xacro (robot description, xacro)
@@ -16,11 +16,4 @@
   <xacro:include filename="$(find kinova_description)/urdf/j2n6s300.xacro"/>
   <link name="root"/>
-  <!-- for gazebo -->
-  <link name="world"/>
-  <joint name="connect_root_and_world" type="fixed">
-    <child link="root" />
-    <parent link="world" />
-    <origin xyz="0 0 0" rpy="0 0 0" />
-  </joint>
   <xacro:property name="robot_root" value="root" />
   <xacro:j2n6s300  base_parent="${robot_root}"/>

File: kinova_description/urdf/j2n7s300_standalone.xacro (robot description, xacro)
@@ -16,11 +16,4 @@
   <xacro:include filename="$(find kinova_description)/urdf/j2n7s300.xacro"/>
   <link name="root"/>
-  <!-- for gazebo -->
-  <link name="world"/>
-  <joint name="connect_root_and_world" type="fixed">
-    <child link="root" />
-    <parent link="world" />
-    <origin xyz="0 0 0" rpy="0 0 0" />
-  </joint>
   <xacro:property name="robot_root" value="root" />
   <xacro:j2n7s300  base_parent="${robot_root}"/>

File: kinova_description/urdf/j2s6s300_standalone.xacro (robot description, xacro)
@@ -16,11 +16,4 @@
   <xacro:include filename="$(find kinova_description)/urdf/j2s6s300.xacro"/>
   <link name="root"/>
-  <!-- for gazebo -->
-  <link name="world"/>
-  <joint name="connect_root_and_world" type="fixed">
-    <child link="root" />
-    <parent link="world" />
-    <origin xyz="0 0 0" rpy="0 0 0" />
-  </joint>
   <xacro:property name="robot_root" value="root" />
   <xacro:j2s6s300  base_parent="${robot_root}"/>

File: kinova_description/urdf/j2s7s300_standalone.xacro (robot description, xacro)
@@ -16,11 +16,4 @@
   <xacro:include filename="$(find kinova_description)/urdf/j2s7s300.xacro"/>
   <link name="root"/>
-  <!-- for gazebo -->
-  <link name="world"/>
-  <joint name="connect_root_and_world" type="fixed">
-    <child link="root" />
-    <parent link="world" />
-    <origin xyz="0 0 0" rpy="0 0 0" />
-  </joint>
   <xacro:property name="robot_root" value="root" />
   <xacro:j2s7s300  base_parent="${robot_root}"/>

File: kinova_description/urdf/m1n4s200_standalone.xacro (robot description, xacro)
@@ -16,11 +16,4 @@
   <xacro:include filename="$(find kinova_description)/urdf/m1n4s200.xacro"/>
   <link name="root"/>
-  <!-- for gazebo -->
-  <link name="world"/>
-  <joint name="connect_root_and_world" type="fixed">
-    <child link="root" />
-    <parent link="world" />
-    <origin xyz="0 0 0" rpy="0 0 0" />
-  </joint>
   <xacro:property name="robot_root" value="root" />
   <xacro:m1n4s200  base_parent="${robot_root}"/>

File: kinova_description/urdf/m1n6s200_standalone.xacro (robot description, xacro)
@@ -16,11 +16,4 @@
   <xacro:include filename="$(find kinova_description)/urdf/m1n6s200.xacro"/>
   <link name="root"/>
-  <!-- for gazebo -->
-  <link name="world"/>
-  <joint name="connect_root_and_world" type="fixed">
-    <child link="root" />
-    <parent link="world" />
-    <origin xyz="0 0 0" rpy="0 0 0" />
-  </joint>
   <xacro:property name="robot_root" value="root" />
   <xacro:m1n6s200  base_parent="${robot_root}"/>

File: kinova_description/urdf/m1n6s300_standalone.xacro (robot description, xacro)
@@ -16,11 +16,4 @@
   <xacro:include filename="$(find kinova_description)/urdf/m1n6s300.xacro"/>
   <link name="root"/>
-  <!-- for gazebo -->
-  <link name="world"/>
-  <joint name="connect_root_and_world" type="fixed">
-    <child link="root" />
-    <parent link="world" />
-    <origin xyz="0 0 0" rpy="0 0 0" />
-  </joint>
   <xacro:property name="robot_root" value="root" />
   <xacro:m1n6s300  base_parent="${robot_root}"/>

Commit message: Revert "remove world frame"
This reverts commit 4727ab980221736fe48542416178b4f9bfa4ff47.

File: kinova_description/urdf/j2n4s300_standalone.xacro (robot description, xacro)
@@ -16,4 +16,11 @@
   <xacro:include filename="$(find kinova_description)/urdf/j2n4s300.xacro"/>
   <link name="root" />
+  <!-- for gazebo -->
+  <link name="world"/>
+  <joint name="connect_root_and_world" type="fixed">
+    <child link="root" />
+    <parent link="world" />
+    <origin xyz="0 0 0" rpy="0 0 0" />
+  </joint>
   <xacro:property name="robot_root" value="root" />
   <xacro:j2n4s300  base_parent="${robot_root}"/>

File: kinova_description/urdf/j2n6s200_standalone.xacro (robot description, xacro)
@@ -16,4 +16,11 @@
   <xacro:include filename="$(find kinova_description)/urdf/j2n6s200.xacro"/>
   <link name="root"/>
+  <!-- for gazebo -->
+  <link name="world"/>
+  <joint name="connect_root_and_world" type="fixed">
+    <child link="root" />
+    <parent link="world" />
+    <origin xyz="0 0 0" rpy="0 0 0" />
+  </joint>
   <xacro:property name="robot_root" value="root" />
   <xacro:j2n6s200  base_parent="${robot_root}"/>

File: kinova_description/urdf/j2n6s300_standalone.xacro (robot description, xacro)
@@ -16,4 +16,11 @@
   <xacro:include filename="$(find kinova_description)/urdf/j2n6s300.xacro"/>
   <link name="root"/>
+  <!-- for gazebo -->
+  <link name="world"/>
+  <joint name="connect_root_and_world" type="fixed">
+    <child link="root" />
+    <parent link="world" />
+    <origin xyz="0 0 0" rpy="0 0 0" />
+  </joint>
   <xacro:property name="robot_root" value="root" />
   <xacro:j2n6s300  base_parent="${robot_root}"/>

File: kinova_description/urdf/j2n7s300_standalone.xacro (robot description, xacro)
@@ -16,4 +16,11 @@
   <xacro:include filename="$(find kinova_description)/urdf/j2n7s300.xacro"/>
   <link name="root"/>
+  <!-- for gazebo -->
+  <link name="world"/>
+  <joint name="connect_root_and_world" type="fixed">
+    <child link="root" />
+    <parent link="world" />
+    <origin xyz="0 0 0" rpy="0 0 0" />
+  </joint>
   <xacro:property name="robot_root" value="root" />
   <xacro:j2n7s300  base_parent="${robot_root}"/>

File: kinova_description/urdf/j2s6s300_standalone.xacro (robot description, xacro)
@@ -16,4 +16,11 @@
   <xacro:include filename="$(find kinova_description)/urdf/j2s6s300.xacro"/>
   <link name="root"/>
+  <!-- for gazebo -->
+  <link name="world"/>
+  <joint name="connect_root_and_world" type="fixed">
+    <child link="root" />
+    <parent link="world" />
+    <origin xyz="0 0 0" rpy="0 0 0" />
+  </joint>
   <xacro:property name="robot_root" value="root" />
   <xacro:j2s6s300  base_parent="${robot_root}"/>

File: kinova_description/urdf/j2s7s300_standalone.xacro (robot description, xacro)
@@ -16,4 +16,11 @@
   <xacro:include filename="$(find kinova_description)/urdf/j2s7s300.xacro"/>
   <link name="root"/>
+  <!-- for gazebo -->
+  <link name="world"/>
+  <joint name="connect_root_and_world" type="fixed">
+    <child link="root" />
+    <parent link="world" />
+    <origin xyz="0 0 0" rpy="0 0 0" />
+  </joint>
   <xacro:property name="robot_root" value="root" />
   <xacro:j2s7s300  base_parent="${robot_root}"/>

File: kinova_description/urdf/m1n4s200_standalone.xacro (robot description, xacro)
@@ -16,4 +16,11 @@
   <xacro:include filename="$(find kinova_description)/urdf/m1n4s200.xacro"/>
   <link name="root"/>
+  <!-- for gazebo -->
+  <link name="world"/>
+  <joint name="connect_root_and_world" type="fixed">
+    <child link="root" />
+    <parent link="world" />
+    <origin xyz="0 0 0" rpy="0 0 0" />
+  </joint>
   <xacro:property name="robot_root" value="root" />
   <xacro:m1n4s200  base_parent="${robot_root}"/>

File: kinova_description/urdf/m1n6s200_standalone.xacro (robot description, xacro)
@@ -16,4 +16,11 @@
   <xacro:include filename="$(find kinova_description)/urdf/m1n6s200.xacro"/>
   <link name="root"/>
+  <!-- for gazebo -->
+  <link name="world"/>
+  <joint name="connect_root_and_world" type="fixed">
+    <child link="root" />
+    <parent link="world" />
+    <origin xyz="0 0 0" rpy="0 0 0" />
+  </joint>
   <xacro:property name="robot_root" value="root" />
   <xacro:m1n6s200  base_parent="${robot_root}"/>

File: kinova_description/urdf/m1n6s300_standalone.xacro (robot description, xacro)
@@ -16,4 +16,11 @@
   <xacro:include filename="$(find kinova_description)/urdf/m1n6s300.xacro"/>
   <link name="root"/>
+  <!-- for gazebo -->
+  <link name="world"/>
+  <joint name="connect_root_and_world" type="fixed">
+    <child link="root" />
+    <parent link="world" />
+    <origin xyz="0 0 0" rpy="0 0 0" />
+  </joint>
   <xacro:property name="robot_root" value="root" />
   <xacro:m1n6s300  base_parent="${robot_root}"/>
