Commit message: Added the realistic velocity limits for joints based on data sheet

File: kinova_description/urdf/j2n4s300.xacro (robot description, xacro)
@@ -46,5 +46,5 @@
     <xacro:property name="joint_1_lower_limit" value="${-2*J_PI}" />
     <xacro:property name="joint_1_upper_limit" value="${2*J_PI}" />
-    <xacro:property name="joint_1_velocity_limit" value="2" />
+    <xacro:property name="joint_1_velocity_limit" value="${36*J_PI/180}" />
     <xacro:property name="joint_1_torque_limit" value="1000" />
     <xacro:property name="joint_2" value="joint_2" />
@@ -55,5 +55,5 @@
     <xacro:property name="joint_2_lower_limit" value="${47/180*J_PI}" />
     <xacro:property name="joint_2_upper_limit" value="${313/180*J_PI}" />
-    <xacro:property name="joint_2_velocity_limit" value="2" />
+    <xacro:property name="joint_2_velocity_limit" value="${36*J_PI/180}" />
     <xacro:property name="joint_2_torque_limit" value="1000" />
     <xacro:property name="joint_3" value="joint_3" />
@@ -64,5 +64,5 @@
     <xacro:property name="joint_3_lower_limit" value="${19/180*J_PI}" />
     <xacro:property name="joint_3_upper_limit" value="${341/180*J_PI}" />
-    <xacro:property name="joint_3_velocity_limit" value="2" />
+    <xacro:property name="joint_3_velocity_limit" value="${36*J_PI/180}" />
     <xacro:property name="joint_3_torque_limit" value="1000" />
     <xacro:property name="joint_4" value="joint_4" />
@@ -73,5 +73,5 @@
     <xacro:property name="joint_4_lower_limit" value="${-2*J_PI}" />
     <xacro:property name="joint_4_upper_limit" value="${2*J_PI}" />
-    <xacro:property name="joint_4_velocity_limit" value="2" />
+    <xacro:property name="joint_4_velocity_limit" value="${48*J_PI/180}" />
     <xacro:property name="joint_4_torque_limit" value="1000" />
     <xacro:property name="joint_end_effector" value="end_effector_offset" />

File: kinova_description/urdf/j2n6s200.xacro (robot description, xacro)
@@ -50,5 +50,5 @@
     <xacro:property name="joint_1_lower_limit" value="${-2*J_PI}" />
     <xacro:property name="joint_1_upper_limit" value="${2*J_PI}" />
-    <xacro:property name="joint_1_velocity_limit" value="2" />
+    <xacro:property name="joint_1_velocity_limit" value="${36*J_PI/180}" />
     <xacro:property name="joint_1_torque_limit" value="1000" />
     <xacro:property name="joint_2" value="joint_2" />
@@ -59,5 +59,5 @@
     <xacro:property name="joint_2_lower_limit" value="${47/180*J_PI}" />
     <xacro:property name="joint_2_upper_limit" value="${313/180*J_PI}" />
-    <xacro:property name="joint_2_velocity_limit" value="2" />
+    <xacro:property name="joint_2_velocity_limit" value="${36*J_PI/180}" />
     <xacro:property name="joint_2_torque_limit" value="1000" />
     <xacro:property name="joint_3" value="joint_3" />
@@ -68,5 +68,5 @@
     <xacro:property name="joint_3_lower_limit" value="${19/180*J_PI}" />
     <xacro:property name="joint_3_upper_limit" value="${341/180*J_PI}" />
-    <xacro:property name="joint_3_velocity_limit" value="2" />
+    <xacro:property name="joint_3_velocity_limit" value="${36*J_PI/180}" />
     <xacro:property name="joint_3_torque_limit" value="1000" />
     <xacro:property name="joint_4" value="joint_4" />
@@ -77,5 +77,5 @@
     <xacro:property name="joint_4_lower_limit" value="${-2*J_PI}" />
     <xacro:property name="joint_4_upper_limit" value="${2*J_PI}" />
-    <xacro:property name="joint_4_velocity_limit" value="2" />
+    <xacro:property name="joint_4_velocity_limit" value="${48*J_PI/180}" />
     <xacro:property name="joint_4_torque_limit" value="1000" />
     <xacro:property name="joint_5" value="joint_5" />
@@ -86,5 +86,5 @@
     <xacro:property name="joint_5_lower_limit" value="${-2*J_PI}" />
     <xacro:property name="joint_5_upper_limit" value="${2*J_PI}" />
-    <xacro:property name="joint_5_velocity_limit" value="2" />
+    <xacro:property name="joint_5_velocity_limit" value="${48*J_PI/180}" />
     <xacro:property name="joint_5_torque_limit" value="1000" />
     <xacro:property name="joint_6" value="joint_6" />
@@ -95,5 +95,5 @@
     <xacro:property name="joint_6_lower_limit" value="${-2*J_PI}" />
     <xacro:property name="joint_6_upper_limit" value="${2*J_PI}" />
-    <xacro:property name="joint_6_velocity_limit" value="2" />
+    <xacro:property name="joint_6_velocity_limit" value="${48*J_PI/180}" />
     <xacro:property name="joint_6_torque_limit" value="1000" />
     <xacro:property name="joint_end_effector" value="end_effector_offset" />

File: kinova_description/urdf/j2n6s300.xacro (robot description, xacro)
@@ -50,5 +50,5 @@
     <xacro:property name="joint_1_lower_limit" value="${-2*J_PI}" />
     <xacro:property name="joint_1_upper_limit" value="${2*J_PI}" />
-    <xacro:property name="joint_1_velocity_limit" value="2" />
+    <xacro:property name="joint_1_velocity_limit" value="${36*J_PI/180}" />
     <xacro:property name="joint_1_torque_limit" value="1000" />
     <xacro:property name="joint_2" value="joint_2" />
@@ -59,5 +59,5 @@
     <xacro:property name="joint_2_lower_limit" value="${47/180*J_PI}" />
     <xacro:property name="joint_2_upper_limit" value="${313/180*J_PI}" />
-    <xacro:property name="joint_2_velocity_limit" value="2" />
+    <xacro:property name="joint_2_velocity_limit" value="${36*J_PI/180}" />
     <xacro:property name="joint_2_torque_limit" value="1000" />
     <xacro:property name="joint_3" value="joint_3" />
@@ -68,5 +68,5 @@
     <xacro:property name="joint_3_lower_limit" value="${19/180*J_PI}" />
     <xacro:property name="joint_3_upper_limit" value="${341/180*J_PI}" />
-    <xacro:property name="joint_3_velocity_limit" value="2" />
+    <xacro:property name="joint_3_velocity_limit" value="${36*J_PI/180}" />
     <xacro:property name="joint_3_torque_limit" value="1000" />
     <xacro:property name="joint_4" value="joint_4" />
@@ -77,5 +77,5 @@
     <xacro:property name="joint_4_lower_limit" value="${-2*J_PI}" />
     <xacro:property name="joint_4_upper_limit" value="${2*J_PI}" />
-    <xacro:property name="joint_4_velocity_limit" value="2" />
+    <xacro:property name="joint_4_velocity_limit" value="${48*J_PI/180}" />
     <xacro:property name="joint_4_torque_limit" value="1000" />
     <xacro:property name="joint_5" value="joint_5" />
@@ -86,5 +86,5 @@
     <xacro:property name="joint_5_lower_limit" value="${-2*J_PI}" />
     <xacro:property name="joint_5_upper_limit" value="${2*J_PI}" />
-    <xacro:property name="joint_5_velocity_limit" value="2" />
+    <xacro:property name="joint_5_velocity_limit" value="${48*J_PI/180}" />
     <xacro:property name="joint_5_torque_limit" value="1000" />
     <xacro:property name="joint_6" value="joint_6" />
@@ -95,5 +95,5 @@
     <xacro:property name="joint_6_lower_limit" value="${-2*J_PI}" />
     <xacro:property name="joint_6_upper_limit" value="${2*J_PI}" />
-    <xacro:property name="joint_6_velocity_limit" value="2" />
+    <xacro:property name="joint_6_velocity_limit" value="${48*J_PI/180}" />
     <xacro:property name="joint_6_torque_limit" value="1000" />
     <xacro:property name="joint_end_effector" value="end_effector_offset" />

File: kinova_description/urdf/j2s6s300.xacro (robot description, xacro)
@@ -50,5 +50,5 @@
     <xacro:property name="joint_1_lower_limit" value="${-2*J_PI}" />
     <xacro:property name="joint_1_upper_limit" value="${2*J_PI}" />
-    <xacro:property name="joint_1_velocity_limit" value="2" />
+    <xacro:property name="joint_1_velocity_limit" value="${36*J_PI/180}" />
     <xacro:property name="joint_1_torque_limit" value="1000" />
     <xacro:property name="joint_2" value="joint_2" />
@@ -59,5 +59,5 @@
     <xacro:property name="joint_2_lower_limit" value="${47/180*J_PI}" />
     <xacro:property name="joint_2_upper_limit" value="${313/180*J_PI}" />
-    <xacro:property name="joint_2_velocity_limit" value="2" />
+    <xacro:property name="joint_2_velocity_limit" value="${36*J_PI/180}" />
     <xacro:property name="joint_2_torque_limit" value="1000" />
     <xacro:property name="joint_3" value="joint_3" />
@@ -68,5 +68,5 @@
     <xacro:property name="joint_3_lower_limit" value="${19/180*J_PI}" />
     <xacro:property name="joint_3_upper_limit" value="${341/180*J_PI}" />
-    <xacro:property name="joint_3_velocity_limit" value="2" />
+    <xacro:property name="joint_3_velocity_limit" value="${36*J_PI/180}" />
     <xacro:property name="joint_3_torque_limit" value="1000" />
     <xacro:property name="joint_4" value="joint_4" />
@@ -77,5 +77,5 @@
     <xacro:property name="joint_4_lower_limit" value="${-2*J_PI}" />
     <xacro:property name="joint_4_upper_limit" value="${2*J_PI}" />
-    <xacro:property name="joint_4_velocity_limit" value="2" />
+    <xacro:property name="joint_4_velocity_limit" value="${48*J_PI/180}" />
     <xacro:property name="joint_4_torque_limit" value="1000" />
     <xacro:property name="joint_5" value="joint_5" />
@@ -86,5 +86,5 @@
     <xacro:property name="joint_5_lower_limit" value="${30/180*J_PI}" />
     <xacro:property name="joint_5_upper_limit" value="${330/180*J_PI}" />
-    <xacro:property name="joint_5_velocity_limit" value="2" />
+    <xacro:property name="joint_5_velocity_limit" value="${48*J_PI/180}" />
     <xacro:property name="joint_5_torque_limit" value="1000" />
     <xacro:property name="joint_6" value="joint_6" />
@@ -95,5 +95,5 @@
     <xacro:property name="joint_6_lower_limit" value="${-2*J_PI}" />
     <xacro:property name="joint_6_upper_limit" value="${2*J_PI}" />
-    <xacro:property name="joint_6_velocity_limit" value="2" />
+    <xacro:property name="joint_6_velocity_limit" value="${48*J_PI/180}" />
     <xacro:property name="joint_6_torque_limit" value="1000" />
     <xacro:property name="joint_end_effector" value="end_effector_offset" />

File: kinova_description/urdf/j2s7s300.xacro (robot description, xacro)
@@ -52,5 +52,5 @@
     <xacro:property name="joint_1_lower_limit" value="${-2*J_PI}" />
     <xacro:property name="joint_1_upper_limit" value="${2*J_PI}" />
-    <xacro:property name="joint_1_velocity_limit" value="2" />
+    <xacro:property name="joint_1_velocity_limit" value="${36*J_PI/180}" />
     <xacro:property name="joint_1_torque_limit" value="1000" />
     <xacro:property name="joint_2" value="joint_2" />
@@ -61,5 +61,5 @@
     <xacro:property name="joint_2_lower_limit" value="${47/180*J_PI}" />
     <xacro:property name="joint_2_upper_limit" value="${313/180*J_PI}" />
-    <xacro:property name="joint_2_velocity_limit" value="2" />
+    <xacro:property name="joint_2_velocity_limit" value="${36*J_PI/180}" />
     <xacro:property name="joint_2_torque_limit" value="1000" />
     <xacro:property name="joint_3" value="joint_3" />
@@ -70,5 +70,5 @@
     <xacro:property name="joint_3_lower_limit" value="${-2*J_PI}" />
     <xacro:property name="joint_3_upper_limit" value="${2*J_PI}" />
-    <xacro:property name="joint_3_velocity_limit" value="2" />
+    <xacro:property name="joint_3_velocity_limit" value="${36*J_PI/180}" />
     <xacro:property name="joint_3_torque_limit" value="1000" />
     <xacro:property name="joint_4" value="joint_4" />
@@ -79,5 +79,5 @@
     <xacro:property name="joint_4_lower_limit" value="${30/180*J_PI}" />
     <xacro:property name="joint_4_upper_limit" value="${330/180*J_PI}" />
-    <xacro:property name="joint_4_velocity_limit" value="2" />
+    <xacro:property name="joint_4_velocity_limit" value="${36*J_PI/180}" />
     <xacro:property name="joint_4_torque_limit" value="1000" />
     <xacro:property name="joint_5" value="joint_5" />
@@ -88,5 +88,5 @@
     <xacro:property name="joint_5_lower_limit" value="${-2*J_PI}" />
     <xacro:property name="joint_5_upper_limit" value="${2*J_PI}" />
-    <xacro:property name="joint_5_velocity_limit" value="2" />
+    <xacro:property name="joint_5_velocity_limit" value="${48*J_PI/180}" />
     <xacro:property name="joint_5_torque_limit" value="1000" />
     <xacro:property name="joint_6" value="joint_6" />
@@ -97,5 +97,5 @@
     <xacro:property name="joint_6_lower_limit" value="${65/180*J_PI}" />
     <xacro:property name="joint_6_upper_limit" value="${295/180*J_PI}" />
-    <xacro:property name="joint_6_velocity_limit" value="2" />
+    <xacro:property name="joint_6_velocity_limit" value="${48*J_PI/180}" />
     <xacro:property name="joint_6_torque_limit" value="1000" />
     <xacro:property name="joint_7" value="joint_7" />
@@ -106,5 +106,5 @@
     <xacro:property name="joint_7_lower_limit" value="${-2*J_PI}" />
     <xacro:property name="joint_7_upper_limit" value="${2*J_PI}" />
-    <xacro:property name="joint_7_velocity_limit" value="2" />
+    <xacro:property name="joint_7_velocity_limit" value="${48*J_PI/180}" />
     <xacro:property name="joint_7_torque_limit" value="1000" />
     <xacro:property name="joint_end_effector" value="end_effector_offset" />

File: kinova_description/urdf/m1n4s200.xacro (robot description, xacro)
@@ -46,5 +46,5 @@
     <xacro:property name="joint_1_lower_limit" value="${-2*J_PI}" />
     <xacro:property name="joint_1_upper_limit" value="${2*J_PI}" />
-    <xacro:property name="joint_1_velocity_limit" value="2" />
+    <xacro:property name="joint_1_velocity_limit" value="${36*J_PI/180}" />
     <xacro:property name="joint_1_torque_limit" value="1000" />
     <xacro:property name="joint_2" value="joint_2" />
@@ -55,5 +55,5 @@
     <xacro:property name="joint_2_lower_limit" value="${50/180*J_PI}" />
     <xacro:property name="joint_2_upper_limit" value="${310/180*J_PI}" />
-    <xacro:property name="joint_2_velocity_limit" value="2" />
+    <xacro:property name="joint_2_velocity_limit" value="${36*J_PI/180}" />
     <xacro:property name="joint_2_torque_limit" value="1000" />
     <xacro:property name="joint_3" value="joint_3" />
@@ -64,5 +64,5 @@
     <xacro:property name="joint_3_lower_limit" value="${35/180*J_PI}" />
     <xacro:property name="joint_3_upper_limit" value="${325/180*J_PI}" />
-    <xacro:property name="joint_3_velocity_limit" value="2" />
+    <xacro:property name="joint_3_velocity_limit" value="${36*J_PI/180}" />
     <xacro:property name="joint_3_torque_limit" value="1000" />
     <xacro:property name="joint_4" value="joint_4" />
@@ -73,5 +73,5 @@
     <xacro:property name="joint_4_lower_limit" value="${-2*J_PI}" />
     <xacro:property name="joint_4_upper_limit" value="${2*J_PI}" />
-    <xacro:property name="joint_4_velocity_limit" value="2" />
+    <xacro:property name="joint_4_velocity_limit" value="${48*J_PI/180}" />
     <xacro:property name="joint_4_torque_limit" value="1000" />
     <xacro:property name="joint_end_effector" value="end_effector_offset" />

File: kinova_description/urdf/m1n6s200.xacro (robot description, xacro)
@@ -50,5 +50,5 @@
     <xacro:property name="joint_1_lower_limit" value="${-2*J_PI}" />
     <xacro:property name="joint_1_upper_limit" value="${2*J_PI}" />
-    <xacro:property name="joint_1_velocity_limit" value="2" />
+    <xacro:property name="joint_1_velocity_limit" value="${36*J_PI/180}" />
     <xacro:property name="joint_1_torque_limit" value="1000" />
     <xacro:property name="joint_2" value="joint_2" />
@@ -59,5 +59,5 @@
     <xacro:property name="joint_2_lower_limit" value="${50/180*J_PI}" />
     <xacro:property name="joint_2_upper_limit" value="${310/180*J_PI}" />
-    <xacro:property name="joint_2_velocity_limit" value="2" />
+    <xacro:property name="joint_2_velocity_limit" value="${36*J_PI/180}" />
     <xacro:property name="joint_2_torque_limit" value="1000" />
     <xacro:property name="joint_3" value="joint_3" />
@@ -68,5 +68,5 @@
     <xacro:property name="joint_3_lower_limit" value="${35/180*J_PI}" />
     <xacro:property name="joint_3_upper_limit" value="${325/180*J_PI}" />
-    <xacro:property name="joint_3_velocity_limit" value="2" />
+    <xacro:property name="joint_3_velocity_limit" value="${36*J_PI/180}" />
     <xacro:property name="joint_3_torque_limit" value="1000" />
     <xacro:property name="joint_4" value="joint_4" />
@@ -77,5 +77,5 @@
     <xacro:property name="joint_4_lower_limit" value="${-2*J_PI}" />
     <xacro:property name="joint_4_upper_limit" value="${2*J_PI}" />
-    <xacro:property name="joint_4_velocity_limit" value="2" />
+    <xacro:property name="joint_4_velocity_limit" value="${48*J_PI/180}" />
     <xacro:property name="joint_4_torque_limit" value="1000" />
     <xacro:property name="joint_5" value="joint_5" />
@@ -86,5 +86,5 @@
     <xacro:property name="joint_5_lower_limit" value="${-2*J_PI}" />
     <xacro:property name="joint_5_upper_limit" value="${2*J_PI}" />
-    <xacro:property name="joint_5_velocity_limit" value="2" />
+    <xacro:property name="joint_5_velocity_limit" value="${48*J_PI/180}" />
     <xacro:property name="joint_5_torque_limit" value="1000" />
     <xacro:property name="joint_6" value="joint_6" />
@@ -95,5 +95,5 @@
     <xacro:property name="joint_6_lower_limit" value="${-2*J_PI}" />
     <xacro:property name="joint_6_upper_limit" value="${2*J_PI}" />
-    <xacro:property name="joint_6_velocity_limit" value="2" />
+    <xacro:property name="joint_6_velocity_limit" value="${48*J_PI/180}" />
     <xacro:property name="joint_6_torque_limit" value="1000" />
     <xacro:property name="joint_end_effector" value="end_effector_offset" />

File: kinova_description/urdf/m1n6s300.xacro (robot description, xacro)
@@ -50,5 +50,5 @@
     <xacro:property name="joint_1_lower_limit" value="${-2*J_PI}" />
     <xacro:property name="joint_1_upper_limit" value="${2*J_PI}" />
-    <xacro:property name="joint_1_velocity_limit" value="2" />
+    <xacro:property name="joint_1_velocity_limit" value="${36*J_PI/180}" />
     <xacro:property name="joint_1_torque_limit" value="1000" />
     <xacro:property name="joint_2" value="joint_2" />
@@ -59,5 +59,5 @@
     <xacro:property name="joint_2_lower_limit" value="${50/180*J_PI}" />
     <xacro:property name="joint_2_upper_limit" value="${310/180*J_PI}" />
-    <xacro:property name="joint_2_velocity_limit" value="2" />
+    <xacro:property name="joint_2_velocity_limit" value="${36*J_PI/180}" />
     <xacro:property name="joint_2_torque_limit" value="1000" />
     <xacro:property name="joint_3" value="joint_3" />
@@ -68,5 +68,5 @@
     <xacro:property name="joint_3_lower_limit" value="${35/180*J_PI}" />
     <xacro:property name="joint_3_upper_limit" value="${325/180*J_PI}" />
-    <xacro:property name="joint_3_velocity_limit" value="2" />
+    <xacro:property name="joint_3_velocity_limit" value="${36*J_PI/180}" />
     <xacro:property name="joint_3_torque_limit" value="1000" />
     <xacro:property name="joint_4" value="joint_4" />
@@ -77,5 +77,5 @@
     <xacro:property name="joint_4_lower_limit" value="${-2*J_PI}" />
     <xacro:property name="joint_4_upper_limit" value="${2*J_PI}" />
-    <xacro:property name="joint_4_velocity_limit" value="2" />
+    <xacro:property name="joint_4_velocity_limit" value="${48*J_PI/180}" />
     <xacro:property name="joint_4_torque_limit" value="1000" />
     <xacro:property name="joint_5" value="joint_5" />
@@ -86,5 +86,5 @@
     <xacro:property name="joint_5_lower_limit" value="${-2*J_PI}" />
     <xacro:property name="joint_5_upper_limit" value="${2*J_PI}" />
-    <xacro:property name="joint_5_velocity_limit" value="2" />
+    <xacro:property name="joint_5_velocity_limit" value="${48*J_PI/180}" />
     <xacro:property name="joint_5_torque_limit" value="1000" />
     <xacro:property name="joint_6" value="joint_6" />
@@ -95,5 +95,5 @@
     <xacro:property name="joint_6_lower_limit" value="${-2*J_PI}" />
     <xacro:property name="joint_6_upper_limit" value="${2*J_PI}" />
-    <xacro:property name="joint_6_velocity_limit" value="2" />
+    <xacro:property name="joint_6_velocity_limit" value="${48*J_PI/180}" />
     <xacro:property name="joint_6_torque_limit" value="1000" />
     <xacro:property name="joint_end_effector" value="end_effector_offset" />
