Commit message: Added more realistic values for effort limits in URDFs

File: kinova_description/urdf/j2n4s300.xacro (robot description, xacro)
@@ -47,5 +47,5 @@
     <xacro:property name="joint_1_upper_limit" value="${2*J_PI}" />
     <xacro:property name="joint_1_velocity_limit" value="${36*J_PI/180}" />
-    <xacro:property name="joint_1_torque_limit" value="1000" />
+    <xacro:property name="joint_1_torque_limit" value="40" />
     <xacro:property name="joint_2" value="joint_2" />
     <xacro:property name="joint_2_type" value="revolute" />
@@ -56,5 +56,5 @@
     <xacro:property name="joint_2_upper_limit" value="${313/180*J_PI}" />
     <xacro:property name="joint_2_velocity_limit" value="${36*J_PI/180}" />
-    <xacro:property name="joint_2_torque_limit" value="1000" />
+    <xacro:property name="joint_2_torque_limit" value="80" />
     <xacro:property name="joint_3" value="joint_3" />
     <xacro:property name="joint_3_type" value="revolute" />
@@ -65,5 +65,5 @@
     <xacro:property name="joint_3_upper_limit" value="${341/180*J_PI}" />
     <xacro:property name="joint_3_velocity_limit" value="${36*J_PI/180}" />
-    <xacro:property name="joint_3_torque_limit" value="1000" />
+    <xacro:property name="joint_3_torque_limit" value="40" />
     <xacro:property name="joint_4" value="joint_4" />
     <xacro:property name="joint_4_type" value="continuous" />
@@ -74,5 +74,5 @@
     <xacro:property name="joint_4_upper_limit" value="${2*J_PI}" />
     <xacro:property name="joint_4_velocity_limit" value="${48*J_PI/180}" />
-    <xacro:property name="joint_4_torque_limit" value="1000" />
+    <xacro:property name="joint_4_torque_limit" value="20" />
     <xacro:property name="joint_end_effector" value="end_effector_offset" />
     <xacro:property name="joint_end_effector_type" value="fixed" />

File: kinova_description/urdf/j2n6s200.xacro (robot description, xacro)
@@ -51,5 +51,5 @@
     <xacro:property name="joint_1_upper_limit" value="${2*J_PI}" />
     <xacro:property name="joint_1_velocity_limit" value="${36*J_PI/180}" />
-    <xacro:property name="joint_1_torque_limit" value="1000" />
+    <xacro:property name="joint_1_torque_limit" value="40" />
     <xacro:property name="joint_2" value="joint_2" />
     <xacro:property name="joint_2_type" value="revolute" />
@@ -60,5 +60,5 @@
     <xacro:property name="joint_2_upper_limit" value="${313/180*J_PI}" />
     <xacro:property name="joint_2_velocity_limit" value="${36*J_PI/180}" />
-    <xacro:property name="joint_2_torque_limit" value="1000" />
+    <xacro:property name="joint_2_torque_limit" value="80" />
     <xacro:property name="joint_3" value="joint_3" />
     <xacro:property name="joint_3_type" value="revolute" />
@@ -69,5 +69,5 @@
     <xacro:property name="joint_3_upper_limit" value="${341/180*J_PI}" />
     <xacro:property name="joint_3_velocity_limit" value="${36*J_PI/180}" />
-    <xacro:property name="joint_3_torque_limit" value="1000" />
+    <xacro:property name="joint_3_torque_limit" value="40" />
     <xacro:property name="joint_4" value="joint_4" />
     <xacro:property name="joint_4_type" value="continuous" />
@@ -78,5 +78,5 @@
     <xacro:property name="joint_4_upper_limit" value="${2*J_PI}" />
     <xacro:property name="joint_4_velocity_limit" value="${48*J_PI/180}" />
-    <xacro:property name="joint_4_torque_limit" value="1000" />
+    <xacro:property name="joint_4_torque_limit" value="20" />
     <xacro:property name="joint_5" value="joint_5" />
     <xacro:property name="joint_5_type" value="continuous" />
@@ -87,5 +87,5 @@
     <xacro:property name="joint_5_upper_limit" value="${2*J_PI}" />
     <xacro:property name="joint_5_velocity_limit" value="${48*J_PI/180}" />
-    <xacro:property name="joint_5_torque_limit" value="1000" />
+    <xacro:property name="joint_5_torque_limit" value="20" />
     <xacro:property name="joint_6" value="joint_6" />
     <xacro:property name="joint_6_type" value="continuous" />
@@ -96,5 +96,5 @@
     <xacro:property name="joint_6_upper_limit" value="${2*J_PI}" />
     <xacro:property name="joint_6_velocity_limit" value="${48*J_PI/180}" />
-    <xacro:property name="joint_6_torque_limit" value="1000" />
+    <xacro:property name="joint_6_torque_limit" value="20" />
     <xacro:property name="joint_end_effector" value="end_effector_offset" />
     <xacro:property name="joint_end_effector_type" value="fixed" />

File: kinova_description/urdf/j2n6s300.xacro (robot description, xacro)
@@ -51,5 +51,5 @@
     <xacro:property name="joint_1_upper_limit" value="${2*J_PI}" />
     <xacro:property name="joint_1_velocity_limit" value="${36*J_PI/180}" />
-    <xacro:property name="joint_1_torque_limit" value="1000" />
+    <xacro:property name="joint_1_torque_limit" value="40" />
     <xacro:property name="joint_2" value="joint_2" />
     <xacro:property name="joint_2_type" value="revolute" />
@@ -60,5 +60,5 @@
     <xacro:property name="joint_2_upper_limit" value="${313/180*J_PI}" />
     <xacro:property name="joint_2_velocity_limit" value="${36*J_PI/180}" />
-    <xacro:property name="joint_2_torque_limit" value="1000" />
+    <xacro:property name="joint_2_torque_limit" value="80" />
     <xacro:property name="joint_3" value="joint_3" />
     <xacro:property name="joint_3_type" value="revolute" />
@@ -69,5 +69,5 @@
     <xacro:property name="joint_3_upper_limit" value="${341/180*J_PI}" />
     <xacro:property name="joint_3_velocity_limit" value="${36*J_PI/180}" />
-    <xacro:property name="joint_3_torque_limit" value="1000" />
+    <xacro:property name="joint_3_torque_limit" value="40" />
     <xacro:property name="joint_4" value="joint_4" />
     <xacro:property name="joint_4_type" value="continuous" />
@@ -78,5 +78,5 @@
     <xacro:property name="joint_4_upper_limit" value="${2*J_PI}" />
     <xacro:property name="joint_4_velocity_limit" value="${48*J_PI/180}" />
-    <xacro:property name="joint_4_torque_limit" value="1000" />
+    <xacro:property name="joint_4_torque_limit" value="20" />
     <xacro:property name="joint_5" value="joint_5" />
     <xacro:property name="joint_5_type" value="continuous" />
@@ -87,5 +87,5 @@
     <xacro:property name="joint_5_upper_limit" value="${2*J_PI}" />
     <xacro:property name="joint_5_velocity_limit" value="${48*J_PI/180}" />
-    <xacro:property name="joint_5_torque_limit" value="1000" />
+    <xacro:property name="joint_5_torque_limit" value="20" />
     <xacro:property name="joint_6" value="joint_6" />
     <xacro:property name="joint_6_type" value="continuous" />
@@ -96,5 +96,5 @@
     <xacro:property name="joint_6_upper_limit" value="${2*J_PI}" />
     <xacro:property name="joint_6_velocity_limit" value="${48*J_PI/180}" />
-    <xacro:property name="joint_6_torque_limit" value="1000" />
+    <xacro:property name="joint_6_torque_limit" value="20" />
     <xacro:property name="joint_end_effector" value="end_effector_offset" />
     <xacro:property name="joint_end_effector_type" value="fixed" />

File: kinova_description/urdf/j2s6s300.xacro (robot description, xacro)
@@ -51,5 +51,5 @@
     <xacro:property name="joint_1_upper_limit" value="${2*J_PI}" />
     <xacro:property name="joint_1_velocity_limit" value="${36*J_PI/180}" />
-    <xacro:property name="joint_1_torque_limit" value="1000" />
+    <xacro:property name="joint_1_torque_limit" value="40" />
     <xacro:property name="joint_2" value="joint_2" />
     <xacro:property name="joint_2_type" value="revolute" />
@@ -60,5 +60,5 @@
     <xacro:property name="joint_2_upper_limit" value="${313/180*J_PI}" />
     <xacro:property name="joint_2_velocity_limit" value="${36*J_PI/180}" />
-    <xacro:property name="joint_2_torque_limit" value="1000" />
+    <xacro:property name="joint_2_torque_limit" value="80" />
     <xacro:property name="joint_3" value="joint_3" />
     <xacro:property name="joint_3_type" value="revolute" />
@@ -69,5 +69,5 @@
     <xacro:property name="joint_3_upper_limit" value="${341/180*J_PI}" />
     <xacro:property name="joint_3_velocity_limit" value="${36*J_PI/180}" />
-    <xacro:property name="joint_3_torque_limit" value="1000" />
+    <xacro:property name="joint_3_torque_limit" value="40" />
     <xacro:property name="joint_4" value="joint_4" />
     <xacro:property name="joint_4_type" value="continuous" />
@@ -78,5 +78,5 @@
     <xacro:property name="joint_4_upper_limit" value="${2*J_PI}" />
     <xacro:property name="joint_4_velocity_limit" value="${48*J_PI/180}" />
-    <xacro:property name="joint_4_torque_limit" value="1000" />
+    <xacro:property name="joint_4_torque_limit" value="20" />
     <xacro:property name="joint_5" value="joint_5" />
     <xacro:property name="joint_5_type" value="revolute" />
@@ -87,5 +87,5 @@
     <xacro:property name="joint_5_upper_limit" value="${330/180*J_PI}" />
     <xacro:property name="joint_5_velocity_limit" value="${48*J_PI/180}" />
-    <xacro:property name="joint_5_torque_limit" value="1000" />
+    <xacro:property name="joint_5_torque_limit" value="20" />
     <xacro:property name="joint_6" value="joint_6" />
     <xacro:property name="joint_6_type" value="continuous" />
@@ -96,5 +96,5 @@
     <xacro:property name="joint_6_upper_limit" value="${2*J_PI}" />
     <xacro:property name="joint_6_velocity_limit" value="${48*J_PI/180}" />
-    <xacro:property name="joint_6_torque_limit" value="1000" />
+    <xacro:property name="joint_6_torque_limit" value="20" />
     <xacro:property name="joint_end_effector" value="end_effector_offset" />
     <xacro:property name="joint_end_effector_type" value="fixed" />

File: kinova_description/urdf/j2s7s300.xacro (robot description, xacro)
@@ -53,5 +53,5 @@
     <xacro:property name="joint_1_upper_limit" value="${2*J_PI}" />
     <xacro:property name="joint_1_velocity_limit" value="${36*J_PI/180}" />
-    <xacro:property name="joint_1_torque_limit" value="1000" />
+    <xacro:property name="joint_1_torque_limit" value="40" />
     <xacro:property name="joint_2" value="joint_2" />
     <xacro:property name="joint_2_type" value="revolute" />
@@ -62,5 +62,5 @@
     <xacro:property name="joint_2_upper_limit" value="${313/180*J_PI}" />
     <xacro:property name="joint_2_velocity_limit" value="${36*J_PI/180}" />
-    <xacro:property name="joint_2_torque_limit" value="1000" />
+    <xacro:property name="joint_2_torque_limit" value="80" />
     <xacro:property name="joint_3" value="joint_3" />
     <xacro:property name="joint_3_type" value="continuous" />
@@ -71,5 +71,5 @@
     <xacro:property name="joint_3_upper_limit" value="${2*J_PI}" />
     <xacro:property name="joint_3_velocity_limit" value="${36*J_PI/180}" />
-    <xacro:property name="joint_3_torque_limit" value="1000" />
+    <xacro:property name="joint_3_torque_limit" value="40" />
     <xacro:property name="joint_4" value="joint_4" />
     <xacro:property name="joint_4_type" value="revolute" />
@@ -80,5 +80,5 @@
     <xacro:property name="joint_4_upper_limit" value="${330/180*J_PI}" />
     <xacro:property name="joint_4_velocity_limit" value="${36*J_PI/180}" />
-    <xacro:property name="joint_4_torque_limit" value="1000" />
+    <xacro:property name="joint_4_torque_limit" value="40" />
     <xacro:property name="joint_5" value="joint_5" />
     <xacro:property name="joint_5_type" value="continuous" />
@@ -89,5 +89,5 @@
     <xacro:property name="joint_5_upper_limit" value="${2*J_PI}" />
     <xacro:property name="joint_5_velocity_limit" value="${48*J_PI/180}" />
-    <xacro:property name="joint_5_torque_limit" value="1000" />
+    <xacro:property name="joint_5_torque_limit" value="20" />
     <xacro:property name="joint_6" value="joint_6" />
     <xacro:property name="joint_6_type" value="revolute" />
@@ -98,5 +98,5 @@
     <xacro:property name="joint_6_upper_limit" value="${295/180*J_PI}" />
     <xacro:property name="joint_6_velocity_limit" value="${48*J_PI/180}" />
-    <xacro:property name="joint_6_torque_limit" value="1000" />
+    <xacro:property name="joint_6_torque_limit" value="20" />
     <xacro:property name="joint_7" value="joint_7" />
     <xacro:property name="joint_7_type" value="continuous" />
@@ -107,5 +107,5 @@
     <xacro:property name="joint_7_upper_limit" value="${2*J_PI}" />
     <xacro:property name="joint_7_velocity_limit" value="${48*J_PI/180}" />
-    <xacro:property name="joint_7_torque_limit" value="1000" />
+    <xacro:property name="joint_7_torque_limit" value="20" />
     <xacro:property name="joint_end_effector" value="end_effector_offset" />
     <xacro:property name="joint_end_effector_type" value="fixed" />

File: kinova_description/urdf/m1n4s200.xacro (robot description, xacro)
@@ -47,5 +47,5 @@
     <xacro:property name="joint_1_upper_limit" value="${2*J_PI}" />
     <xacro:property name="joint_1_velocity_limit" value="${36*J_PI/180}" />
-    <xacro:property name="joint_1_torque_limit" value="1000" />
+    <xacro:property name="joint_1_torque_limit" value="40" />
     <xacro:property name="joint_2" value="joint_2" />
     <xacro:property name="joint_2_type" value="revolute" />
@@ -56,5 +56,5 @@
     <xacro:property name="joint_2_upper_limit" value="${310/180*J_PI}" />
     <xacro:property name="joint_2_velocity_limit" value="${36*J_PI/180}" />
-    <xacro:property name="joint_2_torque_limit" value="1000" />
+    <xacro:property name="joint_2_torque_limit" value="80" />
     <xacro:property name="joint_3" value="joint_3" />
     <xacro:property name="joint_3_type" value="revolute" />
@@ -65,5 +65,5 @@
     <xacro:property name="joint_3_upper_limit" value="${325/180*J_PI}" />
     <xacro:property name="joint_3_velocity_limit" value="${36*J_PI/180}" />
-    <xacro:property name="joint_3_torque_limit" value="1000" />
+    <xacro:property name="joint_3_torque_limit" value="40" />
     <xacro:property name="joint_4" value="joint_4" />
     <xacro:property name="joint_4_type" value="continuous" />
@@ -74,5 +74,5 @@
     <xacro:property name="joint_4_upper_limit" value="${2*J_PI}" />
     <xacro:property name="joint_4_velocity_limit" value="${48*J_PI/180}" />
-    <xacro:property name="joint_4_torque_limit" value="1000" />
+    <xacro:property name="joint_4_torque_limit" value="20" />
     <xacro:property name="joint_end_effector" value="end_effector_offset" />
     <xacro:property name="joint_end_effector_type" value="fixed" />

File: kinova_description/urdf/m1n6s200.xacro (robot description, xacro)
@@ -51,5 +51,5 @@
     <xacro:property name="joint_1_upper_limit" value="${2*J_PI}" />
     <xacro:property name="joint_1_velocity_limit" value="${36*J_PI/180}" />
-    <xacro:property name="joint_1_torque_limit" value="1000" />
+    <xacro:property name="joint_1_torque_limit" value="40" />
     <xacro:property name="joint_2" value="joint_2" />
     <xacro:property name="joint_2_type" value="revolute" />
@@ -60,5 +60,5 @@
     <xacro:property name="joint_2_upper_limit" value="${310/180*J_PI}" />
     <xacro:property name="joint_2_velocity_limit" value="${36*J_PI/180}" />
-    <xacro:property name="joint_2_torque_limit" value="1000" />
+    <xacro:property name="joint_2_torque_limit" value="80" />
     <xacro:property name="joint_3" value="joint_3" />
     <xacro:property name="joint_3_type" value="revolute" />
@@ -69,5 +69,5 @@
     <xacro:property name="joint_3_upper_limit" value="${325/180*J_PI}" />
     <xacro:property name="joint_3_velocity_limit" value="${36*J_PI/180}" />
-    <xacro:property name="joint_3_torque_limit" value="1000" />
+    <xacro:property name="joint_3_torque_limit" value="40" />
     <xacro:property name="joint_4" value="joint_4" />
     <xacro:property name="joint_4_type" value="continuous" />
@@ -78,5 +78,5 @@
     <xacro:property name="joint_4_upper_limit" value="${2*J_PI}" />
     <xacro:property name="joint_4_velocity_limit" value="${48*J_PI/180}" />
-    <xacro:property name="joint_4_torque_limit" value="1000" />
+    <xacro:property name="joint_4_torque_limit" value="20" />
     <xacro:property name="joint_5" value="joint_5" />
     <xacro:property name="joint_5_type" value="continuous" />
@@ -87,5 +87,5 @@
     <xacro:property name="joint_5_upper_limit" value="${2*J_PI}" />
     <xacro:property name="joint_5_velocity_limit" value="${48*J_PI/180}" />
-    <xacro:property name="joint_5_torque_limit" value="1000" />
+    <xacro:property name="joint_5_torque_limit" value="20" />
     <xacro:property name="joint_6" value="joint_6" />
     <xacro:property name="joint_6_type" value="continuous" />
@@ -96,5 +96,5 @@
     <xacro:property name="joint_6_upper_limit" value="${2*J_PI}" />
     <xacro:property name="joint_6_velocity_limit" value="${48*J_PI/180}" />
-    <xacro:property name="joint_6_torque_limit" value="1000" />
+    <xacro:property name="joint_6_torque_limit" value="20" />
     <xacro:property name="joint_end_effector" value="end_effector_offset" />
     <xacro:property name="joint_end_effector_type" value="fixed" />

File: kinova_description/urdf/m1n6s300.xacro (robot description, xacro)
@@ -51,5 +51,5 @@
     <xacro:property name="joint_1_upper_limit" value="${2*J_PI}" />
     <xacro:property name="joint_1_velocity_limit" value="${36*J_PI/180}" />
-    <xacro:property name="joint_1_torque_limit" value="1000" />
+    <xacro:property name="joint_1_torque_limit" value="40" />
     <xacro:property name="joint_2" value="joint_2" />
     <xacro:property name="joint_2_type" value="revolute" />
@@ -60,5 +60,5 @@
     <xacro:property name="joint_2_upper_limit" value="${310/180*J_PI}" />
     <xacro:property name="joint_2_velocity_limit" value="${36*J_PI/180}" />
-    <xacro:property name="joint_2_torque_limit" value="1000" />
+    <xacro:property name="joint_2_torque_limit" value="80" />
     <xacro:property name="joint_3" value="joint_3" />
     <xacro:property name="joint_3_type" value="revolute" />
@@ -69,5 +69,5 @@
     <xacro:property name="joint_3_upper_limit" value="${325/180*J_PI}" />
     <xacro:property name="joint_3_velocity_limit" value="${36*J_PI/180}" />
-    <xacro:property name="joint_3_torque_limit" value="1000" />
+    <xacro:property name="joint_3_torque_limit" value="40" />
     <xacro:property name="joint_4" value="joint_4" />
     <xacro:property name="joint_4_type" value="continuous" />
@@ -78,5 +78,5 @@
     <xacro:property name="joint_4_upper_limit" value="${2*J_PI}" />
     <xacro:property name="joint_4_velocity_limit" value="${48*J_PI/180}" />
-    <xacro:property name="joint_4_torque_limit" value="1000" />
+    <xacro:property name="joint_4_torque_limit" value="20" />
     <xacro:property name="joint_5" value="joint_5" />
     <xacro:property name="joint_5_type" value="continuous" />
@@ -87,5 +87,5 @@
     <xacro:property name="joint_5_upper_limit" value="${2*J_PI}" />
     <xacro:property name="joint_5_velocity_limit" value="${48*J_PI/180}" />
-    <xacro:property name="joint_5_torque_limit" value="1000" />
+    <xacro:property name="joint_5_torque_limit" value="20" />
     <xacro:property name="joint_6" value="joint_6" />
     <xacro:property name="joint_6_type" value="continuous" />
@@ -96,5 +96,5 @@
     <xacro:property name="joint_6_upper_limit" value="${2*J_PI}" />
     <xacro:property name="joint_6_velocity_limit" value="${48*J_PI/180}" />
-    <xacro:property name="joint_6_torque_limit" value="1000" />
+    <xacro:property name="joint_6_torque_limit" value="20" />
     <xacro:property name="joint_end_effector" value="end_effector_offset" />
     <xacro:property name="joint_end_effector_type" value="fixed" />
