Commit message: Changed urdf files to allow custom prefix to be added
Changed urdf files to allow custom prefix to be added
Added structure to be able to control multiple robots from 1 node

File: kinova_description/urdf/j2n7s300.xacro (robot description, xacro)
@@ -16,14 +16,4 @@
     <xacro:include filename="$(find kinova_description)/urdf/kinova_common.xacro" />
     <xacro:include filename="$(find kinova_description)/urdf/kinova_finger_set.xacro" />
-    <property name="prefix" value="j2n7s300" />
-    <property name="link_base" value="${prefix}_link_base" />
-    <property name="link_1" value="${prefix}_link_1" />
-    <property name="link_2" value="${prefix}_link_2" />
-    <property name="link_3" value="${prefix}_link_3" />
-    <property name="link_4" value="${prefix}_link_4" />
-    <property name="link_5" value="${prefix}_link_5" />
-    <property name="link_6" value="${prefix}_link_6" />
-    <property name="link_7" value="${prefix}_link_7" />
-    <property name="link_end_effector" value="${prefix}_end_effector" />
     <property name="link_base_mesh" value="base" />
     <property name="link_1_mesh" value="shoulder" />
@@ -34,10 +24,10 @@
     <property name="link_6_mesh" value="wrist" />
     <property name="link_7_mesh" value="hand_3finger" />
-    <property name="joint_base" value="${prefix}_joint_base" />
+    <property name="joint_base" value="joint_base" />
     <property name="joint_base_type" value="fixed" />
     <property name="joint_base_axis_xyz" value="0 0 0" />
     <property name="joint_base_origin_xyz" value="0 0 0" />
     <property name="joint_base_origin_rpy" value="0 0 0" />
-    <property name="joint_1" value="${prefix}_joint_1" />
+    <property name="joint_1" value="joint_1" />
     <property name="joint_1_type" value="continuous" />
     <property name="joint_1_axis_xyz" value="0 0 1" />
@@ -46,5 +36,5 @@
     <property name="joint_1_lower_limit" value="${-2*J_PI}" />
     <property name="joint_1_upper_limit" value="${2*J_PI}" />
-    <property name="joint_2" value="${prefix}_joint_2" />
+    <property name="joint_2" value="joint_2" />
     <property name="joint_2_type" value="revolute" />
     <property name="joint_2_axis_xyz" value="0 0 1" />
@@ -53,5 +43,5 @@
     <property name="joint_2_lower_limit" value="${30/180*J_PI}" />
     <property name="joint_2_upper_limit" value="${330/180*J_PI}" />
-    <property name="joint_3" value="${prefix}_joint_3" />
+    <property name="joint_3" value="joint_3" />
     <property name="joint_3_type" value="continuous" />
     <property name="joint_3_axis_xyz" value="0 0 1" />
@@ -60,5 +50,5 @@
     <property name="joint_3_lower_limit" value="${-5*J_PI/4}" />
     <property name="joint_3_upper_limit" value="${1*J_PI/4}" />
-    <property name="joint_4" value="${prefix}_joint_4" />
+    <property name="joint_4" value="joint_4" />
     <property name="joint_4_type" value="revolute" />
     <property name="joint_4_axis_xyz" value="0 0 1" />
@@ -67,5 +57,5 @@
     <property name="joint_4_lower_limit" value="${30/180*J_PI}" />
     <property name="joint_4_upper_limit" value="${330/180*J_PI}" />
-    <property name="joint_5" value="${prefix}_joint_5" />
+    <property name="joint_5" value="joint_5" />
     <property name="joint_5_type" value="continuous" />
     <property name="joint_5_axis_xyz" value="0 0 1" />
@@ -74,5 +64,5 @@
     <property name="joint_5_lower_limit" value="${-2*J_PI}" />
     <property name="joint_5_upper_limit" value="${2*J_PI}" />
-    <property name="joint_6" value="${prefix}_joint_6" />
+    <property name="joint_6" value="joint_6" />
     <property name="joint_6_type" value="continuous" />
     <property name="joint_6_axis_xyz" value="0 0 1" />
@@ -81,5 +71,5 @@
     <property name="joint_6_lower_limit" value="${-2*J_PI}" />
     <property name="joint_6_upper_limit" value="${2*J_PI}" />
-    <property name="joint_7" value="${prefix}_joint_7" />
+    <property name="joint_7" value="joint_7" />
     <property name="joint_7_type" value="continuous" />
     <property name="joint_7_axis_xyz" value="0 0 1" />
@@ -88,29 +78,29 @@
     <property name="joint_7_lower_limit" value="${-2*J_PI}" />
     <property name="joint_7_upper_limit" value="${2*J_PI}" />
-    <property name="joint_end_effector" value="${prefix}_end_effector_offset" />
+    <property name="joint_end_effector" value="end_effector_offset" />
     <property name="joint_end_effector_type" value="fixed" />
     <property name="joint_end_effector_axis_xyz" value="0 0 0" />
     <property name="joint_end_effector_origin_xyz" value="0 0 -0.1600" />
     <property name="joint_end_effector_origin_rpy" value="${J_PI} 0 0" />
-    <xacro:macro name="j2n7s300" params="base_parent">
-        <xacro:kinova_armlink link_name="${link_base}" link_mesh="${link_base_mesh}"/>
-        <xacro:kinova_armjoint joint_name="${joint_base}" type="${joint_base_type}" parent="${base_parent}" child="${link_base}" joint_axis_xyz="${joint_base_axis_xyz}" joint_origin_xyz="${joint_base_origin_xyz}" joint_origin_rpy="${joint_base_origin_rpy}" joint_lower_limit="0" joint_upper_limit="0"/>
-        <xacro:kinova_armlink link_name="${link_1}" link_mesh="${link_1_mesh}"/>
-        <xacro:kinova_armjoint joint_name="${joint_1}" type="${joint_1_type}" parent="${link_base}" child="${link_1}" joint_axis_xyz="${joint_1_axis_xyz}" joint_origin_xyz="${joint_1_origin_xyz}" joint_origin_rpy="${joint_1_origin_rpy}" joint_lower_limit="${joint_1_lower_limit}" joint_upper_limit="${joint_1_upper_limit}"/>
-        <xacro:kinova_armlink link_name="${link_2}" link_mesh="${link_2_mesh}"/>
-        <xacro:kinova_armjoint joint_name="${joint_2}" type="${joint_2_type}" parent="${link_1}" child="${link_2}" joint_axis_xyz="${joint_2_axis_xyz}" joint_origin_xyz="${joint_2_origin_xyz}" joint_origin_rpy="${joint_2_origin_rpy}" joint_lower_limit="${joint_2_lower_limit}" joint_upper_limit="${joint_2_upper_limit}"/>
-        <xacro:kinova_armlink link_name="${link_3}" link_mesh="${link_3_mesh}"/>
-        <xacro:kinova_armjoint joint_name="${joint_3}" type="${joint_3_type}" parent="${link_2}" child="${link_3}" joint_axis_xyz="${joint_3_axis_xyz}" joint_origin_xyz="${joint_3_origin_xyz}" joint_origin_rpy="${joint_3_origin_rpy}" joint_lower_limit="${joint_3_lower_limit}" joint_upper_limit="${joint_3_upper_limit}"/>
-        <xacro:kinova_armlink link_name="${link_4}" link_mesh="${link_4_mesh}"/>
-        <xacro:kinova_armjoint joint_name="${joint_4}" type="${joint_4_type}" parent="${link_3}" child="${link_4}" joint_axis_xyz="${joint_4_axis_xyz}" joint_origin_xyz="${joint_4_origin_xyz}" joint_origin_rpy="${joint_4_origin_rpy}" joint_lower_limit="${joint_4_lower_limit}" joint_upper_limit="${joint_4_upper_limit}"/>
-        <xacro:kinova_armlink link_name="${link_5}" link_mesh="${link_5_mesh}"/>
-        <xacro:kinova_armjoint joint_name="${joint_5}" type="${joint_5_type}" parent="${link_4}" child="${link_5}" joint_axis_xyz="${joint_5_axis_xyz}" joint_origin_xyz="${joint_5_origin_xyz}" joint_origin_rpy="${joint_5_origin_rpy}" joint_lower_limit="${joint_5_lower_limit}" joint_upper_limit="${joint_5_upper_limit}"/>
-        <xacro:kinova_armlink link_name="${link_6}" link_mesh="${link_6_mesh}"/>
-        <xacro:kinova_armjoint joint_name="${joint_6}" type="${joint_6_type}" parent="${link_5}" child="${link_6}" joint_axis_xyz="${joint_6_axis_xyz}" joint_origin_xyz="${joint_6_origin_xyz}" joint_origin_rpy="${joint_6_origin_rpy}" joint_lower_limit="${joint_6_lower_limit}" joint_upper_limit="${joint_6_upper_limit}"/>
-        <xacro:kinova_armlink link_name="${link_7}" link_mesh="${link_7_mesh}"/>
-        <xacro:kinova_armjoint joint_name="${joint_7}" type="${joint_7_type}" parent="${link_6}" child="${link_7}" joint_axis_xyz="${joint_7_axis_xyz}" joint_origin_xyz="${joint_7_origin_xyz}" joint_origin_rpy="${joint_7_origin_rpy}" joint_lower_limit="${joint_7_lower_limit}" joint_upper_limit="${joint_7_upper_limit}"/>
-        <xacro:kinova_virtual_link link_name="${link_end_effector}"/>
-        <xacro:kinova_virtual_joint joint_name="${joint_end_effector}" type="${joint_end_effector_type}" parent="${link_7}" child="${link_end_effector}" joint_axis_xyz="${joint_end_effector_axis_xyz}" joint_origin_xyz="${joint_end_effector_origin_xyz}" joint_origin_rpy="${joint_end_effector_origin_rpy}" joint_lower_limit="0" joint_upper_limit="0"/>
+    <xacro:macro name="j2n7s300" params="base_parent prefix:=j2n7s300_">
+        <xacro:kinova_armlink link_name="${prefix}link_base" link_mesh="${link_base_mesh}"/>
+        <xacro:kinova_armjoint joint_name="${prefix}joint_base" type="${joint_base_type}" parent="${prefix}base_parent" child="${prefix}link_base" joint_axis_xyz="${joint_base_axis_xyz}" joint_origin_xyz="${joint_base_origin_xyz}" joint_origin_rpy="${joint_base_origin_rpy}" joint_lower_limit="0" joint_upper_limit="0"/>
+        <xacro:kinova_armlink link_name="${prefix}link_1" link_mesh="${link_1_mesh}"/>
+        <xacro:kinova_armjoint joint_name="${prefix}joint_1" type="${joint_1_type}" parent="${prefix}link_base" child="${prefix}link_1" joint_axis_xyz="${joint_1_axis_xyz}" joint_origin_xyz="${joint_1_origin_xyz}" joint_origin_rpy="${joint_1_origin_rpy}" joint_lower_limit="${joint_1_lower_limit}" joint_upper_limit="${joint_1_upper_limit}"/>
+        <xacro:kinova_armlink link_name="${prefix}link_2" link_mesh="${link_2_mesh}"/>
+        <xacro:kinova_armjoint joint_name="${prefix}joint_2" type="${joint_2_type}" parent="$prefix}link_1" child="${prefix}link_2" joint_axis_xyz="${joint_2_axis_xyz}" joint_origin_xyz="${joint_2_origin_xyz}" joint_origin_rpy="${joint_2_origin_rpy}" joint_lower_limit="${joint_2_lower_limit}" joint_upper_limit="${joint_2_upper_limit}"/>
+        <xacro:kinova_armlink link_name="${prefix}link_3" link_mesh="${link_3_mesh}"/>
+        <xacro:kinova_armjoint joint_name="${prefix}joint_3" type="${joint_3_type}" parent="${prefix}link_2" child="${prefix}link_3" joint_axis_xyz="${joint_3_axis_xyz}" joint_origin_xyz="${joint_3_origin_xyz}" joint_origin_rpy="${joint_3_origin_rpy}" joint_lower_limit="${joint_3_lower_limit}" joint_upper_limit="${joint_3_upper_limit}"/>
+        <xacro:kinova_armlink link_name="${prefix}link_4" link_mesh="${link_4_mesh}"/>
+        <xacro:kinova_armjoint joint_name="${prefix}joint_4" type="${joint_4_type}" parent="${prefix}link_3" child="${prefix}link_4" joint_axis_xyz="${joint_4_axis_xyz}" joint_origin_xyz="${joint_4_origin_xyz}" joint_origin_rpy="${joint_4_origin_rpy}" joint_lower_limit="${joint_4_lower_limit}" joint_upper_limit="${joint_4_upper_limit}"/>
+        <xacro:kinova_armlink link_name="${prefix}link_5" link_mesh="${link_5_mesh}"/>
+        <xacro:kinova_armjoint joint_name="${prefix}joint_5" type="${joint_5_type}" parent="${prefix}link_4" child="${prefix}link_5" joint_axis_xyz="${joint_5_axis_xyz}" joint_origin_xyz="${joint_5_origin_xyz}" joint_origin_rpy="${joint_5_origin_rpy}" joint_lower_limit="${joint_5_lower_limit}" joint_upper_limit="${joint_5_upper_limit}"/>
+        <xacro:kinova_armlink link_name="${prefix}link_6" link_mesh="${link_6_mesh}"/>
+        <xacro:kinova_armjoint joint_name="${prefix}joint_6" type="${joint_6_type}" parent="${prefix}link_5" child="${prefix}link_6" joint_axis_xyz="${joint_6_axis_xyz}" joint_origin_xyz="${joint_6_origin_xyz}" joint_origin_rpy="${joint_6_origin_rpy}" joint_lower_limit="${joint_6_lower_limit}" joint_upper_limit="${joint_6_upper_limit}"/>
+        <xacro:kinova_armlink link_name="${prefix}link_7" link_mesh="${link_7_mesh}"/>
+        <xacro:kinova_armjoint joint_name="${prefix}joint_7" type="${joint_7_type}" parent="${prefix}link_6" child="${prefix}link_7" joint_axis_xyz="${joint_7_axis_xyz}" joint_origin_xyz="${joint_7_origin_xyz}" joint_origin_rpy="${joint_7_origin_rpy}" joint_lower_limit="${joint_7_lower_limit}" joint_upper_limit="${joint_7_upper_limit}"/>
+        <xacro:kinova_virtual_link link_name="${prefix}end_effector"/>
+        <xacro:kinova_virtual_joint joint_name="${prefix}joint_end_effector" type="${joint_end_effector_type}" parent="${prefix}link_7" child="${prefix}link_end_effector" joint_axis_xyz="${joint_end_effector_axis_xyz}" joint_origin_xyz="${joint_end_effector_origin_xyz}" joint_origin_rpy="${joint_end_effector_origin_rpy}" joint_lower_limit="0" joint_upper_limit="0"/>
+				<!--xacro:kinova_3fingers link_hand="link_7" prefix="${prefix}"/-->
     </xacro:macro>
-    <xacro:kinova_3fingers link_hand="${link_7}" prefix="${prefix}"/>
 </root>
