Commit message: Changed urdf files to allow custom prefix to be added
Changed urdf files to allow custom prefix to be added
Added structure to be able to control multiple robots from 1 node

File: kinova_description/urdf/j2s7s300.xacro (robot description, xacro)
@@ -16,14 +16,4 @@
     <xacro:include filename="$(find kinova_description)/urdf/kinova_common.xacro" />
     <xacro:include filename="$(find kinova_description)/urdf/kinova_finger_set.xacro" />
-    <property name="prefix" value="j2s7s300" />
-    <property name="link_base" value="${prefix}_link_base" />
-    <property name="link_1" value="${prefix}_link_1" />
-    <property name="link_2" value="${prefix}_link_2" />
-    <property name="link_3" value="${prefix}_link_3" />
-    <property name="link_4" value="${prefix}_link_4" />
-    <property name="link_5" value="${prefix}_link_5" />
-    <property name="link_6" value="${prefix}_link_6" />
-    <property name="link_7" value="${prefix}_link_7" />
-    <property name="link_end_effector" value="${prefix}_end_effector" />
     <property name="link_base_mesh" value="base" />
     <property name="link_1_mesh" value="shoulder" />
@@ -34,10 +24,10 @@
     <property name="link_6_mesh" value="wrist_spherical_2" />
     <property name="link_7_mesh" value="hand_3finger" />
-    <property name="joint_base" value="${prefix}_joint_base" />
+    <property name="joint_base" value="joint_base" />
     <property name="joint_base_type" value="fixed" />
     <property name="joint_base_axis_xyz" value="0 0 0" />
     <property name="joint_base_origin_xyz" value="0 0 0" />
     <property name="joint_base_origin_rpy" value="0 0 0" />
-    <property name="joint_1" value="${prefix}_joint_1" />
+    <property name="joint_1" value="joint_1" />
     <property name="joint_1_type" value="continuous" />
     <property name="joint_1_axis_xyz" value="0 0 1" />
@@ -46,5 +36,5 @@
     <property name="joint_1_lower_limit" value="${-2*J_PI}" />
     <property name="joint_1_upper_limit" value="${2*J_PI}" />
-    <property name="joint_2" value="${prefix}_joint_2" />
+    <property name="joint_2" value="joint_2" />
     <property name="joint_2_type" value="revolute" />
     <property name="joint_2_axis_xyz" value="0 0 1" />
@@ -53,5 +43,5 @@
     <property name="joint_2_lower_limit" value="${30/180*J_PI}" />
     <property name="joint_2_upper_limit" value="${330/180*J_PI}" />
-    <property name="joint_3" value="${prefix}_joint_3" />
+    <property name="joint_3" value="joint_3" />
     <property name="joint_3_type" value="continuous" />
     <property name="joint_3_axis_xyz" value="0 0 1" />
@@ -60,5 +50,5 @@
     <property name="joint_3_lower_limit" value="${-2*J_PI}" />
     <property name="joint_3_upper_limit" value="${2*J_PI}" />
-    <property name="joint_4" value="${prefix}_joint_4" />
+    <property name="joint_4" value="joint_4" />
     <property name="joint_4_type" value="revolute" />
     <property name="joint_4_axis_xyz" value="0 0 1" />
@@ -67,5 +57,5 @@
     <property name="joint_4_lower_limit" value="${30/180*J_PI}" />
     <property name="joint_4_upper_limit" value="${330/180*J_PI}" />
-    <property name="joint_5" value="${prefix}_joint_5" />
+    <property name="joint_5" value="joint_5" />
     <property name="joint_5_type" value="continuous" />
     <property name="joint_5_axis_xyz" value="0 0 1" />
@@ -74,5 +64,5 @@
     <property name="joint_5_lower_limit" value="${-2*J_PI}" />
     <property name="joint_5_upper_limit" value="${2*J_PI}" />
-    <property name="joint_6" value="${prefix}_joint_6" />
+    <property name="joint_6" value="joint_6" />
     <property name="joint_6_type" value="revolute" />
     <property name="joint_6_axis_xyz" value="0 0 1" />
@@ -81,5 +71,5 @@
     <property name="joint_6_lower_limit" value="${30/180*J_PI}" />
     <property name="joint_6_upper_limit" value="${330/180*J_PI}" />
-    <property name="joint_7" value="${prefix}_joint_7" />
+    <property name="joint_7" value="joint_7" />
     <property name="joint_7_type" value="continuous" />
     <property name="joint_7_axis_xyz" value="0 0 1" />
@@ -88,29 +78,29 @@
     <property name="joint_7_lower_limit" value="${-2*J_PI}" />
     <property name="joint_7_upper_limit" value="${2*J_PI}" />
-    <property name="joint_end_effector" value="${prefix}_end_effector_offset" />
+    <property name="joint_end_effector" value="end_effector_offset" />
     <property name="joint_end_effector_type" value="fixed" />
     <property name="joint_end_effector_axis_xyz" value="0 0 0" />
     <property name="joint_end_effector_origin_xyz" value="0 0 -0.1600" />
     <property name="joint_end_effector_origin_rpy" value="${J_PI} 0 0" />
-    <xacro:macro name="j2s7s300" params="base_parent">
-        <xacro:kinova_armlink link_name="${link_base}" link_mesh="${link_base_mesh}"/>
-        <xacro:kinova_armjoint joint_name="${joint_base}" type="${joint_base_type}" parent="${base_parent}" child="${link_base}" joint_axis_xyz="${joint_base_axis_xyz}" joint_origin_xyz="${joint_base_origin_xyz}" joint_origin_rpy="${joint_base_origin_rpy}" joint_lower_limit="0" joint_upper_limit="0"/>
-        <xacro:kinova_armlink link_name="${link_1}" link_mesh="${link_1_mesh}" use_ring_mesh="true"/>
-        <xacro:kinova_armjoint joint_name="${joint_1}" type="${joint_1_type}" parent="${link_base}" child="${link_1}" joint_axis_xyz="${joint_1_axis_xyz}" joint_origin_xyz="${joint_1_origin_xyz}" joint_origin_rpy="${joint_1_origin_rpy}" joint_lower_limit="${joint_1_lower_limit}" joint_upper_limit="${joint_1_upper_limit}"/>
-        <xacro:kinova_armlink link_name="${link_2}" link_mesh="${link_2_mesh}" use_ring_mesh="true"/>
+    <xacro:macro name="j2s7s300" params="base_parent prefix:=${j2s7s300_}">
+        <xacro:kinova_armlink link_name="${prefixlink_base}" link_mesh="${link_base_mesh}"/>
+        <xacro:kinova_armjoint joint_name="${prefixjoint_base}" type="${joint_base_type}" parent="${base_parent}" child="${link_base}" joint_axis_xyz="${joint_base_axis_xyz}" joint_origin_xyz="${joint_base_origin_xyz}" joint_origin_rpy="${joint_base_origin_rpy}" joint_lower_limit="0" joint_upper_limit="0"/>
+        <xacro:kinova_armlink link_name="${prefixlink_1}" link_mesh="${link_1_mesh}" use_ring_mesh="true"/>
+        <xacro:kinova_armjoint joint_name="${prefixjoint_1}" type="${joint_1_type}" parent="${link_base}" child="${link_1}" joint_axis_xyz="${joint_1_axis_xyz}" joint_origin_xyz="${joint_1_origin_xyz}" joint_origin_rpy="${joint_1_origin_rpy}" joint_lower_limit="${joint_1_lower_limit}" joint_upper_limit="${joint_1_upper_limit}"/>
+        <xacro:kinova_armlink link_name="${prefixlink_2}" link_mesh="${link_2_mesh}" use_ring_mesh="true"/>
         <xacro:kinova_armjoint joint_name="${joint_2}" type="${joint_2_type}" parent="${link_1}" child="${link_2}" joint_axis_xyz="${joint_2_axis_xyz}" joint_origin_xyz="${joint_2_origin_xyz}" joint_origin_rpy="${joint_2_origin_rpy}" joint_lower_limit="${joint_2_lower_limit}" joint_upper_limit="${joint_2_upper_limit}"/>
-        <xacro:kinova_armlink link_name="${link_3}" link_mesh="${link_3_mesh}" use_ring_mesh="true"/>
-        <xacro:kinova_armjoint joint_name="${joint_3}" type="${joint_3_type}" parent="${link_2}" child="${link_3}" joint_axis_xyz="${joint_3_axis_xyz}" joint_origin_xyz="${joint_3_origin_xyz}" joint_origin_rpy="${joint_3_origin_rpy}" joint_lower_limit="${joint_3_lower_limit}" joint_upper_limit="${joint_3_upper_limit}"/>
-        <xacro:kinova_armlink link_name="${link_4}" link_mesh="${link_4_mesh}" use_ring_mesh="true"/>
-        <xacro:kinova_armjoint joint_name="${joint_4}" type="${joint_4_type}" parent="${link_3}" child="${link_4}" joint_axis_xyz="${joint_4_axis_xyz}" joint_origin_xyz="${joint_4_origin_xyz}" joint_origin_rpy="${joint_4_origin_rpy}" joint_lower_limit="${joint_4_lower_limit}" joint_upper_limit="${joint_4_upper_limit}"/>
-        <xacro:kinova_armlink link_name="${link_5}" link_mesh="${link_5_mesh}" use_ring_mesh="true" ring_mesh="ring_small"/>
-        <xacro:kinova_armjoint joint_name="${joint_5}" type="${joint_5_type}" parent="${link_4}" child="${link_5}" joint_axis_xyz="${joint_5_axis_xyz}" joint_origin_xyz="${joint_5_origin_xyz}" joint_origin_rpy="${joint_5_origin_rpy}" joint_lower_limit="${joint_5_lower_limit}" joint_upper_limit="${joint_5_upper_limit}"/>
-        <xacro:kinova_armlink link_name="${link_6}" link_mesh="${link_6_mesh}" use_ring_mesh="true" ring_mesh="ring_small"/>
-        <xacro:kinova_armjoint joint_name="${joint_6}" type="${joint_6_type}" parent="${link_5}" child="${link_6}" joint_axis_xyz="${joint_6_axis_xyz}" joint_origin_xyz="${joint_6_origin_xyz}" joint_origin_rpy="${joint_6_origin_rpy}" joint_lower_limit="${joint_6_lower_limit}" joint_upper_limit="${joint_6_upper_limit}"/>
-        <xacro:kinova_armlink link_name="${link_7}" link_mesh="${link_7_mesh}" use_ring_mesh="true" ring_mesh="ring_small"/>
-        <xacro:kinova_armjoint joint_name="${joint_7}" type="${joint_7_type}" parent="${link_6}" child="${link_7}" joint_axis_xyz="${joint_7_axis_xyz}" joint_origin_xyz="${joint_7_origin_xyz}" joint_origin_rpy="${joint_7_origin_rpy}" joint_lower_limit="${joint_7_lower_limit}" joint_upper_limit="${joint_7_upper_limit}"/>
-        <xacro:kinova_virtual_link link_name="${link_end_effector}"/>
-        <xacro:kinova_virtual_joint joint_name="${joint_end_effector}" type="${joint_end_effector_type}" parent="${link_7}" child="${link_end_effector}" joint_axis_xyz="${joint_end_effector_axis_xyz}" joint_origin_xyz="${joint_end_effector_origin_xyz}" joint_origin_rpy="${joint_end_effector_origin_rpy}" joint_lower_limit="0" joint_upper_limit="0"/>
+        <xacro:kinova_armlink link_name="${prefixlink_3}" link_mesh="${link_3_mesh}" use_ring_mesh="true"/>
+        <xacro:kinova_armjoint joint_name="${prefixjoint_3}" type="${joint_3_type}" parent="${link_2}" child="${link_3}" joint_axis_xyz="${joint_3_axis_xyz}" joint_origin_xyz="${joint_3_origin_xyz}" joint_origin_rpy="${joint_3_origin_rpy}" joint_lower_limit="${joint_3_lower_limit}" joint_upper_limit="${joint_3_upper_limit}"/>
+        <xacro:kinova_armlink link_name="${prefixlink_4}" link_mesh="${link_4_mesh}" use_ring_mesh="true"/>
+        <xacro:kinova_armjoint joint_name="${prefixjoint_4}" type="${joint_4_type}" parent="${link_3}" child="${link_4}" joint_axis_xyz="${joint_4_axis_xyz}" joint_origin_xyz="${joint_4_origin_xyz}" joint_origin_rpy="${joint_4_origin_rpy}" joint_lower_limit="${joint_4_lower_limit}" joint_upper_limit="${joint_4_upper_limit}"/>
+        <xacro:kinova_armlink link_name="${prefixlink_5}" link_mesh="${link_5_mesh}" use_ring_mesh="true" ring_mesh="ring_small"/>
+        <xacro:kinova_armjoint joint_name="${prefixjoint_5}" type="${joint_5_type}" parent="${link_4}" child="${link_5}" joint_axis_xyz="${joint_5_axis_xyz}" joint_origin_xyz="${joint_5_origin_xyz}" joint_origin_rpy="${joint_5_origin_rpy}" joint_lower_limit="${joint_5_lower_limit}" joint_upper_limit="${joint_5_upper_limit}"/>
+        <xacro:kinova_armlink link_name="${prefixlink_6}" link_mesh="${link_6_mesh}" use_ring_mesh="true" ring_mesh="ring_small"/>
+        <xacro:kinova_armjoint joint_name="${prefixjoint_6}" type="${joint_6_type}" parent="${link_5}" child="${link_6}" joint_axis_xyz="${joint_6_axis_xyz}" joint_origin_xyz="${joint_6_origin_xyz}" joint_origin_rpy="${joint_6_origin_rpy}" joint_lower_limit="${joint_6_lower_limit}" joint_upper_limit="${joint_6_upper_limit}"/>
+        <xacro:kinova_armlink link_name="${prefixlink_7}" link_mesh="${link_7_mesh}" use_ring_mesh="true" ring_mesh="ring_small"/>
+        <xacro:kinova_armjoint joint_name="${prefixjoint_7}" type="${joint_7_type}" parent="${link_6}" child="${link_7}" joint_axis_xyz="${joint_7_axis_xyz}" joint_origin_xyz="${joint_7_origin_xyz}" joint_origin_rpy="${joint_7_origin_rpy}" joint_lower_limit="${joint_7_lower_limit}" joint_upper_limit="${joint_7_upper_limit}"/>
+        <xacro:kinova_virtual_link link_name="${prefixlink_end_effector}"/>
+        <xacro:kinova_virtual_joint joint_name="${prefixjoint_end_effector}" type="${joint_end_effector_type}" parent="${link_7}" child="${link_end_effector}" joint_axis_xyz="${joint_end_effector_axis_xyz}" joint_origin_xyz="${joint_end_effector_origin_xyz}" joint_origin_rpy="${joint_end_effector_origin_rpy}" joint_lower_limit="0" joint_upper_limit="0"/>
     </xacro:macro>
-    <xacro:kinova_3fingers link_hand="${link_7}" prefix="${prefix}"/>
+    <xacro:kinova_3fingers link_hand="link_7" prefix="${prefix}"/>
 </root>

File: kinova_description/urdf/two_arm_robot_example_for_moveIt.xacro (robot description, xacro)
@@ -14,5 +14,5 @@
     xmlns:physics="http://playerstage.sourceforge.net/gazebo/xmlschema/#physics"
 	xmlns:xacro="http://ros.org/wiki/xacro" name="j2s6a300">
-  <xacro:include filename="$(find kinova_description)/urdf/j2s6a300.xacro"/>
+  <xacro:include filename="$(find kinova_description)/urdf/j2n6s300.xacro"/>
   <link name="root">
     <visual>
@@ -21,5 +21,4 @@
         <box size = "0 0 0"/>
       </geometry>
-    <!--<material name="Black" /> -->
     </visual>
     <collision>
@@ -31,4 +30,5 @@
   </link>
   <property name="robot_root" value="root" />
-  <xacro:j2s6a300  base_parent="${robot_root}"/>
+  <xacro:j2s6a300  base_parent="${robot_root}" prefix="left_"/>
+	<xacro:j2s6a300  base_parent="${robot_root}" prefix="right_"/>
 </robot>

Commit message: bugfix for inertial values
bugfix for inertial values
joint damping set to 0, was causing the robot to go unstable

File: kinova_description/urdf/j2n7s300.xacro (robot description, xacro)
@@ -36,5 +36,5 @@
     <property name="link_2_mesh_no" value="6" />
     <property name="link_3_mesh_no" value="7" />
-    <property name="link_4_mesh_no" value="4" />
+    <property name="link_4_mesh_no" value="3" />
     <property name="link_5_mesh_no" value="4" />
     <property name="link_6_mesh_no" value="4" />

File: kinova_description/urdf/j2s7s300.xacro (robot description, xacro)
@@ -36,5 +36,5 @@
     <property name="link_2_mesh_no" value="6" />
     <property name="link_3_mesh_no" value="7" />
-    <property name="link_4_mesh_no" value="4" />
+    <property name="link_4_mesh_no" value="3" />
     <property name="link_5_mesh_no" value="8" />
     <property name="link_6_mesh_no" value="9" />

File: kinova_description/urdf/kinova_common.xacro (robot description, xacro)
@@ -51,5 +51,5 @@
         <limit effort="2000" velocity="1" lower="${joint_lower_limit}" upper="${joint_upper_limit}"/>
         <origin xyz="${joint_origin_xyz}" rpy="${joint_origin_rpy}"/>
-        <dynamics damping="0.3" friction="0.0"/>
+        <dynamics damping="0.0" friction="0.0"/>
      </joint>
    <xacro:unless value="${fixed}">

File: kinova_description/urdf/kinova_inertial.xacro (robot description, xacro)
@@ -87,5 +87,5 @@
         <mass value="0.1785" />
         <origin xyz="0 -0.037 -0.0642" />
-        <xacro:inertia_cylinder height="0.1"  radius = "0.03" mass="0.1785"/>
+        <xacro:inertia_cylinder height="0.02"  radius = "0.04" mass="0.1785"/>
     </inertial>
   </xacro:unless>
@@ -95,5 +95,5 @@
         <mass value="0.85968" />
         <origin xyz="0 -0.145  -0.0076"/>
-        <xacro:inertia_cylinder height="0.3"  radius = "0.03" mass="0.85968"/>
+        <xacro:inertia_cylinder height="0.25"  radius = "0.03" mass="0.85968" axis="1"/>
     </inertial>
   </xacro:unless>
@@ -103,5 +103,5 @@
         <mass value="0.8447" />
         <origin xyz="0 -0.103563213 0" />
-        <xacro:inertia_cylinder height="0.2"  radius = "0.03" mass="0.8447"/>
+        <xacro:inertia_cylinder height="0.18"  radius = "0.03" mass="0.8447" axis="1"/>
     </inertial>
   </xacro:unless>
@@ -111,5 +111,5 @@
         <mass value="0.8447" />
         <origin xyz="0 0 -0.1022447445" />
-        <xacro:inertia_cylinder height="0.2"  radius = "0.03" mass="0.8447"/>
+        <xacro:inertia_cylinder height="0.18"  radius = "0.03" mass="0.8447"/>
     </inertial>
   </xacro:unless>
@@ -119,5 +119,5 @@
         <mass value="0.463" />
         <origin xyz="0 0.0028848942 -0.0541932613" />
-        <xacro:inertia_cylinder height="0.005"  radius = "0.02" mass="0.463"/>
+        <xacro:inertia_cylinder height="0.1"  radius = "0.02" mass="0.463"/>
     </inertial>
   </xacro:unless>
@@ -127,5 +127,5 @@
         <mass value="0.463" />
         <origin xyz="0 0.0497208855 -0.0028562765" />
-        <xacro:inertia_cylinder height="0.005"  radius = "0.02" mass="0.463"/>
+        <xacro:inertia_cylinder height="0.1"  radius = "0.02" mass="0.463" axis="1"/>
     </inertial>
   </xacro:unless>
@@ -135,5 +135,5 @@
         <mass value="0.606" />
         <origin xyz="0 0.0463 -0.0065" />
-        <xacro:inertia_cylinder height="0.005"  radius = "0.02" mass="0.606"/>
+        <xacro:inertia_cylinder height="0.08"  radius = "0.02" mass="0.606" axis="1"/>
     </inertial>
   </xacro:unless>
@@ -143,5 +143,5 @@
         <mass value="0.727" />
         <origin xyz="0 0 -0.06" />
-        <xacro:inertia_cylinder height="0.03"  radius = "0.1" mass="0.727"/>
+        <xacro:inertia_cylinder height="0.03"  radius = "0.04" mass="0.727"/>
     </inertial>
   </xacro:unless>
@@ -151,5 +151,5 @@
         <mass value="0.78" />
         <origin xyz="0 0 -0.06" />
-        <xacro:inertia_cylinder height="0.1"  radius = "0.1" mass="0.78"/>
+        <xacro:inertia_cylinder height="0.03"  radius = "0.04" mass="0.78"/>
     </inertial>
   </xacro:unless>
@@ -158,5 +158,5 @@
     <inertial>
         <mass value="0.01" />
-        <origin xyz="0 0 -0.15" />
+        <origin xyz="0.022 0 0" />
         <xacro:inertia_cylinder height="0.03"  radius = "0.004" mass="0.01"/>
     </inertial>
@@ -166,5 +166,5 @@
     <inertial>
         <mass value="0.01" />
-        <origin xyz="0 0 -0.15" />
+        <origin xyz="0.022 0 0" />
         <xacro:inertia_cylinder height="0.03"  radius = "0.004" mass="0.01"/>
     </inertial>
