Commit message: [kinova_description] j2s6s200: Change joint type to revolute for continuous joints with limits

File: kinova_description/urdf/j2s6s200.xacro (robot description, xacro)
@@ -44,5 +44,5 @@
     <xacro:property name="joint_base_origin_rpy" value="0 0 0" />
     <xacro:property name="joint_1" value="joint_1" />
-    <xacro:property name="joint_1_type" value="continuous" />
+    <xacro:property name="joint_1_type" value="revolute" />
     <xacro:property name="joint_1_axis_xyz" value="0 0 1" />
     <xacro:property name="joint_1_origin_xyz" value="0 0 0.15675" />
@@ -71,5 +71,5 @@
     <xacro:property name="joint_3_torque_limit" value="40" />
     <xacro:property name="joint_4" value="joint_4" />
-    <xacro:property name="joint_4_type" value="continuous" />
+    <xacro:property name="joint_4_type" value="revolute" />
     <xacro:property name="joint_4_axis_xyz" value="0 0 1" />
     <xacro:property name="joint_4_origin_xyz" value="0 0.2073 -0.0114" />
@@ -89,5 +89,5 @@
     <xacro:property name="joint_5_torque_limit" value="20" />
     <xacro:property name="joint_6" value="joint_6" />
-    <xacro:property name="joint_6_type" value="continuous" />
+    <xacro:property name="joint_6_type" value="revolute" />
     <xacro:property name="joint_6_axis_xyz" value="0 0 1" />
     <xacro:property name="joint_6_origin_xyz" value="0 0.10375 0" />

Commit message: Revert "[kinova_description] j2s6s200: Change joint type to revolute for continuous joints with limits"
This reverts commit e145ae8136cbe3dfedb9ddb26ffaeeec866b2a94.

File: kinova_description/urdf/j2s6s200.xacro (robot description, xacro)
@@ -44,5 +44,5 @@
     <xacro:property name="joint_base_origin_rpy" value="0 0 0" />
     <xacro:property name="joint_1" value="joint_1" />
-    <xacro:property name="joint_1_type" value="revolute" />
+    <xacro:property name="joint_1_type" value="continuous" />
     <xacro:property name="joint_1_axis_xyz" value="0 0 1" />
     <xacro:property name="joint_1_origin_xyz" value="0 0 0.15675" />
@@ -71,5 +71,5 @@
     <xacro:property name="joint_3_torque_limit" value="40" />
     <xacro:property name="joint_4" value="joint_4" />
-    <xacro:property name="joint_4_type" value="revolute" />
+    <xacro:property name="joint_4_type" value="continuous" />
     <xacro:property name="joint_4_axis_xyz" value="0 0 1" />
     <xacro:property name="joint_4_origin_xyz" value="0 0.2073 -0.0114" />
@@ -89,5 +89,5 @@
     <xacro:property name="joint_5_torque_limit" value="20" />
     <xacro:property name="joint_6" value="joint_6" />
-    <xacro:property name="joint_6_type" value="revolute" />
+    <xacro:property name="joint_6_type" value="continuous" />
     <xacro:property name="joint_6_axis_xyz" value="0 0 1" />
     <xacro:property name="joint_6_origin_xyz" value="0 0.10375 0" />
