Commit message: create finger macro (finger and tip) in kinova_common

File: kinova_description/urdf/kinova_common.xacro (robot description, xacro)
@@ -65,21 +65,21 @@
      </joint>
     </xacro:macro>
-    <xacro:macro name="kinova_finger" params="joint_name type parent joint_axis_xyz joint_origin_xyz joint_origin_rpy lower_limit upper_limit lower_limit_tip upper_limit_tip mimic_joint mimic_multiplier mimic_offset">
-        <LINK />
-        <joint name="${joint_name}" type="${type}">
-            <parent link="${parent}"/>
-            <child link="${child}"/>
-            <axis xyz="${joint_axis_xyz}"/>
-            <origin xyz="${joint_origin_xyz}" rpy="${joint_origin_rpy}"/>
-            <limit lower="${lower_limit}" upper="${upper_limit}" effort="30" velocity="5"/>
+    <xacro:macro name="kinova_finger" params="prefix finger_number hand finger_origin_xyz finger_origin_rpy">
+        <xacro:kinova_armlink link_name="${prefix}_finger_link_${finger_number}" link_mesh="finger_proximal"/>
+        <joint name="${prefix}_finger_joint_${finger_number}" type="revolute">
+            <parent link="${hand}"/>
+            <child link="${prefix}_finger_link_${finger_number}"/>
+            <axis xyz="0 0 1"/>
+            <origin xyz="${finger_origin_xyz}" rpy="${finger_origin_rpy}"/>
+            <limit lower="0" upper="2" effort="30" velocity="5"/>
         </joint>
-        <LINK />
-        <joint name="${joint_name}" type="${type}">
-            <parent link="${parent}"/>
-            <child link="${child}"/>
-            <axis xyz="${joint_axis_xyz}"/>
-            <origin xyz="${joint_origin_xyz}" rpy="${joint_origin_rpy}"/>
-            <limit lower="${lower_limit_tip}" upper="${upper_limit_tip}" effort="30" velocity="5"/>
-            <mimic joint="${mimic_joint}" multiplier="${mimic_multiplier}" offset="${mimic_offset}"/>
+        <xacro:kinova_armlink link_name="${prefix}_finger_tip_link_${finger_number}" link_mesh="finger_distal"/>
+        <joint name="${prefix}_finger_tip_joint_${finger_number}" type="revolute">
+            <parent link="${prefix}_finger_link_${finger_number}"/>
+            <child link="${prefix}_finger_tip_link_${finger_number}"/>
+            <axis xyz="0 0 1"/>
+            <origin xyz="0.044 -0.003 0" rpy="0 0 0"/>
+            <limit lower="0" upper="2" effort="30" velocity="5"/>
+            <!-- <mimic joint="${J_PI/180*40}" multiplier="1.0" offset="0.0"/> -->
         </joint>
     </xacro:macro>

Commit message: show jan6a300 in kinova_robot.launch

File: kinova_description/urdf/kinova_common.xacro (robot description, xacro)
@@ -66,20 +66,20 @@
     </xacro:macro>
     <xacro:macro name="kinova_finger" params="prefix finger_number hand finger_origin_xyz finger_origin_rpy">
-        <xacro:kinova_armlink link_name="${prefix}_finger_link_${finger_number}" link_mesh="finger_proximal"/>
-        <joint name="${prefix}_finger_joint_${finger_number}" type="revolute">
+        <xacro:kinova_armlink link_name="${prefix}_link_finger_${finger_number}" link_mesh="finger_proximal"/>
+        <joint name="${prefix}_joint_finger_${finger_number}" type="revolute">
             <parent link="${hand}"/>
-            <child link="${prefix}_finger_link_${finger_number}"/>
+            <child link="${prefix}_link_finger_${finger_number}"/>
             <axis xyz="0 0 1"/>
             <origin xyz="${finger_origin_xyz}" rpy="${finger_origin_rpy}"/>
             <limit lower="0" upper="2" effort="30" velocity="5"/>
         </joint>
-        <xacro:kinova_armlink link_name="${prefix}_finger_tip_link_${finger_number}" link_mesh="finger_distal"/>
-        <joint name="${prefix}_finger_tip_joint_${finger_number}" type="revolute">
-            <parent link="${prefix}_finger_link_${finger_number}"/>
-            <child link="${prefix}_finger_tip_link_${finger_number}"/>
+        <xacro:kinova_armlink link_name="${prefix}_link_finger_tip_${finger_number}" link_mesh="finger_distal"/>
+        <joint name="${prefix}_joint_finger_tip_${finger_number}" type="fixed">
+            <parent link="${prefix}_link_finger_${finger_number}"/>
+            <child link="${prefix}_link_finger_tip_${finger_number}"/>
             <axis xyz="0 0 1"/>
             <origin xyz="0.044 -0.003 0" rpy="0 0 0"/>
             <limit lower="0" upper="2" effort="30" velocity="5"/>
-            <!-- <mimic joint="${J_PI/180*40}" multiplier="1.0" offset="0.0"/> -->
+            <mimic joint="${J_PI/180*40}" multiplier="1.0" offset="0.0"/>
         </joint>
     </xacro:macro>

Commit message: Added damping to joint
Added damping to joint

File: kinova_description/urdf/kinova_common.xacro (robot description, xacro)
@@ -51,5 +51,5 @@
         <limit effort="30" velocity="0.35" lower="${joint_lower_limit}" upper="${joint_upper_limit}"/>
         <origin xyz="${joint_origin_xyz}" rpy="${joint_origin_rpy}"/>
-        <dynamics damping="0.0" friction="0.0"/>
+        <dynamics damping="0.7" friction="0.0"/>
      </joint>
    <xacro:unless value="${fixed}">

Commit message: Added inertia parameters for 7dof robot
Added inertia parameters for 7dof robot
Fixed finger mesh model number

File: kinova_description/urdf/kinova_common.xacro (robot description, xacro)
@@ -90,5 +90,5 @@
     </xacro:macro>
     <xacro:macro name="kinova_finger" params="prefix finger_number hand finger_origin_xyz finger_origin_rpy">
-        <xacro:kinova_armlink link_name="${prefix}link_finger_${finger_number}" link_mesh="finger_proximal" mesh_no="1"/>
+        <xacro:kinova_armlink link_name="${prefix}link_finger_${finger_number}" link_mesh="finger_proximal" mesh_no="57"/>
         <joint name="${prefix}joint_finger_${finger_number}" type="revolute">
             <parent link="${hand}"/>

File: kinova_description/urdf/kinova_inertial.xacro (robot description, xacro)
@@ -55,5 +55,5 @@
         <mass value="0.46784" />
         <origin xyz="0 0 0.1255" rpy="0 0 0"/>
-        <xacro:inertia_cylinder height="0.15"  radius = "0.04" mass="0.46784"/>
+        <xacro:inertia_cylinder height="0.14"  radius = "0.04" mass="0.46784"/>
     </inertial>
   </xacro:unless>
@@ -63,5 +63,5 @@
         <mass value="0.7477" />
         <origin xyz="0 -0.002 -0.0605" />
-        <xacro:inertia_cylinder height="0.15"  radius = "0.04" mass="0.7477"/>
+        <xacro:inertia_cylinder height="0.14"  radius = "0.04" mass="0.7477"/>
     </inertial>
   </xacro:unless>
@@ -71,5 +71,5 @@
         <mass value="0.99" />
         <origin xyz="0 -0.2065 -0.01" />
-        <xacro:inertia_cylinder height="0.4"  radius = "0.04" mass="0.99" axis="1"/>
+        <xacro:inertia_cylinder height="0.35"  radius = "0.04" mass="0.99" axis="1"/>
     </inertial>
   </xacro:unless>
@@ -79,5 +79,5 @@
         <mass value="0.6763" />
         <origin xyz="0 0.081 -0.0086" />
-        <xacro:inertia_cylinder height="0.2"  radius = "0.03" mass="0.6763" axis="1"/>
+        <xacro:inertia_cylinder height="0.15"  radius = "0.03" mass="0.6763" axis="1"/>
     </inertial>
   </xacro:unless>
@@ -87,5 +87,5 @@
         <mass value="0.1785" />
         <origin xyz="0 -0.037 -0.0642" />
-        <xacro:inertia_cylinder height="0.06"  radius = "0.03" mass="0.1785"/>
+        <xacro:inertia_cylinder height="0.03"  radius = "0.03" mass="0.1785"/>
     </inertial>
   </xacro:unless>
@@ -93,9 +93,7 @@
   <xacro:unless value="${mesh_no-5}">
     <inertial>
-        <mass value="0.441232" />
-        <origin xyz="0 0 0" />
-        <inertia  ixx="0.000924"  ixy="0.000000"  ixz="-0.000294"
-                          iyx="0.000000"  iyy="0.001034"  iyz="0.000000"
-                          izx="-0.000294"  izy="0.000000"  izz="0.000312" />
+        <mass value="0.85968" />
+        <origin xyz="0 -0.145  -0.1043782058" />
+        <xacro:inertia_cylinder height="0.3"  radius = "0.03" mass="0.85968"/>
     </inertial>
   </xacro:unless>
@@ -103,9 +101,7 @@
   <xacro:unless value="${mesh_no-6}">
     <inertial>
-        <mass value="0.441232" />
-        <origin xyz="0 0 0" />
-        <inertia  ixx="0.000924"  ixy="0.000000"  ixz="-0.000294"
-                          iyx="0.000000"  iyy="0.001034"  iyz="0.000000"
-                          izx="-0.000294"  izy="0.000000"  izz="0.000312" />
+        <mass value="0.8447" />
+        <origin xyz="0 -0.103563213 0" />
+        <xacro:inertia_cylinder height="0.2"  radius = "0.03" mass="0.8447"/>
     </inertial>
   </xacro:unless>
@@ -113,9 +109,7 @@
   <xacro:unless value="${mesh_no-7}">
     <inertial>
-        <mass value="0.441232" />
-        <origin xyz="0 0 0" />
-        <inertia  ixx="0.000924"  ixy="0.000000"  ixz="-0.000294"
-                          iyx="0.000000"  iyy="0.001034"  iyz="0.000000"
-                          izx="-0.000294"  izy="0.000000"  izz="0.000312" />
+        <mass value="0.8447" />
+        <origin xyz="0 0 -0.1022447445" />
+        <xacro:inertia_cylinder height="0.2"  radius = "0.03" mass="0.8447"/>
     </inertial>
   </xacro:unless>
@@ -123,9 +117,7 @@
   <xacro:unless value="${mesh_no-8}">
     <inertial>
-        <mass value="0.441232" />
-        <origin xyz="0 0 0" />
-        <inertia  ixx="0.000924"  ixy="0.000000"  ixz="-0.000294"
-                          iyx="0.000000"  iyy="0.001034"  iyz="0.000000"
-                          izx="-0.000294"  izy="0.000000"  izz="0.000312" />
+        <mass value="0.463" />
+        <origin xyz="0 0.0028848942 -0.0541932613" />
+        <xacro:inertia_cylinder height="0.005"  radius = "0.02" mass="0.463"/>
     </inertial>
   </xacro:unless>
@@ -133,9 +125,7 @@
   <xacro:unless value="${mesh_no-9}">
     <inertial>
-        <mass value="0.441232" />
-        <origin xyz="0 0 0" />
-        <inertia  ixx="0.000924"  ixy="0.000000"  ixz="-0.000294"
-                          iyx="0.000000"  iyy="0.001034"  iyz="0.000000"
-                          izx="-0.000294"  izy="0.000000"  izz="0.000312" />
+        <mass value="0.463" />
+        <origin xyz="0 0.0497208855 -0.0028562765" />
+        <xacro:inertia_cylinder height="0.005"  radius = "0.02" mass="0.463"/>
     </inertial>
   </xacro:unless>
@@ -144,16 +134,14 @@
     <inertial>
         <mass value="0.727" />
-        <origin xyz="0 -0.004029 -0.059694" />
-        <xacro:inertia_cylinder height="0.05"  radius = "0.04" mass="0.727"/>
+        <origin xyz="0 0 -0.06" />
+        <xacro:inertia_cylinder height="0.02"  radius = "0.06" mass="0.727"/>
     </inertial>
   </xacro:unless>
   <!-- hand 2 finger = 56 -->
   <xacro:unless value="${mesh_no - 56}">
-    <inertial>
-        <mass value="0.363290" />
-        <origin xyz="0 0 0" />
-        <inertia  ixx="0.001908"  ixy="0.000000"  ixz="0.000000"
-                          iyx="0.000000"  iyy="0.001907"  iyz="0.000000"
-                          izx="0.000000"  izy="0.000001"  izz="0.000209" />
+   <inertial>
+        <mass value="0.48" />
+        <origin xyz="0 0 -0.06" />
+        <xacro:inertia_cylinder height="0.02"  radius = "0.06" mass="0.48"/>
     </inertial>
   </xacro:unless>
@@ -162,6 +150,6 @@
     <inertial>
         <mass value="0.01" />
-        <origin xyz="0 0 0" />
-        <xacro:inertia_cylinder height="0.05"  radius = "0.004" mass="0.01"/>
+        <origin xyz="0 0 -0.15" />
+        <xacro:inertia_cylinder height="0.03"  radius = "0.004" mass="0.01"/>
     </inertial>
   </xacro:unless>
@@ -170,6 +158,6 @@
     <inertial>
         <mass value="0.01" />
-        <origin xyz="0 0 0" />
-        <xacro:inertia_cylinder height="0.05"  radius = "0.004" mass="0.01"/>
+        <origin xyz="0 0 -0.15" />
+        <xacro:inertia_cylinder height="0.03"  radius = "0.004" mass="0.01"/>
     </inertial>
   </xacro:unless>

Commit message: Changed control parameters to make the robot more stiff
Changed control parameters to make the robot more stiff

File: kinova_description/urdf/kinova_common.xacro (robot description, xacro)
@@ -49,7 +49,7 @@
         <child link="${child}"/>
         <axis xyz="${joint_axis_xyz}"/>
-        <limit effort="60" velocity="0.35" lower="${joint_lower_limit}" upper="${joint_upper_limit}"/>
+        <limit effort="2000" velocity="1" lower="${joint_lower_limit}" upper="${joint_upper_limit}"/>
         <origin xyz="${joint_origin_xyz}" rpy="${joint_origin_rpy}"/>
-        <dynamics damping="0.7" friction="0.0"/>
+        <dynamics damping="0.3" friction="0.0"/>
      </joint>
    <xacro:unless value="${fixed}">
@@ -85,5 +85,5 @@
         <child link="${child}"/>
         <axis xyz="${joint_axis_xyz}"/>
-        <limit effort="60" velocity="0.35" lower="${joint_lower_limit}" upper="${joint_upper_limit}"/>
+        <limit effort="2000" velocity="1" lower="${joint_lower_limit}" upper="${joint_upper_limit}"/>
         <origin xyz="${joint_origin_xyz}" rpy="${joint_origin_rpy}"/>
      </joint>
@@ -96,5 +96,5 @@
             <axis xyz="0 0 1"/>
             <origin xyz="${finger_origin_xyz}" rpy="${finger_origin_rpy}"/>
-            <limit lower="0" upper="2" effort="60" velocity="5"/>
+            <limit lower="0" upper="2" effort="2000" velocity="1"/>
         </joint>
 		    <transmission name="${prefix}joint_finger_${finger_number}_trans">
@@ -114,5 +114,5 @@
             <axis xyz="0 0 1"/>
             <origin xyz="0.044 -0.003 0" rpy="0 0 0"/>
-            <limit lower="0" upper="2" effort="60" velocity="5"/>
+            <limit lower="0" upper="2" effort="2000" velocity="1"/>
         </joint>
     </xacro:macro>
