Commit message: Removed erroneous macros and updated m1n6s200 gripper definition

File: kinova_description/urdf/kinova_common.xacro (robot description, xacro)
@@ -14,5 +14,5 @@
 	xmlns:xacro="http://ros.org/wiki/xacro">
 <xacro:include filename="$(find kinova_description)/urdf/kinova_inertial.xacro" />
-    <property name="J_PI" value="3.1415926535897931" />
+    <xacro:property name="J_PI" value="3.1415926535897931" />
     <xacro:macro name="kinova_armlink" params="link_name link_mesh ring_mesh:=ring_big use_ring_mesh:=false mesh_no">
         <link name="${link_name}">
@@ -89,31 +89,3 @@
      </joint>
     </xacro:macro>
-    <xacro:macro name="kinova_finger" params="prefix finger_number hand finger_origin_xyz finger_origin_rpy">
-        <xacro:kinova_armlink link_name="${prefix}link_finger_${finger_number}" link_mesh="finger_proximal" mesh_no="57"/>
-        <joint name="${prefix}joint_finger_${finger_number}" type="revolute">
-            <parent link="${hand}"/>
-            <child link="${prefix}link_finger_${finger_number}"/>
-            <axis xyz="0 0 1"/>
-            <origin xyz="${finger_origin_xyz}" rpy="${finger_origin_rpy}"/>
-            <limit lower="0" upper="2" effort="2000" velocity="1"/>
-        </joint>
-		    <transmission name="${prefix}joint_finger_${finger_number}_trans">
-					<type>transmission_interface/SimpleTransmission</type>
-					<joint name="${prefix}joint_finger_${finger_number}">
-					  <hardwareInterface>EffortJointInterface</hardwareInterface>
-					</joint>
-					<actuator name="${prefix}joint_finger_${finger_number}_actuator">
-					<hardwareInterface>EffortJointInterface</hardwareInterface>
-					<mechanicalReduction>1</mechanicalReduction>
-					</actuator>
-		    </transmission>
-        <xacro:kinova_armlink link_name="${prefix}link_finger_tip_${finger_number}" link_mesh="finger_distal" mesh_no="58"/>
-        <joint name="${prefix}joint_finger_tip_${finger_number}" type="fixed">
-            <parent link="${prefix}link_finger_${finger_number}"/>
-            <child link="${prefix}link_finger_tip_${finger_number}"/>
-            <axis xyz="0 0 1"/>
-            <origin xyz="0.044 -0.003 0" rpy="0 0 0"/>
-            <limit lower="0" upper="2" effort="2000" velocity="1"/>
-        </joint>
-    </xacro:macro>
 </root>

File: kinova_description/urdf/kinova_finger_set.xacro (robot description, xacro)
@@ -24,8 +24,67 @@
     </xacro:macro>
     <xacro:macro name="kinova_2fingers" params="link_hand prefix">
-        <!-- finger1 Rot := Ry((1/2)*Pi) . Rx(Pi) . Rz(-52.8*((1/180)*Pi)) -->
-        <xacro:kinova_finger prefix="${prefix}" finger_number="1" hand="${link_hand}" finger_origin_xyz="-0.0025 0.03095 -0.11482" finger_origin_rpy="-1.570796327 .649262481663582 1.57079632679490"/>
-        <!-- finger2 Rot := Ry((1/2)*Pi) . Rz(-52.8*((1/180)*Pi))  -->
-        <xacro:kinova_finger prefix="${prefix}" finger_number="2" hand="${link_hand}" finger_origin_xyz="-0.0025 -0.03095 -0.11482" finger_origin_rpy="-1.570796327 .649262481663582 -1.57079632679490"/>
+                <!-- FINGER 1 -->
+                <!--<xacro:macro name="kinova_finger" params="prefix finger_number hand finger_origin_xyz finger_origin_rpy">-->
+                    <!-- finger1 Rot := Ry((1/2)*Pi) . Rx(Pi) . Rz(-52.8*((1/180)*Pi)) -->
+                    <!--<xacro:kinova_finger prefix="${prefix}" finger_number="1" hand="${link_hand}" finger_origin_xyz="-0.0025 0.03095 -0.11482" finger_origin_rpy="-1.570796327 .649262481663582 1.57079632679490"/>-->
+                    <xacro:kinova_armlink link_name="${prefix}link_finger_1" link_mesh="finger_proximal" mesh_no="57"/>
+                    <joint name="${prefix}joint_finger_1" type="revolute">
+                        <parent link="${link_hand}"/>
+                        <child link="${prefix}link_finger_1"/>
+                        <axis xyz="0 0 1"/>
+                        <origin xyz="-0.0025 0.03095 -0.11482" rpy="-1.570796327 .649262481663582 1.57079632679490"/>
+                        <limit lower="0" upper="2" effort="2000" velocity="1"/>
+                    </joint>
+                        <transmission name="${prefix}joint_finger_1_trans">
+                                <type>transmission_interface/SimpleTransmission</type>
+                                <joint name="${prefix}joint_finger_1">
+                                  <hardwareInterface>EffortJointInterface</hardwareInterface>
+                                </joint>
+                                <actuator name="${prefix}joint_finger_1_actuator">
+                                <hardwareInterface>EffortJointInterface</hardwareInterface>
+                                <mechanicalReduction>1</mechanicalReduction>
+                                </actuator>
+                        </transmission>
+                    <xacro:kinova_armlink link_name="${prefix}link_finger_tip_1" link_mesh="finger_distal" mesh_no="58"/>
+                    <joint name="${prefix}joint_finger_tip_1" type="fixed">
+                        <parent link="${prefix}link_finger_1"/>
+                        <child link="${prefix}link_finger_tip_1"/>
+                        <axis xyz="0 0 1"/>
+                        <origin xyz="0.044 -0.003 0" rpy="0 0 0"/>
+                        <limit lower="0" upper="2" effort="2000" velocity="1"/>
+                    </joint>
+                <!--</xacro:macro>-->
+                <!-- FINGER 2 -->
+               <!--<xacro:macro name="kinova_finger" params="prefix finger_number hand finger_origin_xyz finger_origin_rpy">-->
+                    <!-- finger2 Rot := Ry((1/2)*Pi) . Rz(-52.8*((1/180)*Pi))  -->
+                    <!--<xacro:kinova_finger prefix="${prefix}" finger_number="2" hand="${link_hand}" finger_origin_xyz="-0.0025 -0.03095 -0.11482" finger_origin_rpy="-1.570796327 .649262481663582 -1.57079632679490"/>-->
+                    <xacro:kinova_armlink link_name="${prefix}link_finger_2" link_mesh="finger_proximal" mesh_no="57"/>
+                    <joint name="${prefix}joint_finger_2" type="revolute">
+                        <parent link="${link_hand}"/>
+                        <child link="${prefix}link_finger_2"/>
+                        <axis xyz="0 0 1"/>
+                        <mimic joint="${prefix}joint_finger_1" multiplier="1"/>
+                        <origin xyz="-0.0025 -0.03095 -0.11482" rpy="-1.570796327 .649262481663582 -1.57079632679490"/>
+                        <limit lower="0" upper="2" effort="2000" velocity="1"/>
+                    </joint>
+                        <transmission name="${prefix}joint_finger_2_trans">
+                                <type>transmission_interface/SimpleTransmission</type>
+                                <joint name="${prefix}joint_finger_2">
+                                  <hardwareInterface>EffortJointInterface</hardwareInterface>
+                                </joint>
+                                <actuator name="${prefix}joint_finger_2_actuator">
+                                <hardwareInterface>EffortJointInterface</hardwareInterface>
+                                <mechanicalReduction>1</mechanicalReduction>
+                                </actuator>
+                        </transmission>
+                    <xacro:kinova_armlink link_name="${prefix}link_finger_tip_2" link_mesh="finger_distal" mesh_no="58"/>
+                    <joint name="${prefix}joint_finger_tip_2" type="fixed">
+                        <parent link="${prefix}link_finger_2"/>
+                        <child link="${prefix}link_finger_tip_2"/>
+                        <axis xyz="0 0 1"/>
+                        <origin xyz="0.044 -0.003 0" rpy="0 0 0"/>
+                        <limit lower="0" upper="2" effort="2000" velocity="1"/>
+                    </joint>
+                <!--</xacro:macro>-->
     </xacro:macro>
 </root>

File: kinova_description/urdf/m1n6s200.xacro (robot description, xacro)
@@ -18,11 +18,11 @@
     <!-- Import all Gazebo-customization elements -->
     <xacro:include filename="$(find kinova_description)/urdf/kinova.gazebo" />
-    <property name="link_base_mesh" value="base" />
-    <property name="link_1_mesh" value="shoulder" />
-    <property name="link_2_mesh" value="arm_mico" />
-    <property name="link_3_mesh" value="forearm_mico" />
-    <property name="link_4_mesh" value="wrist" />
-    <property name="link_5_mesh" value="wrist" />
-    <property name="link_6_mesh" value="hand_2finger" />
+    <xacro:property name="link_base_mesh" value="base" />
+    <xacro:property name="link_1_mesh" value="shoulder" />
+    <xacro:property name="link_2_mesh" value="arm_mico" />
+    <xacro:property name="link_3_mesh" value="forearm_mico" />
+    <xacro:property name="link_4_mesh" value="wrist" />
+    <xacro:property name="link_5_mesh" value="wrist" />
+    <xacro:property name="link_6_mesh" value="hand_2finger" />
     <!--Used for conditional arguments for setting inertial parameters
         base 0, shoulder 1, arm 2, forearm 3, wrist 4, arm_mico 5,
@@ -31,63 +31,65 @@
         hand 3 finger 55, hand_2finger 56, finger_proximal 57, finger_distal 58
     -->
-    <property name="link_base_mesh_no" value="0" />
-    <property name="link_1_mesh_no" value="1" />
-    <property name="link_2_mesh_no" value="5" />
-    <property name="link_3_mesh_no" value="10" />
-    <property name="link_4_mesh_no" value="4" />
-    <property name="link_5_mesh_no" value="4" />
-    <property name="link_6_mesh_no" value="56" />
-    <property name="joint_base" value="joint_base" />
-    <property name="joint_base_type" value="fixed" />
-    <property name="joint_base_axis_xyz" value="0 0 0" />
-    <property name="joint_base_origin_xyz" value="0 0 0" />
-    <property name="joint_base_origin_rpy" value="0 0 0" />
-    <property name="joint_1" value="joint_1" />
-    <property name="joint_1_type" value="continuous" />
-    <property name="joint_1_axis_xyz" value="0 0 1" />
-    <property name="joint_1_origin_xyz" value="0 0 0.15675" />
-    <property name="joint_1_origin_rpy" value="0 ${J_PI} 0" />
-    <property name="joint_1_lower_limit" value="${-2*J_PI}" />
-    <property name="joint_1_upper_limit" value="${2*J_PI}" />
-    <property name="joint_2" value="joint_2" />
-    <property name="joint_2_type" value="revolute" />
-    <property name="joint_2_axis_xyz" value="0 0 1" />
-    <property name="joint_2_origin_xyz" value="0 0.0016 -0.11875" />
-    <property name="joint_2_origin_rpy" value="${-J_PI/2} 0 ${J_PI}" />
-    <property name="joint_2_lower_limit" value="${30/180*J_PI}" />
-    <property name="joint_2_upper_limit" value="${330/180*J_PI}" />
-    <property name="joint_3" value="joint_3" />
-    <property name="joint_3_type" value="revolute" />
-    <property name="joint_3_axis_xyz" value="0 0 1" />
-    <property name="joint_3_origin_xyz" value="0 -0.290 0" />
-    <property name="joint_3_origin_rpy" value="0 ${J_PI} 0" />
-    <property name="joint_3_lower_limit" value="${30/180*J_PI}" />
-    <property name="joint_3_upper_limit" value="${330/180*J_PI}" />
-    <property name="joint_4" value="joint_4" />
-    <property name="joint_4_type" value="continuous" />
-    <property name="joint_4_axis_xyz" value="0 0 1" />
-    <property name="joint_4_origin_xyz" value="0 0.1231 -0.0086" />
-    <property name="joint_4_origin_rpy" value="${-J_PI/2} 0 ${J_PI}" />
-    <property name="joint_4_lower_limit" value="${-2*J_PI}" />
-    <property name="joint_4_upper_limit" value="${2*J_PI}" />
-    <property name="joint_5" value="joint_5" />
-    <property name="joint_5_type" value="continuous" />
-    <property name="joint_5_axis_xyz" value="0 0 1" />
-    <property name="joint_5_origin_xyz" value="0 -0.03703 -0.06414" />
-    <property name="joint_5_origin_rpy" value="${J_PI/3} 0 ${J_PI}" />
-    <property name="joint_5_lower_limit" value="${-2*J_PI}" />
-    <property name="joint_5_upper_limit" value="${2*J_PI}" />
-    <property name="joint_6" value="joint_6" />
-    <property name="joint_6_type" value="continuous" />
-    <property name="joint_6_axis_xyz" value="0 0 1" />
-    <property name="joint_6_origin_xyz" value="0 -0.03703 -0.06414" />
-    <property name="joint_6_origin_rpy" value="${J_PI/3} 0 ${J_PI}" />
-    <property name="joint_6_lower_limit" value="${-2*J_PI}" />
-    <property name="joint_6_upper_limit" value="${2*J_PI}" />
-    <property name="joint_end_effector" value="end_effector_offset" />
-    <property name="joint_end_effector_type" value="fixed" />
-    <property name="joint_end_effector_axis_xyz" value="0 0 0" />
-    <property name="joint_end_effector_origin_xyz" value="0 0 -0.1600" />
-    <property name="joint_end_effector_origin_rpy" value="${J_PI} 0 0" />
+    <xacro:property name="link_base_mesh_no" value="0" />
+    <xacro:property name="link_1_mesh_no" value="1" />
+    <xacro:property name="link_2_mesh_no" value="5" />
+    <xacro:property name="link_3_mesh_no" value="10" />
+    <xacro:property name="link_4_mesh_no" value="4" />
+    <xacro:property name="link_5_mesh_no" value="4" />
+    <xacro:property name="link_6_mesh_no" value="56" />
+    <xacro:property name="joint_base" value="joint_base" />
+    <xacro:property name="joint_base_type" value="fixed" />
+    <xacro:property name="joint_base_axis_xyz" value="0 0 0" />
+    <xacro:property name="joint_base_origin_xyz" value="0 0 0" />
+    <xacro:property name="joint_base_origin_rpy" value="0 0 0" />
+    <xacro:property name="joint_1" value="joint_1" />
+    <xacro:property name="joint_1_type" value="continuous" />
+    <xacro:property name="joint_1_axis_xyz" value="0 0 1" />
+    <xacro:property name="joint_1_origin_xyz" value="0 0 0.15675" />
+    <xacro:property name="joint_1_origin_rpy" value="0 ${J_PI} 0" />
+    <xacro:property name="joint_1_lower_limit" value="${-2*J_PI}" />
+    <xacro:property name="joint_1_upper_limit" value="${2*J_PI}" />
+    <xacro:property name="joint_2" value="joint_2" />
+    <xacro:property name="joint_2_type" value="revolute" />
+    <xacro:property name="joint_2_axis_xyz" value="0 0 1" />
+    <xacro:property name="joint_2_origin_xyz" value="0 0.0016 -0.11875" />
+    <xacro:property name="joint_2_origin_rpy" value="${-J_PI/2} 0 ${J_PI}" />
+    <xacro:property name="joint_2_lower_limit" value="${30/180*J_PI}" />
+    <xacro:property name="joint_2_upper_limit" value="${330/180*J_PI}" />
+    <xacro:property name="joint_3" value="joint_3" />
+    <xacro:property name="joint_3_type" value="revolute" />
+    <xacro:property name="joint_3_axis_xyz" value="0 0 1" />
+    <xacro:property name="joint_3_origin_xyz" value="0 -0.290 0" />
+    <xacro:property name="joint_3_origin_rpy" value="0 ${J_PI} 0" />
+    <xacro:property name="joint_3_lower_limit" value="${30/180*J_PI}" />
+    <xacro:property name="joint_3_upper_limit" value="${330/180*J_PI}" />
+    <xacro:property name="joint_4" value="joint_4" />
+    <xacro:property name="joint_4_type" value="continuous" />
+    <xacro:property name="joint_4_axis_xyz" value="0 0 1" />
+    <xacro:property name="joint_4_origin_xyz" value="0 0.1231 -0.0086" />
+    <xacro:property name="joint_4_origin_rpy" value="${-J_PI/2} 0 ${J_PI}" />
+    <xacro:property name="joint_4_lower_limit" value="${-2*J_PI}" />
+    <xacro:property name="joint_4_upper_limit" value="${2*J_PI}" />
+    <xacro:property name="joint_5" value="joint_5" />
+    <xacro:property name="joint_5_type" value="continuous" />
+    <xacro:property name="joint_5_axis_xyz" value="0 0 1" />
+    <xacro:property name="joint_5_origin_xyz" value="0 -0.03703 -0.06414" />
+    <xacro:property name="joint_5_origin_rpy" value="${J_PI/3} 0 ${J_PI}" />
+    <xacro:property name="joint_5_lower_limit" value="${-2*J_PI}" />
+    <xacro:property name="joint_5_upper_limit" value="${2*J_PI}" />
+    <xacro:property name="joint_6" value="joint_6" />
+    <xacro:property name="joint_6_type" value="continuous" />
+    <xacro:property name="joint_6_axis_xyz" value="0 0 1" />
+    <xacro:property name="joint_6_origin_xyz" value="0 -0.03703 -0.06414" />
+    <xacro:property name="joint_6_origin_rpy" value="${J_PI/3} 0 ${J_PI}" />
+    <xacro:property name="joint_6_lower_limit" value="${-2*J_PI}" />
+    <xacro:property name="joint_6_upper_limit" value="${2*J_PI}" />
+    <xacro:property name="joint_end_effector" value="end_effector_offset" />
+    <xacro:property name="joint_end_effector_type" value="fixed" />
+    <xacro:property name="joint_end_effector_axis_xyz" value="0 0 0" />
+    <!--<xacro:property name="joint_end_effector_origin_xyz" value="0 0 -0.1600" />-->
+    <xacro:property name="joint_end_effector_origin_xyz" value="0 0 0" />
+    <!--<xacro:property name="joint_end_effector_origin_rpy" value="${J_PI} 0 0" />-->
+    <xacro:property name="joint_end_effector_origin_rpy" value="0 0 0" />
     <xacro:macro name="m1n6s200" params="base_parent prefix:=m1n6s200">
         <xacro:gazebo_config robot_namespace="${prefix}"/>
@@ -104,9 +106,11 @@
         <xacro:kinova_armlink link_name="${prefix}_link_5" link_mesh="${link_5_mesh}" use_ring_mesh="true" ring_mesh="ring_small" mesh_no="${link_5_mesh_no}"/>
         <xacro:kinova_armjoint joint_name="${prefix}_joint_5" type="${joint_5_type}" parent="${prefix}_link_4" child="${prefix}_link_5" joint_axis_xyz="${joint_5_axis_xyz}" joint_origin_xyz="${joint_5_origin_xyz}" joint_origin_rpy="${joint_5_origin_rpy}" joint_lower_limit="${joint_5_lower_limit}" joint_upper_limit="${joint_5_upper_limit}"/>
+        <xacro:kinova_virtual_link link_name="${prefix}_end_effector"/>
+        <xacro:kinova_armjoint joint_name="${prefix}_joint_6" type="${joint_6_type}" parent="${prefix}_link_5" child="${prefix}_end_effector" joint_axis_xyz="${joint_6_axis_xyz}" joint_origin_xyz="${joint_6_origin_xyz}" joint_origin_rpy="${joint_6_origin_rpy}" joint_lower_limit="${joint_6_lower_limit}" joint_upper_limit="${joint_6_upper_limit}"/>
         <xacro:kinova_armlink link_name="${prefix}_link_6" link_mesh="${link_6_mesh}" use_ring_mesh="true" ring_mesh="ring_small" mesh_no="${link_6_mesh_no}"/>
-        <xacro:kinova_armjoint joint_name="${prefix}_joint_6" type="${joint_6_type}" parent="${prefix}_link_5" child="${prefix}_link_6" joint_axis_xyz="${joint_6_axis_xyz}" joint_origin_xyz="${joint_6_origin_xyz}" joint_origin_rpy="${joint_6_origin_rpy}" joint_lower_limit="${joint_6_lower_limit}" joint_upper_limit="${joint_6_upper_limit}"/>
-        <xacro:kinova_virtual_link link_name="${prefix}_end_effector"/>
-        <xacro:kinova_virtual_joint joint_name="${prefix}_joint_end_effector" type="${joint_end_effector_type}" parent="${prefix}_link_6" child="${prefix}_end_effector" joint_axis_xyz="${joint_end_effector_axis_xyz}" joint_origin_xyz="${joint_end_effector_origin_xyz}" joint_origin_rpy="${joint_end_effector_origin_rpy}" joint_lower_limit="0" joint_upper_limit="0"/>
-    <xacro:kinova_2fingers link_hand="${prefix}_link_6" prefix="${prefix}_"/>
+        <xacro:kinova_virtual_joint joint_name="${prefix}_joint_end_effector" type="${joint_end_effector_type}" parent="${prefix}_end_effector" child="${prefix}_link_6" joint_axis_xyz="${joint_end_effector_axis_xyz}" joint_origin_xyz="${joint_end_effector_origin_xyz}" joint_origin_rpy="${joint_end_effector_origin_rpy}" joint_lower_limit="0" joint_upper_limit="0"/>
+        <!--<xacro:kinova_armjoint joint_name="${prefix}_joint_6" type="${joint_6_type}" parent="${prefix}_link_5" child="${prefix}_link_6" joint_axis_xyz="${joint_6_axis_xyz}" joint_origin_xyz="${joint_6_origin_xyz}" joint_origin_rpy="${joint_6_origin_rpy}" joint_lower_limit="${joint_6_lower_limit}" joint_upper_limit="${joint_6_upper_limit}"/>-->
+        <!--<xacro:kinova_virtual_joint joint_name="${prefix}_joint_end_effector" type="${joint_end_effector_type}" parent="${prefix}_link_6" child="${prefix}_end_effector" joint_axis_xyz="${joint_end_effector_axis_xyz}" joint_origin_xyz="${joint_end_effector_origin_xyz}" joint_origin_rpy="${joint_end_effector_origin_rpy}" joint_lower_limit="0" joint_upper_limit="0"/>-->
+        <xacro:kinova_2fingers link_hand="${prefix}_link_6" prefix="${prefix}_"/>
     </xacro:macro>
 </root>

File: kinova_description/urdf/m1n6s200_standalone.xacro (robot description, xacro)
@@ -30,5 +30,5 @@
     </collision>
   </link>
-  <property name="robot_root" value="root" />
+  <xacro:property name="robot_root" value="root" />
   <xacro:m1n6s200  base_parent="${robot_root}"/>
 </robot>
