Commit message: Gear reduction ratios updated

File: kinova_description/urdf/kinova_common.xacro (robot description, xacro)
@@ -54,10 +54,10 @@
      </joint>
    <xacro:unless value="${fixed}">
-     <transmission name="${joint_name}_trans">
+     <transmission name="${prefix}_joint_1_trans">
         <type>transmission_interface/SimpleTransmission</type>
-        <joint name="${joint_name}">
+        <joint name="${prefix}_joint_1">
           <hardwareInterface>EffortJointInterface</hardwareInterface>
         </joint>
-        <actuator name="${joint_name}_actuator">
+        <actuator name="${prefix}_joint_1_actuator">
           <hardwareInterface>EffortJointInterface</hardwareInterface>
         <mechanicalReduction>160</mechanicalReduction>
@@ -66,14 +66,64 @@
      </xacro:unless>
   </xacro:macro>
+<transmission name="${prefix}_joint_2_trans">
+        <type>transmission_interface/SimpleTransmission</type>
+        <joint name="${prefix}_joint_2">
+          <hardwareInterface>EffortJointInterface</hardwareInterface>
+        </joint>
+        <actuator name="${prefix}_joint_2_actuator">
+          <hardwareInterface>EffortJointInterface</hardwareInterface>
+        <mechanicalReduction>160</mechanicalReduction>
+        </actuator>
+     </transmission>
+     <transmission name="${prefix}_joint_3_trans">
+        <type>transmission_interface/SimpleTransmission</type>
+        <joint name="${prefix}_joint_3">
+          <hardwareInterface>EffortJointInterface</hardwareInterface>
+        </joint>
+        <actuator name="${prefix}_joint_3_actuator">
+          <hardwareInterface>EffortJointInterface</hardwareInterface>
+        <mechanicalReduction>160</mechanicalReduction>
+        </actuator>
+     </transmission>
+     <transmission name="${prefix}_joint_4_trans">
+        <type>transmission_interface/SimpleTransmission</type>
+        <joint name="${prefix}_joint_4">
+          <hardwareInterface>EffortJointInterface</hardwareInterface>
+        </joint>
+        <actuator name="${prefix}_joint_4_actuator">
+          <hardwareInterface>EffortJointInterface</hardwareInterface>
+        <mechanicalReduction>110</mechanicalReduction>
+        </actuator>
+     </transmission>
+     <transmission name="${prefix}_joint_5_trans">
+        <type>transmission_interface/SimpleTransmission</type>
+        <joint name="${prefix}_joint_5">
+          <hardwareInterface>EffortJointInterface</hardwareInterface>
+        </joint>
+        <actuator name="${prefix}_joint_5_actuator">
+          <hardwareInterface>EffortJointInterface</hardwareInterface>
+        <mechanicalReduction>110</mechanicalReduction>
+        </actuator>
+     </transmission>
+     <transmission name="${prefix}_joint_6_trans">
+        <type>transmission_interface/SimpleTransmission</type>
+        <joint name="${prefix}_joint_6">
+          <hardwareInterface>EffortJointInterface</hardwareInterface>
+        </joint>
+        <actuator name="${prefix}_joint_6_actuator">
+          <hardwareInterface>EffortJointInterface</hardwareInterface>
+        <mechanicalReduction>110</mechanicalReduction>
+        </actuator>
+     </transmission>
     <xacro:macro name="kinova_virtual_link" params="link_name">
         <link name="${link_name}">
             <visual>
                 <geometry>
-                    <box size = "0 0 0"/>
+                    <box size = "0.00001 0.00001 0.00001"/>
                 </geometry>
             </visual>
             <collision>
                 <geometry>
-                    <box size = "0 0 0"/>
+                    <box size = "0.00001 0.00001 0.00001"/>
                 </geometry>
             </collision>

Commit message: Update kinova_common.xacro

File: kinova_description/urdf/kinova_common.xacro (robot description, xacro)
@@ -64,6 +64,4 @@
         </actuator>
      </transmission>
-     </xacro:unless>
-  </xacro:macro>
 <transmission name="${prefix}_joint_2_trans">
         <type>transmission_interface/SimpleTransmission</type>
@@ -116,4 +114,6 @@
         </actuator>
      </transmission>
+    </xacro:unless>
+  </xacro:macro>
     <xacro:macro name="kinova_virtual_link" params="link_name">
         <link name="${link_name}">

Commit message: Revert "Small changes  in the mass and transmission interface"

File: kinova_description/urdf/kinova_common.xacro (robot description, xacro)
@@ -54,65 +54,15 @@
      </joint>
    <xacro:unless value="${fixed}">
-     <transmission name="${prefix}_joint_1_trans">
+     <transmission name="${joint_name}_trans">
         <type>transmission_interface/SimpleTransmission</type>
-        <joint name="${prefix}_joint_1">
+        <joint name="${joint_name}">
           <hardwareInterface>EffortJointInterface</hardwareInterface>
         </joint>
-        <actuator name="${prefix}_joint_1_actuator">
+        <actuator name="${joint_name}_actuator">
           <hardwareInterface>EffortJointInterface</hardwareInterface>
         <mechanicalReduction>160</mechanicalReduction>
         </actuator>
      </transmission>
-<transmission name="${prefix}_joint_2_trans">
-        <type>transmission_interface/SimpleTransmission</type>
-        <joint name="${prefix}_joint_2">
-          <hardwareInterface>EffortJointInterface</hardwareInterface>
-        </joint>
-        <actuator name="${prefix}_joint_2_actuator">
-          <hardwareInterface>EffortJointInterface</hardwareInterface>
-        <mechanicalReduction>160</mechanicalReduction>
-        </actuator>
-     </transmission>
-     <transmission name="${prefix}_joint_3_trans">
-        <type>transmission_interface/SimpleTransmission</type>
-        <joint name="${prefix}_joint_3">
-          <hardwareInterface>EffortJointInterface</hardwareInterface>
-        </joint>
-        <actuator name="${prefix}_joint_3_actuator">
-          <hardwareInterface>EffortJointInterface</hardwareInterface>
-        <mechanicalReduction>160</mechanicalReduction>
-        </actuator>
-     </transmission>
-     <transmission name="${prefix}_joint_4_trans">
-        <type>transmission_interface/SimpleTransmission</type>
-        <joint name="${prefix}_joint_4">
-          <hardwareInterface>EffortJointInterface</hardwareInterface>
-        </joint>
-        <actuator name="${prefix}_joint_4_actuator">
-          <hardwareInterface>EffortJointInterface</hardwareInterface>
-        <mechanicalReduction>110</mechanicalReduction>
-        </actuator>
-     </transmission>
-     <transmission name="${prefix}_joint_5_trans">
-        <type>transmission_interface/SimpleTransmission</type>
-        <joint name="${prefix}_joint_5">
-          <hardwareInterface>EffortJointInterface</hardwareInterface>
-        </joint>
-        <actuator name="${prefix}_joint_5_actuator">
-          <hardwareInterface>EffortJointInterface</hardwareInterface>
-        <mechanicalReduction>110</mechanicalReduction>
-        </actuator>
-     </transmission>
-     <transmission name="${prefix}_joint_6_trans">
-        <type>transmission_interface/SimpleTransmission</type>
-        <joint name="${prefix}_joint_6">
-          <hardwareInterface>EffortJointInterface</hardwareInterface>
-        </joint>
-        <actuator name="${prefix}_joint_6_actuator">
-          <hardwareInterface>EffortJointInterface</hardwareInterface>
-        <mechanicalReduction>110</mechanicalReduction>
-        </actuator>
-     </transmission>
-    </xacro:unless>
+     </xacro:unless>
   </xacro:macro>
     <xacro:macro name="kinova_virtual_link" params="link_name">
@@ -120,10 +70,10 @@
             <visual>
                 <geometry>
-                    <box size = "0.00001 0.00001 0.00001"/>
+                    <box size = "0 0 0"/>
                 </geometry>
             </visual>
             <collision>
                 <geometry>
-                    <box size = "0.00001 0.00001 0.00001"/>
+                    <box size = "0 0 0"/>
                 </geometry>
             </collision>

File: kinova_description/urdf/kinova_inertial.xacro (robot description, xacro)
@@ -61,7 +61,7 @@
   <xacro:unless value="${mesh_no-1}">
     <inertial>
-        <mass value="0.7487" />
+        <mass value="0.7477" />
         <origin xyz="0 -0.002 -0.0605" />
-        <xacro:inertia_cylinder height="0.14"  radius = "0.04" mass="0.7487"/>
+        <xacro:inertia_cylinder height="0.14"  radius = "0.04" mass="0.7477"/>
     </inertial>
   </xacro:unless>
@@ -69,7 +69,7 @@
   <xacro:unless value="${mesh_no-2}">
     <inertial>
-        <mass value="0.9907" />
+        <mass value="0.99" />
         <origin xyz="0 -0.2065 -0.01" />
-        <xacro:inertia_cylinder height="0.35"  radius = "0.04" mass="0.9907" axis="1"/>
+        <xacro:inertia_cylinder height="0.35"  radius = "0.04" mass="0.99" axis="1"/>
     </inertial>
   </xacro:unless>
@@ -77,7 +77,7 @@
   <xacro:unless value="${mesh_no-3}">
     <inertial>
-        <mass value="0.6685" />
+        <mass value="0.6763" />
         <origin xyz="0 0.081 -0.0086" />
-        <xacro:inertia_cylinder height="0.15"  radius = "0.03" mass="0.6685" axis="1"/>
+        <xacro:inertia_cylinder height="0.15"  radius = "0.03" mass="0.6763" axis="1"/>
     </inertial>
   </xacro:unless>
@@ -87,5 +87,5 @@
         <mass value="0.426367" />
         <origin xyz="0 -0.037 -0.0642" />
-        <xacro:inertia_cylinder height="0.02"  radius = "0.04" mass="0.4104"/>
+        <xacro:inertia_cylinder height="0.02"  radius = "0.04" mass="0.1785"/>
     </inertial>
   </xacro:unless>
@@ -143,5 +143,5 @@
         <mass value="0.99" />
         <origin xyz="0 0 -0.06" />
-        <xacro:inertia_cylinder height="0.03"  radius = "0.04" mass="0.8977"/>
+        <xacro:inertia_cylinder height="0.03"  radius = "0.04" mass="0.727"/>
     </inertial>
   </xacro:unless>

Commit message: remove visual from virtual links

File: kinova_description/urdf/kinova_common.xacro (robot description, xacro)
@@ -67,16 +67,5 @@
   </xacro:macro>
     <xacro:macro name="kinova_virtual_link" params="link_name">
-        <link name="${link_name}">
-            <visual>
-                <geometry>
-                    <box size = "0 0 0"/>
-                </geometry>
-            </visual>
-            <collision>
-                <geometry>
-                    <box size = "0 0 0"/>
-                </geometry>
-            </collision>
-        </link>
+        <link name="${link_name}"/>
     </xacro:macro>
     <xacro:macro name="kinova_virtual_joint" params="joint_name type parent child joint_axis_xyz joint_origin_xyz joint_origin_rpy joint_lower_limit joint_upper_limit">

Commit message: make the finger tip a revolute joint

File: kinova_description/urdf/kinova_common.xacro (robot description, xacro)
@@ -98,5 +98,5 @@
 		    </transmission>
         <xacro:kinova_armlink link_name="${prefix}link_finger_tip_${finger_number}" link_mesh="finger_distal" mesh_no="58"/>
-        <joint name="${prefix}joint_finger_tip_${finger_number}" type="fixed">
+        <joint name="${prefix}joint_finger_tip_${finger_number}" type="revolute">
             <parent link="${prefix}link_finger_${finger_number}"/>
             <child link="${prefix}link_finger_tip_${finger_number}"/>

Commit message: Add transmission elements for finger tips for Gazebo simulation

File: kinova_description/urdf/kinova_common.xacro (robot description, xacro)
@@ -105,4 +105,14 @@
             <limit lower="0" upper="2" effort="2000" velocity="1"/>
         </joint>
+        <transmission name="${prefix}joint_finger_tip_${finger_number}_trans">
+					<type>transmission_interface/SimpleTransmission</type>
+					<joint name="${prefix}joint_finger_tip_${finger_number}">
+					  <hardwareInterface>hardware_interface/EffortJointInterface</hardwareInterface>
+					</joint>
+					<actuator name="${prefix}joint_finger_tip_${finger_number}_actuator">
+					<hardwareInterface>hardware_interface/EffortJointInterface</hardwareInterface>
+					<mechanicalReduction>1</mechanicalReduction>
+					</actuator>
+        </transmission>
     </xacro:macro>
 </root>

Commit message: Added better values for position limits for the fingers

File: kinova_description/urdf/kinova_common.xacro (robot description, xacro)
@@ -85,5 +85,5 @@
             <axis xyz="0 0 1"/>
             <origin xyz="${finger_origin_xyz}" rpy="${finger_origin_rpy}"/>
-            <limit lower="0" upper="2" effort="2000" velocity="1"/>
+            <limit lower="0" upper="1.51" effort="2000" velocity="1"/>
         </joint>
 		    <transmission name="${prefix}joint_finger_${finger_number}_trans">

Commit message: Add torque limit for fingers in kinova_common

File: kinova_description/urdf/kinova_common.xacro (robot description, xacro)
@@ -85,5 +85,5 @@
             <axis xyz="0 0 1"/>
             <origin xyz="${finger_origin_xyz}" rpy="${finger_origin_rpy}"/>
-            <limit lower="0" upper="1.51" effort="2000" velocity="1"/>
+            <limit lower="0" upper="1.51" effort="2" velocity="1"/>
         </joint>
 		    <transmission name="${prefix}joint_finger_${finger_number}_trans">
@@ -103,5 +103,5 @@
             <axis xyz="0 0 1"/>
             <origin xyz="0.044 -0.003 0" rpy="0 0 0"/>
-            <limit lower="0" upper="2" effort="2000" velocity="1"/>
+            <limit lower="0" upper="2" effort="2" velocity="1"/>
         </joint>
         <transmission name="${prefix}joint_finger_tip_${finger_number}_trans">

Commit message: [kinova_description] Omit limits for fixed or continuous joint types
Resolves kinovarobotics/kinova-ros#289

File: kinova_description/urdf/kinova_common.xacro (robot description, xacro)
@@ -49,5 +49,10 @@
         <child link="${child}"/>
         <axis xyz="${joint_axis_xyz}"/>
+        <xacro:if value="${type == 'revolute'}">
         <limit effort="${joint_torque_limit}" velocity="${joint_velocity_limit}" lower="${joint_lower_limit}" upper="${joint_upper_limit}"/>
+        </xacro:if>
+        <xacro:if value="${type == 'continuous'}">
+        <limit effort="${joint_torque_limit}" velocity="${joint_velocity_limit}"/>
+        </xacro:if>
         <origin xyz="${joint_origin_xyz}" rpy="${joint_origin_rpy}"/>
         <dynamics damping="0.0" friction="0.0"/>
@@ -85,5 +90,7 @@
         <child link="${child}"/>
         <axis xyz="${joint_axis_xyz}"/>
+        <xacro:unless value="${type == 'fixed'}">
         <limit effort="2000" velocity="1" lower="${joint_lower_limit}" upper="${joint_upper_limit}"/>
+        </xacro:unless>
         <origin xyz="${joint_origin_xyz}" rpy="${joint_origin_rpy}"/>
      </joint>

Commit message: [kinova_description] Make limits optional and add input validation

File: kinova_description/urdf/kinova_common.xacro (robot description, xacro)
@@ -44,5 +44,34 @@
       </link>
     </xacro:macro>
-  <xacro:macro name="kinova_armjoint" params="joint_name type parent child joint_axis_xyz joint_origin_xyz joint_origin_rpy joint_lower_limit joint_upper_limit joint_velocity_limit joint_torque_limit fixed:=false">
+  <!--
+    We use dummy default values for values only required when type=='revolute':
+    joint_lower_limit and joint_upper_limit (set to 1234567890)
+    We check during macro execution that these values have been set properly if
+    the joint type requires it (revolute).
+    Similarly, we check that velocity and torque limits are set unless the joint
+    type is fixed, and that the fixed parameter is set consistently.
+  -->
+  <xacro:property name="dummy_default_value" value="1234567890"/>
+  <xacro:macro name="kinova_armjoint" params="joint_name
+                                              type
+                                              parent
+                                              child
+                                              joint_axis_xyz
+                                              joint_origin_xyz
+                                              joint_origin_rpy
+                                              joint_lower_limit:=${dummy_default_value}
+                                              joint_upper_limit:=${dummy_default_value}
+                                              joint_velocity_limit:=${dummy_default_value}
+                                              joint_torque_limit:=${dummy_default_value}
+                                              fixed:=false">
+    <xacro:if value="${(type == 'fixed' and not fixed) or (type != 'fixed' and fixed)}"><xacro:ERROR_inconsistent_joint_type_specification/></xacro:if>
+    <xacro:if value="${type == 'revolute'}">
+      <xacro:if value="${joint_lower_limit == dummy_default_value}"><xacro:ERROR_joint_lower_limit_needs_to_be_set_for_a_revolute_joint/></xacro:if>
+      <xacro:if value="${joint_upper_limit == dummy_default_value}"><xacro:ERROR_joint_upper_limit_needs_to_be_set_for_a_revolute_joint/></xacro:if>
+    </xacro:if>
+    <xacro:unless value="${type =='fixed'}">
+      <xacro:if value="${joint_velocity_limit == dummy_default_value}"><xacro:ERROR_joint_velocity_limit_needs_to_be_set_for_a_non_fixed_joint/></xacro:if>
+      <xacro:if value="${joint_torque_limit == dummy_default_value}"><xacro:ERROR_joint_torque_limit_needs_to_be_set_for_a_non_fixed_joint/></xacro:if>
+    </xacro:unless>
     <joint name="${joint_name}" type="${type}">
         <parent link="${parent}"/>
