Commit message: workstation joint_state_publisher implemented, edits to readme formatting

File: urdf/workstation_depth_cameras_gazebo.xacro (robot description, xacro)
@@ -40,11 +40,11 @@
           <alwaysOn>true</alwaysOn>
           <updateRate>0.0</updateRate>
-          <cameraName>left_camera_ir</cameraName>
-          <imageTopicName>/left_camera/color/image_raw</imageTopicName>
-          <cameraInfoTopicName>/left_camera/color/camera_info</cameraInfoTopicName>
-          <depthImageTopicName>/left_camera/depth/image_raw</depthImageTopicName>
-          <depthImageCameraInfoTopicName>/left_camera/depth/camera_info</depthImageCameraInfoTopicName>
-          <pointCloudTopicName>/left_camera/depth/points</pointCloudTopicName>
-          <frameName>"${prefix}left_camera_link"</frameName>
+          <cameraName>camera_ir</cameraName>
+          <imageTopicName>/camera/color/image_raw</imageTopicName>
+          <cameraInfoTopicName>/camera/color/camera_info</cameraInfoTopicName>
+          <depthImageTopicName>/camera/depth/image_raw</depthImageTopicName>
+          <depthImageCameraInfoTopicName>/camera/depth/camera_info</depthImageCameraInfoTopicName>
+          <pointCloudTopicName>/camera/depth/points</pointCloudTopicName>
+          <frameName>${prefix}left_gazebo_depth_camera</frameName>
           <pointCloudCutoff>0.5</pointCloudCutoff>
           <pointCloudCutoffMax>10</pointCloudCutoffMax>

File: urdf/workstation_model.urdf.xacro (robot description, xacro)
@@ -48,5 +48,5 @@
     <axis xyz="0 0 0" />
   </joint>
-  <!-- PEDESTAL LINK -->
+  <!-- TOP CAMERA LINK -->
   <link name="${prefix}top_camera_link">
     <inertial>
@@ -222,4 +222,12 @@
     </collision>
   </link>
+  <!-- Create a virtual joint between left_camera_link and left_gazebo_depth_camera link -->
+  <joint name="${prefix}left_camera_to_left_gazebo_depth_camera_joint" type="fixed">
+    <origin xyz="0.0 0.0 0.1" rpy="0.0 0.0 0.0" />
+    <parent link="${prefix}left_camera_link" />
+    <child link="${prefix}left_gazebo_depth_camera" />
+    <axis xyz="0 0 0" />
+  </joint>
+  <link name="${prefix}left_gazebo_depth_camera" />
   <!-- TABLE TO RIGHT HORIZONTAL ARM JOINT -->
   <joint name="table_to_right_horizontal_arm_joint" type="fixed">

File: urdf/workstation_model_gazebo.xacro (robot description, xacro)
@@ -35,4 +35,7 @@
       <selfCollide>true</selfCollide>
     </gazebo>
+    <gazebo reference="${prefix}left_gazebo_depth_camera">
+      <selfCollide>true</selfCollide>
+    </gazebo>
     <gazebo reference="${prefix}right_horizontal_arm_link">
       <selfCollide>true</selfCollide>

File: urdf/workstation_model_macro.urdf.xacro (robot description, xacro)
@@ -14,6 +14,7 @@
     xmlns:xacro="http://ros.org/wiki/xacro" name="ur5e_d435_millibar_combined_r2f85" >
   <xacro:include filename="$(find uml_hri_nerve_pick_and_place)/urdf/workstation_model.urdf.xacro" />
+  <xacro:workstation prefix="table_"/>
+  <!--
   <link name="world" />
-  <xacro:workstation prefix="table_"/>
   <joint name="world_joint" type="fixed">
     <parent link="world" />
@@ -21,3 +22,4 @@
     <origin xyz="0.0 0.0 0.0" rpy="0.0 0.0 0.0" />
   </joint>
+  -->
 </robot>

Commit message: fixed: workstation gazebo sim; depth camera setup

File: urdf/workstation_depth_cameras_gazebo.xacro (robot description, xacro)
@@ -17,11 +17,12 @@
     <gazebo reference="${prefix}left_camera_link">
       <sensor type="depth" name="left_camera">
-        <pose frame="${prefix}left_camera_link">-0.0125 0.0 0.0 0.0 0.0 0.0</pose>
+      <!-- <pose frame="${prefix}left_camera_link" 0.0 0.0 0.0 0.0 0.0 0.0</pose> -->
         <update_rate>30.0</update_rate>
-        <camera name="head">
-          <horizontal_fov>1.3962634</horizontal_fov>
+        <camera>
+          <pose>0.0 0.0 0.0 0.0 0.0 0.0</pose>
+          <horizontal_fov>1.50098</horizontal_fov>
           <image>
-            <width>640</width>
-            <height>480</height>
+            <width>1280</width>
+            <height>720</height>
             <format>R8G8B8</format>
           </image>
@@ -36,27 +37,17 @@
           </noise>
         </camera>
-        <plugin name="camera_plugin" filename="libgazebo_ros_openni_kinect.so">
+        <plugin name="left_camera_plugin" filename="libgazebo_ros_openni_kinect.so">
           <baseline>0.2</baseline>
           <alwaysOn>true</alwaysOn>
           <updateRate>0.0</updateRate>
-          <cameraName>camera_ir</cameraName>
-          <imageTopicName>/camera/color/image_raw</imageTopicName>
-          <cameraInfoTopicName>/camera/color/camera_info</cameraInfoTopicName>
-          <depthImageTopicName>/camera/depth/image_raw</depthImageTopicName>
-          <depthImageCameraInfoTopicName>/camera/depth/camera_info</depthImageCameraInfoTopicName>
-          <pointCloudTopicName>/camera/depth/points</pointCloudTopicName>
-          <frameName>${prefix}left_gazebo_depth_camera</frameName>
-          <pointCloudCutoff>0.5</pointCloudCutoff>
+          <cameraName>left_camera</cameraName>
+          <imageTopicName>/left_camera/color/image_raw</imageTopicName>
+          <cameraInfoTopicName>/left_camera/color/camera_info</cameraInfoTopicName>
+          <depthImageTopicName>/left_camera/depth/image_raw</depthImageTopicName>
+          <depthImageCameraInfoTopicName>/left_camera/depth/camera_info</depthImageCameraInfoTopicName>
+          <pointCloudTopicName>/left_camera/depth/points</pointCloudTopicName>
+          <frameName>${prefix}left_optical</frameName>
+          <pointCloudCutoff>0.1</pointCloudCutoff>
           <pointCloudCutoffMax>10</pointCloudCutoffMax>
-          <distortionK1>0</distortionK1>
-          <distortionK2>0</distortionK2>
-          <distortionK3>0</distortionK3>
-          <distortionT1>0</distortionT1>
-          <distortionT2>0</distortionT2>
-          <CxPrime>0</CxPrime>
-          <Cx>0</Cx>
-          <Cy>0</Cy>
-          <focalLength>0</focalLength>
-          <hackBaseline>0</hackBaseline>
         </plugin>
       </sensor>
@@ -65,11 +56,11 @@
     <gazebo reference="${prefix}right_camera_link">
       <sensor type="depth" name="right_camera">
-        <pose frame="${prefix}right_camera_link">0.0125 0.0 0.0 0.0 0.0 0.0</pose>
         <update_rate>30.0</update_rate>
-        <camera name="head">
-          <horizontal_fov>1.3962634</horizontal_fov>
+        <camera>
+          <pose>0.0 0.0 0.0 0.0 0.0 0.0</pose>
+          <horizontal_fov>1.50098</horizontal_fov>
           <image>
-            <width>640</width>
-            <height>480</height>
+            <width>1280</width>
+            <height>720</height>
             <format>R8G8B8</format>
           </image>
@@ -84,9 +75,9 @@
           </noise>
         </camera>
-        <plugin name="camera_plugin" filename="libgazebo_ros_openni_kinect.so">
+        <plugin name="right_camera_plugin" filename="libgazebo_ros_openni_kinect.so">
           <baseline>0.2</baseline>
           <alwaysOn>true</alwaysOn>
           <updateRate>0.0</updateRate>
-          <cameraName>right_camera_ir</cameraName>
+          <cameraName>right_camera</cameraName>
           <imageTopicName>/right_camera/color/image_raw</imageTopicName>
           <cameraInfoTopicName>/right_camera/color/camera_info</cameraInfoTopicName>
@@ -94,17 +85,7 @@
           <depthImageCameraInfoTopicName>/right_camera/depth/camera_info</depthImageCameraInfoTopicName>
           <pointCloudTopicName>/right_camera/depth/points</pointCloudTopicName>
-          <frameName>table_right_camera_link</frameName>
-          <pointCloudCutoff>0.5</pointCloudCutoff>
+          <frameName>${prefix}right_optical</frameName>
+          <pointCloudCutoff>0.1</pointCloudCutoff>
           <pointCloudCutoffMax>10</pointCloudCutoffMax>
-          <distortionK1>0</distortionK1>
-          <distortionK2>0</distortionK2>
-          <distortionK3>0</distortionK3>
-          <distortionT1>0</distortionT1>
-          <distortionT2>0</distortionT2>
-          <CxPrime>0</CxPrime>
-          <Cx>0</Cx>
-          <Cy>0</Cy>
-          <focalLength>0</focalLength>
-          <hackBaseline>0</hackBaseline>
         </plugin>
       </sensor>
@@ -113,11 +94,11 @@
     <gazebo reference="${prefix}rear_camera_link">
       <sensor type="depth" name="rear_camera">
-        <pose frame="${prefix}rear_camera_link">-0.0125 0.0 0.0 0.0 0.0 0.0</pose>
         <update_rate>30.0</update_rate>
-        <camera name="head">
-          <horizontal_fov>1.3962634</horizontal_fov>
+        <camera>
+          <pose>0.0 0.0 0.0 0.0 0.0 0.0</pose>
+          <horizontal_fov>1.50098</horizontal_fov>
           <image>
-            <width>640</width>
-            <height>480</height>
+            <width>1280</width>
+            <height>720</height>
             <format>R8G8B8</format>
           </image>
@@ -132,9 +113,9 @@
           </noise>
         </camera>
-        <plugin name="camera_plugin" filename="libgazebo_ros_openni_kinect.so">
+        <plugin name="rear_camera_plugin" filename="libgazebo_ros_openni_kinect.so">
           <baseline>0.2</baseline>
           <alwaysOn>true</alwaysOn>
           <updateRate>0.0</updateRate>
-          <cameraName>rear_camera_ir</cameraName>
+          <cameraName>rear_camera</cameraName>
           <imageTopicName>/rear_camera/color/image_raw</imageTopicName>
           <cameraInfoTopicName>/rear_camera/color/camera_info</cameraInfoTopicName>
@@ -142,17 +123,7 @@
           <depthImageCameraInfoTopicName>/rear_camera/depth/camera_info</depthImageCameraInfoTopicName>
           <pointCloudTopicName>/rear_camera/depth/points</pointCloudTopicName>
-          <frameName>table_rear_camera_link</frameName>
-          <pointCloudCutoff>0.5</pointCloudCutoff>
+          <frameName>${prefix}rear_optical</frameName>
+          <pointCloudCutoff>0.1</pointCloudCutoff>
           <pointCloudCutoffMax>10</pointCloudCutoffMax>
-          <distortionK1>0</distortionK1>
-          <distortionK2>0</distortionK2>
-          <distortionK3>0</distortionK3>
-          <distortionT1>0</distortionT1>
-          <distortionT2>0</distortionT2>
-          <CxPrime>0</CxPrime>
-          <Cx>0</Cx>
-          <Cy>0</Cy>
-          <focalLength>0</focalLength>
-          <hackBaseline>0</hackBaseline>
         </plugin>
       </sensor>
@@ -161,11 +132,11 @@
     <gazebo reference="${prefix}top_camera_link">
       <sensor type="depth" name="top_camera">
-        <pose frame="${prefix}top_camera_link">-0.0125 0.0 0.0 0.0 0.0 0.0</pose>
         <update_rate>30.0</update_rate>
-        <camera name="head">
-          <horizontal_fov>1.3962634</horizontal_fov>
+        <camera>
+          <pose>0.0 0.0 0.0 0.0 0.0 0.0</pose>
+          <horizontal_fov>1.50098</horizontal_fov>
           <image>
-            <width>640</width>
-            <height>480</height>
+            <width>1280</width>
+            <height>720</height>
             <format>R8G8B8</format>
           </image>
@@ -180,9 +151,9 @@
           </noise>
         </camera>
-        <plugin name="camera_plugin" filename="libgazebo_ros_openni_kinect.so">
+        <plugin name="top_camera_plugin" filename="libgazebo_ros_openni_kinect.so">
           <baseline>0.2</baseline>
           <alwaysOn>true</alwaysOn>
           <updateRate>0.0</updateRate>
-          <cameraName>top_camera_ir</cameraName>
+          <cameraName>top_camera</cameraName>
           <imageTopicName>/top_camera/color/image_raw</imageTopicName>
           <cameraInfoTopicName>/top_camera/color/camera_info</cameraInfoTopicName>
@@ -190,17 +161,7 @@
           <depthImageCameraInfoTopicName>/top_camera/depth/camera_info</depthImageCameraInfoTopicName>
           <pointCloudTopicName>/top_camera/depth/points</pointCloudTopicName>
-          <frameName>table_top_camera_link</frameName>
-          <pointCloudCutoff>0.5</pointCloudCutoff>
+          <frameName>${prefix}top_optical</frameName>
+          <pointCloudCutoff>0.1</pointCloudCutoff>
           <pointCloudCutoffMax>10</pointCloudCutoffMax>
-          <distortionK1>0</distortionK1>
-          <distortionK2>0</distortionK2>
-          <distortionK3>0</distortionK3>
-          <distortionT1>0</distortionT1>
-          <distortionT2>0</distortionT2>
-          <CxPrime>0</CxPrime>
-          <Cx>0</Cx>
-          <Cy>0</Cy>
-          <focalLength>0</focalLength>
-          <hackBaseline>0</hackBaseline>
         </plugin>
       </sensor>

File: urdf/workstation_model.urdf.xacro (robot description, xacro)
@@ -20,9 +20,4 @@
   <!-- TABLE BASE LINK -->
   <link name="${prefix}base_link">
-    <inertial>
-      <origin xyz="0 0 1" rpy="0 0 0" />
-      <mass value="1" />
-      <inertia ixx="1" ixy="0" ixz="0" iyy="1" iyz="0" izz="1" />
-    </inertial>
     <visual>
       <origin xyz="0.0 0.0 0.0" rpy="0 0 0" />
@@ -43,5 +38,5 @@
   <!-- TABLE TO TOP CAMERA JOINT -->
   <joint name="table_to_top_camera_joint" type="fixed">
-    <origin xyz="0.0 0.0 1.51" rpy="3.1416 0.0 0.0" />
+    <origin xyz="0.0 0.0 1.5" rpy="0.0 ${pi/2} ${pi/2}" />
     <parent link="${prefix}base_link" />
     <child link="${prefix}top_camera_link" />
@@ -58,17 +53,26 @@
       <origin xyz="0.0 0.0 0.0" rpy="0 0 0" />
       <geometry>
-        <box size="0.09 0.025 0.025"/>
-      </geometry>
-      <material name="">
-        <color rgba="0.79216 0.81961 0.93333 1" />
-      </material>
-    </visual>
-    <collision>
-      <origin xyz="0.0 0.0 0.0" rpy="0 0 0" />
-      <geometry>
-        <box size="0.09 0.025 0.025"/>
-      </geometry>
-    </collision>
-  </link>
+        <box size="0.025 0.09 0.025"/>
+      </geometry>
+      <material name="">
+        <color rgba="0.79216 0.81961 0.93333 1" />
+      </material>
+    </visual>
+    <collision>
+      <origin xyz="0.0 0.0 0.0" rpy="0 0 0" />
+      <geometry>
+        <box size="0.025 0.09 0.025"/>
+      </geometry>
+    </collision>
+  </link>
+  <!-- Create a virtual joint between left_camera_link and left_gazebo_depth_camera link -->
+  <joint name="${prefix}top_camera_to_top_optical_joint" type="fixed">
+    <origin xyz="0.0 0.0 0.0" rpy="${-pi/2} 0.0 ${-pi/2}" />
+    <parent link="${prefix}top_camera_link" />
+    <child link="${prefix}top_optical" />
+    <axis xyz="0 0 0" />
+  </joint>
+  <!-- TOP OPTICAL -->
+  <link name="${prefix}top_optical" />
   <!-- TABLE TO PEDESTAL JOINT -->
   <joint name="table_to_pedestal_joint" type="fixed">
@@ -223,11 +227,12 @@
   </link>
   <!-- Create a virtual joint between left_camera_link and left_gazebo_depth_camera link -->
-  <joint name="${prefix}left_camera_to_left_gazebo_depth_camera_joint" type="fixed">
-    <origin xyz="0.0 0.0 0.1" rpy="0.0 0.0 0.0" />
+  <joint name="${prefix}left_camera_to_left_optical_joint" type="fixed">
+    <origin xyz="0.0 0.0 0.0" rpy="${-pi/2} 0.0 ${-pi/2}" />
     <parent link="${prefix}left_camera_link" />
-    <child link="${prefix}left_gazebo_depth_camera" />
-    <axis xyz="0 0 0" />
-  </joint>
-  <link name="${prefix}left_gazebo_depth_camera" />
+    <child link="${prefix}left_optical" />
+    <axis xyz="0 0 0" />
+  </joint>
+  <!-- LEFT OPTICAL -->
+  <link name="${prefix}left_optical" />
   <!-- TABLE TO RIGHT HORIZONTAL ARM JOINT -->
   <joint name="table_to_right_horizontal_arm_joint" type="fixed">
@@ -290,7 +295,8 @@
     </collision>
   </link>
+  <!-- change these values for camera direction -->
   <!-- RIGHT VERTICAL ARM TO RIGHT CAMERA JOINT -->
   <joint name="right_vertical_arm_to_right_camera_joint" type="fixed">
-    <origin xyz="-0.0325 0.0 -0.125" rpy="0.0 0.0 0.0" />
+    <origin xyz="-0.0325 0.0 -0.125" rpy="0.0 0.0 ${pi}" />
     <parent link="${prefix}right_vertical_arm_link" />
     <child link="${prefix}right_camera_link" />
@@ -320,4 +326,17 @@
     </collision>
   </link>
+  <!-- ${-pi/2} ${pi/2} ${-pi} ${pi} -->
+  <!-- change these values for location of camera frame -->
+  <!-- Create a virtual joint between right_camera_link and right_gazebo_depth_camera link -->
+  <!-- <origin xyz="2.095 0.0 2.075" rpy="0 ${pi} ${pi}" /> OLD_LINE -->
+  <joint name="${prefix}right_camera_to_right_optical_joint" type="fixed">
+    <!-- <origin xyz="0.0 0.0 0.0" rpy="0 0 ${pi}" /> -->
+    <origin xyz="0.0 0.0 0.0" rpy="${-pi/2} 0.0 ${-pi/2}" />
+    <parent link="${prefix}right_camera_link" />
+    <child link="${prefix}right_optical" />
+    <axis xyz="0 0 0" />
+  </joint>
+  <!-- RIGHT OPTICAL -->
+  <link name="${prefix}right_optical" />
   <!-- TABLE TO REAR HORIZONTAL ARM JOINT -->
   <joint name="table_to_rear_horizontal_arm_joint" type="fixed">
@@ -382,5 +401,5 @@
   <!-- REAR VERTICAL ARM TO REAR CAMERA JOINT -->
   <joint name="rear_vertical_arm_to_rear_camera_joint" type="fixed">
-    <origin xyz="0.0 -0.0325 -0.125" rpy="0.0 0.0 0.0" />
+    <origin xyz="0.0 -0.0325 -0.125" rpy="0.0 0.0 ${-pi/2}" />
     <parent link="${prefix}rear_vertical_arm_link" />
     <child link="${prefix}rear_camera_link" />
@@ -397,17 +416,27 @@
       <origin xyz="0.0 0.0 0.0" rpy="0 0 0" />
       <geometry>
-        <box size="0.09 0.025 0.025"/>
-      </geometry>
-      <material name="">
-        <color rgba="0.79216 0.81961 0.93333 1" />
-      </material>
-    </visual>
-    <collision>
-      <origin xyz="0.0 0.0 0.0" rpy="0 0 0" />
-      <geometry>
-        <box size="0.09 0.025 0.025"/>
-      </geometry>
-    </collision>
-  </link>
+        <box size="0.025 0.09 0.025"/>
+      </geometry>
+      <material name="">
+        <color rgba="0.79216 0.81961 0.93333 1" />
+      </material>
+    </visual>
+    <collision>
+      <origin xyz="0.0 0.0 0.0" rpy="0 0 0" />
+      <geometry>
+        <box size="0.025 0.09 0.025"/>
+      </geometry>
+    </collision>
+  </link>
+    <!-- Create a virtual joint between left_camera_link and left_gazebo_depth_camera link -->
+    <!-- <origin xyz="0.9 -1.945 1.035" rpy="0 ${pi/2} 0" /> X=Z, -Y=Y, Z=X OLD_LINE -->
+  <joint name="${prefix}rear_camera_to_rear_optical_joint" type="fixed">
+    <origin xyz="0.0 0.0 0.0" rpy="${-pi/2} 0.0 ${-pi/2}" /> <!-- X=Z, -Y=Y, Z=X-->
+    <parent link="${prefix}rear_camera_link" />
+    <child link="${prefix}rear_optical" />
+    <axis xyz="0 0 0" />
+  </joint>
+  <!-- REAR OPTICAL -->
+  <link name="${prefix}rear_optical" />
   </xacro:macro>
 </robot>

File: urdf/workstation_model_gazebo.xacro (robot description, xacro)
@@ -14,46 +14,26 @@
     xmlns:xacro="http://ros.org/wiki/xacro">
   <xacro:macro name="workstation_gazebo" params="prefix">
-    <gazebo reference="${prefix}base_link">
-      <selfCollide>true</selfCollide>
-    </gazebo>
-    <gazebo reference="${prefix}top_camera_link">
-      <selfCollide>true</selfCollide>
-    </gazebo>
-    <gazebo reference="${prefix}pedestal_link">
-      <selfCollide>true</selfCollide>
-    </gazebo>
-    <gazebo reference="${prefix}mounting_plate_link">
-      <selfCollide>true</selfCollide>
-    </gazebo>
-    <gazebo reference="${prefix}left_horizontal_arm_link">
-      <selfCollide>true</selfCollide>
-    </gazebo>
-    <gazebo reference="${prefix}left_vertical_arm_link">
-      <selfCollide>true</selfCollide>
-    </gazebo>
-    <gazebo reference="${prefix}left_camera_link">
-      <selfCollide>true</selfCollide>
-    </gazebo>
-    <gazebo reference="${prefix}left_gazebo_depth_camera">
-      <selfCollide>true</selfCollide>
-    </gazebo>
-    <gazebo reference="${prefix}right_horizontal_arm_link">
-      <selfCollide>true</selfCollide>
-    </gazebo>
-    <gazebo reference="${prefix}right_vertical_arm_link">
-      <selfCollide>true</selfCollide>
-    </gazebo>
-    <gazebo reference="${prefix}right_camera_link">
-      <selfCollide>true</selfCollide>
-    </gazebo>
-    <gazebo reference="${prefix}rear_horizontal_arm_link">
-      <selfCollide>true</selfCollide>
-    </gazebo>
-    <gazebo reference="${prefix}rear_vertical_arm_link">
-      <selfCollide>true</selfCollide>
-    </gazebo>
-    <gazebo reference="${prefix}rear_camera_link">
-      <selfCollide>true</selfCollide>
-    </gazebo>
+    <!-- Table/Pedestal parts -->
+    <gazebo reference="${prefix}base_link" />
+    <gazebo reference="${prefix}pedestal_link" />
+    <gazebo reference="${prefix}mounting_plate_link" />
+    <!-- Top Camera parts -->
+    <gazebo reference="${prefix}top_camera_link" />
+    <gazebo reference="${prefix}top_optical" />
+    <!-- Left Camera parts -->
+    <gazebo reference="${prefix}left_horizontal_arm_link" />
+    <gazebo reference="${prefix}left_vertical_arm_link" />
+    <gazebo reference="${prefix}left_camera_link" />
+    <gazebo reference="${prefix}left_optical" />
+    <!-- Right Camera parts -->
+    <gazebo reference="${prefix}right_horizontal_arm_link" />
+    <gazebo reference="${prefix}right_vertical_arm_link" />
+    <gazebo reference="${prefix}right_camera_link" />
+    <gazebo reference="${prefix}right_optical" />
+    <!-- Rear Camera parts -->
+    <gazebo reference="${prefix}rear_horizontal_arm_link" />
+    <gazebo reference="${prefix}rear_vertical_arm_link" />
+    <gazebo reference="${prefix}rear_camera_link" />
+    <gazebo reference="${prefix}rear_optical" />
   </xacro:macro>
 </robot>

File: urdf/workstation_model_macro.urdf.xacro (robot description, xacro)
@@ -15,5 +15,5 @@
   <xacro:include filename="$(find uml_hri_nerve_pick_and_place)/urdf/workstation_model.urdf.xacro" />
   <xacro:workstation prefix="table_"/>
-  <!--
+  <!-- This is not required because the "world" link already exists
   <link name="world" />
   <joint name="world_joint" type="fixed">
